File: kicad/main/Main.kicad_pcb (KiCad board)
At the start: 4 copper layers, 115.7 x 88.3 mm, 370 parts, among them CN2 EV2400, IC5 TPS25730DREFR, J2 1-2199119-5, M2_ACT1 YLED0603B, Q1 2302V, Q11 2N3904, Q12 2N3906_C49023424, Q13 2N3906_C49023424, Q14 2N3904, Q15 2N3904, Q2 2302V, Q21 SQJ844AEP-T1_GE3, Q4 SQJ844AEP-T1_GE3, Q6 2302V, Q7 2302V, Q8 AO3401, Q9 2302V, U1 NCP1117ST33T3G, U10 ICS-43434_C5656610, U11 MAX98357AETE_T, U12 XRNR4030-10UH_M, U13 STM32G473VCT6, U14 DRV8870DDAR, U15 DRV8870DDAR, U18 DRV8870DDAR, U19 ICM-42607-P, U20 DRV8870DDAR, U21 AP64501SP-13, U22 AP64501SP-13, U23 BV1HAL45EFJ-E2, U24 AP64501SP-13, U3 STWD100NYWY3F, U4 RS8422XK, U5 MT3608, U6 RT9742GGJ5, U7 BQ25792RQMR, U8 BV1HAL45EFJ-E2, U9 ICS-43434_C5656610, X1 ABM3-8_000MHZ-D2Y-T, X3 XKXEL89CII-SUAYLC-32_768K, Y1 ASEK-32.768KHZ-LRT

Commit message: Cliff/bumper connector reverse engineered
Parts:
- removed C14: 100nF/50V, Capacitor_SMD:C_0603_1608Metric
- removed IMU_IO1: HX_PM2_54-2X8P_WT, JLCImport:HX_PM2_54-2X8P_WT
- removed Q6, Q7: 2302V, JLCImport:2302V
- removed R38, R41: 10k, Resistor_SMD:R_0603_1608Metric
- removed R43: 100k, Resistor_SMD:R_0603_1608Metric
- added MCU_IO1: HX_PM2_54-2X6P_WT, JLCImport:HX_PM2_54-2X6P_WT, F.Cu at (341.7, 76.6)
- added R53: 47k, Resistor_SMD:R_0603_1608Metric, F.Cu at (354.0, 81.4)
- added R64: 47k, Resistor_SMD:R_0603_1608Metric, F.Cu at (354.0, 83.9)
- added R73: 47k, Resistor_SMD:R_0603_1608Metric, F.Cu at (354.0, 86.4)
- C101, C104, C107, C108, C109, C110, C112, C118, C120, C124, C128, C130, C137, C138, C140, C141, C148, C149, C150, C151, C19, C34, C35, C37, C45, C47, C50, C58, C59, C6, C61, C62, C63, C64, C65, C66, C7, C71, C72, C73, C74, C76, C90, C91, C92, D2, D24, D25, D26, D27, D28, D34, D37, D38, D4, D5, IC5, Q1, Q11, R1, R113, R117, R128, R130, R131, R133, R136, R137, R138, R139, R14, R140, R143, R144, R145, R147, R148, R149, R150, R151, R152, R153, R155, R156, R157, R158, R159, R160, R18, R19, R2, R21, R22, R28, R29, R31, R32, R34, R36, R40, R42, R45, R5, R58, R59, R6, R61, R62, R7, R80, R92, R93, R94, R95, U1, U12, U13, U18, U23, U5, U8, X1, Y1: moved to F.Cu
- R35: value 330 -> 22
- R39, R44: value 10k -> 47k; moved to F.Cu
- R48: value 100k -> 47k; moved to F.Cu
- US1: value WAFER-GH1_25-2PWB -> S2B-ZR-SM4A-TF_LF_SN; footprint JLCImport:WAFER-GH1_25-2PWB -> JLCImport:S2B-ZR-SM4A-TF_LF_SN
- moved R80 263.2 mm to (399.6, 99.0), turned to 180 degrees
- moved R95 263.0 mm to (399.6, 110.2), turned to 0 degrees
- moved R94 263.0 mm to (399.6, 111.8)
- moved C37 260.9 mm to (396.1, 117.8), turned to 180 degrees
- moved C33 257.2 mm to (399.6, 108.7)
- moved C31 254.9 mm to (399.6, 104.0), turned to 0 degrees
- moved C32 254.7 mm to (399.6, 107.1), turned to 0 degrees
- moved R21 254.0 mm to (392.8, 119.7), turned to 90 degrees
- moved C16 251.6 mm to (399.6, 100.6), turned to 0 degrees
- moved C30 247.3 mm to (399.6, 105.6), turned to 0 degrees
- moved C35 244.1 mm to (389.2, 124.3), turned to 180 degrees
- moved R19 242.7 mm to (388.9, 118.2), turned to 0 degrees
- moved X1 240.9 mm to (387.6, 121.1), turned to 0 degrees
- moved U13 239.8 mm to (387.3, 106.1)
- moved JTAG1 239.0 mm to (353.8, 111.9)
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Connections:
- net /CLIFF/L1- renamed /CLIFF/BUMPER_LED_EN
- net /CLIFF/R2+ renamed Net-(BUMP_CLIFF1-Pad15)
- net /CLIFF/RR+ renamed Net-(BUMP_CLIFF1-Pad1)
- BUMP_CLIFF1 pad 11: /CLIFF/ANTI-FALL-RIGHT-UP-ADC -> /CLIFF/BUMP-L-Q+
- BUMP_CLIFF1 pad 12: /CLIFF/ANTI-FALL-LEFT-UP-ADC -> GND
- BUMP_CLIFF1 pad 13: VCC-3V3-P -> /CLIFF/BUMP-R-Q+
- BUMP_CLIFF1 pad 14: VCC-3V3-P -> GND
- BUMP_CLIFF1 pad 2: /CLIFF/LR- -> /CLIFF/CLIFF_LED_EN
- BUMP_CLIFF1 pad 3: /CLIFF/ANTI-FALL-RIGHT-DOWN-ADC -> /CLIFF/RR-Q+
- BUMP_CLIFF1 pad 4: /CLIFF/ANTI-FALL-LEFT-DOWN-ADC -> GND
- BUMP_CLIFF1 pad 5: VCC-3V3-P -> /CLIFF/RF-Q+
- BUMP_CLIFF1 pad 6: VCC-3V3-P -> GND
- BUMP_CLIFF1 pad 7: GND -> /CLIFF/LF-Q+
- BUMP_CLIFF1 pad 9: GND -> /CLIFF/LR-Q+
- Q8 pad 1: Net-(Q7-D) -> /MCU-STM32/WATER-PUMPU-CTRL
- R25 pad 1: Net-(Q7-D) -> /MCU-STM32/WATER-PUMPU-CTRL
- R35 pad 2: VCC-5V-REG -> VCC-3V3-P
- R39 pad 1: /CLIFF/ANTI-FALL-RIGHT-UP-ADC -> /CLIFF/RR-Q+
- R39 pad 2: GND -> VCC-3V3-P
- R44 pad 1: /CLIFF/ANTI-FALL-RIGHT-DOWN-ADC -> /CLIFF/BUMP-R-Q+
- R44 pad 2: GND -> VCC-3V3-P
- R48 pad 1: /CLIFF/CLIFF_LED_EN -> /CLIFF/BUMP-L-Q+
- R48 pad 2: GND -> VCC-3V3-P
- U13 pad 19: /MCU-STM32/PF2 -> /BUTTON-LED/LED-PWR
- U13 pad 20: /CLIFF/ANTI-FALL-LEFT-UP-ADC -> /CLIFF/RR-Q+
- U13 pad 21: /CLIFF/ANTI-FALL-LEFT-DOWN-ADC -> /CLIFF/RF-Q+
- U13 pad 22: /CLIFF/ANTI-FALL-RIGHT-UP-ADC -> /CLIFF/LR-Q+
- U13 pad 25: /CLIFF/ANTI-FALL-RIGHT-DOWN-ADC -> /CLIFF/LF-Q+
- U13 pad 26: /MAIN-BRUSH MOTOR/MAIN-BRUSH-CURRENT-ADC -> /CLIFF/BUMP-L-Q+
- U13 pad 27: /MCU-STM32/WATER-PUMP-SENSE-ADC -> /CLIFF/BUMP-R-Q+
- U13 pad 28: /BUTTON-LED/LED-PWR -> /MAIN-BRUSH MOTOR/MAIN-BRUSH-CURRENT-ADC
- U13 pad 29: /MCU-STM32/PA7 -> /MCU-STM32/WATER-PUMP-SENSE-ADC
