File: kicad/main/Main.kicad_pcb (KiCad board)
At the start: 4 copper layers, 146.1 x 105.2 mm, 377 parts, among them CN1 91302-85-067RDM, CN2 EV2400, IC5 TPS25730DREFR, M2_ACT2 YLED0603B, Q1 2302V, Q11 2N3904, Q12 2N3906_C49023424, Q13 2N3906_C49023424, Q14 2N3904, Q15 2N3904, Q2 2302V, Q21 SQJ844AEP-T1_GE3, Q3 2302V, Q4 SQJ844AEP-T1_GE3, Q8 AO3401, Q9 2302V, T1 NTCG164KF104FT1, U1 NCP1117ST33T3G, U10 ICS-43434_C5656610, U11 MAX98357AETE_T, U12 XRNR4030-10UH_M, U13 STM32G473VCT6, U14 DRV8870DDAR, U15 DRV8870DDAR, U18 DRV8870DDAR, U19 ICM-42607-P, U20 DRV8870DDAR, U21 AP64501SP-13, U22 AP64501SP-13, U23 BV1HAL45EFJ-E2, U24 AP64501SP-13, U3 STWD100NYWY3F, U4 RS8422XK, U5 MT3608, U6 RT9742GGJ5, U7 BQ25792RQMR, U8 BV1HAL45EFJ-E2, U9 ICS-43434_C5656610, X1 ABM3-8_000MHZ-D2Y-T, X3 XKXEL89CII-SUAYLC-32_768K, Y2 ASEK-32.768KHZ-LRT

Commit message: STM32 power rail switch
Parts:
- removed C47, C58: 330pF/25V, Capacitor_SMD:C_0603_1608Metric
- removed C59, C61, C65, C73: 100nF/50V, Capacitor_SMD:C_0603_1608Metric
- removed C60, C66, C71, C72, C74, C76, C94: 10uF/25V, Capacitor_SMD:C_0603_1608Metric
- removed D40: BZT52C12T-7, JLCImport:BZT52C12T-7
- removed IC5: TPS25730DREFR, LIB_TPS25730DREFR:TPS25730DREFR
- removed Q21: SQJ844AEP-T1_GE3, JLCImport:SQJ844AEP-T1_GE3
- removed R128, R130, R133, R138, R139: 100k, Resistor_SMD:R_0603_1608Metric
- removed R131: 20k, Resistor_SMD:R_0603_1608Metric
- removed R136, R137: 5.24k, Resistor_SMD:R_0603_1608Metric
- removed R140: 1k, Resistor_SMD:R_0603_1608Metric
- removed R150: 10k, Resistor_SMD:R_0603_1608Metric
- removed R151: 47k, Resistor_SMD:R_0603_1608Metric
- removed R158: 100, Resistor_SMD:R_0805_2012Metric
- removed R75: 100, Resistor_SMD:R_0603_1608Metric
- removed U1: NCP1117ST33T3G, NCP1117ST33T3G:SOT230P700X180-4N
- removed U8: BV1HAL45EFJ-E2, JLCImport:BV1HAL45EFJ-E2
- added 3.3V_SENSORS1: 3V3_SENSORS, oomwoo_altium:LED0603-B, F.Cu at (211.0, 123.1)
- added 5V1: ~, oomwoo_altium:LED0603-B, F.Cu at (180.6, 100.5)
- added C139: 10uF/25V, Capacitor_SMD:C_0603_1608Metric, F.Cu at (105.0, 59.0)
- added C154: 10uF/25V, Capacitor_SMD:C_0603_1608Metric, F.Cu at (104.8, 57.3)
- added C155: 100nF/25V, Capacitor_SMD:C_0603_1608Metric, F.Cu at (105.0, 60.6)
- added C156: 100nF/25V, Capacitor_SMD:C_0603_1608Metric, F.Cu at (100.3, 62.5)
- added C157: 100nF/25V, Capacitor_SMD:C_0603_1608Metric, F.Cu at (109.4, 64.0)
- added C159: 10uF/6.3V, Capacitor_SMD:C_0603_1608Metric, F.Cu at (100.3, 67.2)
- added C160: 10uF/6.3V, Capacitor_SMD:C_0603_1608Metric, F.Cu at (100.6, 58.6)
- added C161: 10uF/6.3V, Capacitor_SMD:C_0603_1608Metric, F.Cu at (96.4, 79.2)
- added C162: 1.2nF/50V, Capacitor_SMD:C_0603_1608Metric, F.Cu at (96.9, 70.9)
- added C163: 100nF/10V, Capacitor_SMD:C_0603_1608Metric, F.Cu at (94.4, 70.9)
- added C85: 1.2nF/50V, Capacitor_SMD:C_0603_1608Metric, F.Cu at (100.5, 60.5)
- added D10: SS34, Diode_SMD:D_SMA, F.Cu at (91.7, 73.9)
- added D11: SS34, Diode_SMD:D_SMA, F.Cu at (189.7, 59.5)
- added DC1: DC-005-5A-2_0, JLCImport:DC-005-5A-2_0, F.Cu at (216.9, 69.6)
- added L5: CYA0630-3_3UH, JLCImport:CYA0630-3_3UH, F.Cu at (104.2, 74.6)
- added Q10: AO3401, oomwoo_altium:SOT23-3D, F.Cu at (199.2, 95.0)
- added Q16: AO3401, oomwoo_altium:SOT23-3D, F.Cu at (204.8, 128.2)
- added Q17: AO3401, oomwoo_altium:SOT23-3D, F.Cu at (204.7, 124.3)
- added Q19: 2302V, JLCImport:2302V, F.Cu at (192.4, 135.3)
- added Q20: AO3400, oomwoo_altium:SOT23-3D, F.Cu at (183.3, 63.0)
- added R101: 215k, Resistor_SMD:R_0603_1608Metric, F.Cu at (98.7, 76.5)
- added R102: 10k, Resistor_SMD:R_0603_1608Metric, F.Cu at (103.5, 113.6)
- added R161: 10, Resistor_SMD:R_0603_1608Metric, F.Cu at (109.4, 67.9)
- added R162: 20k, Resistor_SMD:R_0603_1608Metric, F.Cu at (96.6, 66.9)
- added R163: 12k, Resistor_SMD:R_0603_1608Metric, F.Cu at (96.6, 64.4)
- added R164: 2.2k, Resistor_SMD:R_0603_1608Metric, F.Cu at (96.6, 61.9)
- added R165: 100k, Resistor_SMD:R_0603_1608Metric, F.Cu at (179.4, 134.6)
- added R166: 100k, Resistor_SMD:R_0603_1608Metric, F.Cu at (189.5, 134.7)
- added R168: 100k, Resistor_SMD:R_0603_1608Metric, F.Cu at (169.4, 98.5)
- added R41: 100k, Resistor_SMD:R_0603_1608Metric, F.Cu at (98.7, 73.3)
- added R43: 100k, Resistor_SMD:R_0603_1608Metric, F.Cu at (100.5, 65.1)
- added R74: 100k, Resistor_SMD:R_0603_1608Metric, F.Cu at (98.6, 138.0)
- added R79: 10, Resistor_SMD:R_0603_1608Metric, F.Cu at (207.8, 94.5)
- added R88: 10, Resistor_SMD:R_0603_1608Metric, F.Cu at (207.8, 97.0)
- added R89: 1k, Resistor_SMD:R_0603_1608Metric, F.Cu at (181.2, 92.5)
- added R90: 10k, Resistor_SMD:R_0603_1608Metric, F.Cu at (201.0, 130.6)
- added R91: 10k, Resistor_SMD:R_0603_1608Metric, F.Cu at (203.6, 130.6)
- added R96: 10, Resistor_SMD:R_0603_1608Metric, F.Cu at (206.1, 130.6)
- added R97: 10, Resistor_SMD:R_0603_1608Metric, F.Cu at (208.6, 130.6)
- added R98: 1k, Resistor_SMD:R_0603_1608Metric, F.Cu at (211.1, 130.6)
- added U16: HT7533-1_C14289, JLCImport:HT7533-1_C14289, F.Cu at (181.5, 80.1)
- added U2: TMI6240, JLCImport:TMI6240, F.Cu at (95.9, 76.5)
- added U25: AP64501SP-13, JLCImport:AP64501SP-13, F.Cu at (105.2, 65.9)
- C10: value 100nF/50V -> 100nF/10V
- C102, C103, C107, C111, C117, C118, C119, C127, C128, C129, C18, C21, C22, C84, C88, C92: value 100nF/50V -> 100nF/25V
- C108, C113, C114, C131, C132, C144, C145, C146, C17, C19, C20, C23, C24, C31, C33, C6, C90, C91: value 10uF/25V -> 10uF/6.3V
- C109, C12, C13, C142, C143, C15, C16, C30, C32, C36, C37, C5, C51, C56, C9: value 100nF/50V -> 100nF/6.3V
- C11, C121, C122, C133, C147, C148, C149, C152, C153, C63: value 10uF/25V -> 10uF/10V
- C125: value 1nF/50V -> 10uF/50V; footprint Capacitor_SMD:C_0603_1608Metric -> Capacitor_SMD:C_0805_2012Metric
- C126: value 1nF/50V -> 100nF/25V
- C39, C42: value 18pF/10V -> 18pF/50V
- C64: value 100nF/50V -> 10uF/6.3V
- C67, C68, C69, C78, C80, C81, C82: value 10uF/25V -> 10uF/50V; footprint Capacitor_SMD:C_0603_1608Metric -> Capacitor_SMD:C_0805_2012Metric
- C70: value 10uF/25V -> 4.7uF/10V
- D1: value TVS2200DRVR -> SMBJ24A_C908801; footprint JLCImport:TVS2200DRVR -> JLCImport:SMBJ24A_C908801
- D2: value TVS2200DRVR -> ZMM9V1_C2891750; footprint JLCImport:TVS2200DRVR -> JLCImport:ZMM9V1_C2891750
- D39: value BZT52C12T-7 -> SS34; footprint JLCImport:BZT52C12T-7 -> Diode_SMD:D_SMA
- MCU_IO1: value HX_PM2_54-2X6P_WT -> HX_PM2_54-2X4P_WT; footprint JLCImport:HX_PM2_54-2X6P_WT -> JLCImport:HX_PM2_54-2X4P_WT
- Q1: value 2302V -> AOD407_C6396162; footprint JLCImport:2302V -> JLCImport:AOD407_C6396162
- Q4: value SQJ844AEP-T1_GE3 -> AOD407_C6396162; footprint JLCImport:SQJ844AEP-T1_GE3 -> JLCImport:AOD407_C6396162
- R36, R42: value 10k -> 10
- R76: value 100 -> 10k
- moved USB2 140.8 mm to (84.2, 73.7), turned to -90 degrees
- moved D35 130.8 mm to (217.5, 107.1), turned to 0 degrees
- moved D34 122.7 mm to (95.3, 73.9), turned to 180 degrees
- moved FAN1 120.8 mm to (172.0, 148.2), turned to 0 degrees
- moved D9 115.5 mm to (170.4, 141.2), turned to 90 degrees
- moved Q3 114.3 mm to (174.8, 143.0), turned to 90 degrees
- moved R87 109.0 mm to (175.0, 139.9), turned to 0 degrees
- moved C126 99.2 mm to (109.0, 112.6), turned to 0 degrees
- moved R42 89.4 mm to (184.9, 134.6), turned to 90 degrees
- moved Q1 79.5 mm to (177.1, 127.1), turned to -90 degrees
- moved R36 75.8 mm to (174.8, 134.6)
- moved C64 53.6 mm to (200.3, 126.1), turned to 90 degrees
- moved Q8 49.8 mm to (204.6, 93.4)
- moved R25 49.8 mm to (203.6, 91.6)
- moved Q4 40.4 mm to (187.2, 127.1)
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- renumbered D23 to 3.3V_STM1
Connections:
- 3.3V_STM1 pad 1: VCC-3V3-P -> VCC-3V3
- BAT2 pad 1: /BATTERY-CHARGER/P+/C+ -> Net-(BAT2-Pad1)
- C1 pad 1: +3.3VP -> 3.3V-PI
- C100 pad 2: Net-(U7-SYS) -> BAT-VCC
- C108 pad 2: VCC-3V3-P -> VCC-3V3-REG
- C109 pad 2: VCC-3V3-P -> VCC-3V3-REG
- C110 pad 2: VCC-3V3-P -> VCC-3V3-REG
- C113 pad 1: VCC-3V3-P -> VCC-3V3
- C114 pad 1: VCC-3V3-P -> VCC-3V3
- C12 pad 1: VCC-3V3-P -> VCC-3V3
- C125 pad 1: Net-(D39-A) -> VCC-CHARGE
- C125 pad 2: Net-(D39-K) -> GND
- C126 pad 1: Net-(D40-A) -> Net-(C126-Pad1)
- C126 pad 2: Net-(D40-K) -> /BUTTON-LED/POWER-BTN
- C13 pad 1: VCC-3V3-P -> VCC-3V3
- C140 pad 1: Net-(U1-IN) -> Net-(D2-A)
- C142 pad 1: VCC-3V3-P -> VCC-3V3-REG
- C143 pad 1: VCC-3V3-P -> VCC-3V3-REG
- C146 pad 1: VCC-3V3-P -> VCC-3V3
- C15 pad 1: VCC-3V3-P -> VCC-3V3
- C16 pad 1: VCC-3V3-P -> VCC-3V3
- C17 pad 1: VCC-3V3-P -> VCC-3V3
- C19 pad 1: VCC-3V3-P -> VCC-3V3-REG
- C20 pad 1: VCC-3V3-P -> VCC-3V3-REG
- C23 pad 1: VCC-3V3-P -> VCC-3V3-REG
- C24 pad 1: VCC-3V3-P -> VCC-3V3-REG
- C30 pad 1: VCC-3V3-P -> VCC-3V3
- C31 pad 1: VCC-3V3-P -> VCC-3V3
- C32 pad 1: VCC-3V3-P -> VCC-3V3
- C33 pad 1: VCC-3V3-P -> VCC-3V3
- C5 pad 1: VCC-3V3-P -> VCC-3V3-REG
- C56 pad 1: VCC-3V3-P -> VCC-3V3
- C6 pad 1: Net-(C6-Pad1) -> VCC-3V3-REG
- C64 pad 1: GND -> VCC-3V3-REG
- C64 pad 2: /BATTERY-CHARGER/VBUS -> /MCU-STM32/3.3V_EN
- C67 pad 2: VCC-CHARG -> VCC-CHARGE
- C68 pad 2: VCC-CHARG -> VCC-CHARGE
- C69 pad 1: VCC-CHARG -> VCC-CHARGE
- C7 pad 1: Net-(Q1-D) -> /MAIN-FAN/MAIN-FAN-S-CTRL
- C83 pad 1: Net-(U7-SYS) -> BAT-VCC
- C9 pad 1: VCC-3V3-P -> VCC-3V3-REG
- C90 pad 1: VCC-3V3-P -> VCC-3V3-REG
- C91 pad 1: VCC-3V3-P -> VCC-3V3-REG
- C96 pad 2: Net-(U7-SYS) -> BAT-VCC
- C97 pad 2: Net-(U7-SYS) -> BAT-VCC
- C98 pad 2: Net-(U7-SYS) -> BAT-VCC
- C99 pad 2: Net-(U7-SYS) -> BAT-VCC
- CAM0 pad 15: VCC-3V3-P -> VCC-3V3-REG
- CM_IO1 pad 11: VCC-3V3-P -> VCC-3V3-REG
- CM_IO1 pad 12: GND -> VCC-5V-REG
- CM_IO1 pad 2: /CM5-GPIO/GPIO9 -> /CM5-GPIO/GPIO11
- CM_IO1 pad 4: /CM5-GPIO/GPIO11 -> /CM5-GPIO/GPIO23
- CM_IO1 pad 6: /CM5-GPIO/GPIO23 -> /CM5-GPIO/GPIO13
- CM_IO1 pad 8: /CM5-GPIO/GPIO13 -> GND
- CM_IO1 pad 9: VCC-3V3-P -> GND
- CN1 pad 70: unconnected-(CN1-Pad70) -> VCC3V3_M2
- CN1 pad 72: unconnected-(CN1-Pad72) -> VCC3V3_M2
- CN1 pad 76: unconnected-(CN1-Pad76) -> GND
- CN1 pad 77: unconnected-(CN1-Pad77) -> GND
- CONTACT_CHGR1 pad 1: GND -> Net-(CONTACT_CHGR1-Pad1)
- CONTACT_CHGR1 pad 2: GND -> Net-(CONTACT_CHGR1-Pad1)
- CONTACT_CHGR1 pad 3: Net-(Q4-D2) -> VCC-CHARGE
- CONTACT_CHGR1 pad 4: Net-(Q4-D2) -> VCC-CHARGE
- D1 pad 1: GND -> VCC-CHARGE
- D2 pad 1: GND -> BAT-VCC
- D2 pad 2: GND -> Net-(D2-A)
- D39 pad 1: Net-(D39-K) -> /MCU-STM32/3.3V_EN
- D39 pad 2: Net-(D39-A) -> VCC-3V3-REG
- D5 pad 1: VCC-3V3-P -> VCC-3V3
- D7 pad 1: VCC-3V3-P -> VCC-3V3-REG
- F1 pad 1: Net-(U7-SYS) -> /BATTERY-CHARGER/P+/C+
- F1 pad 2: BAT-VCC -> Net-(BAT2-Pad1)
- FAN1 pad 0: unconnected-(FAN1-Pad0) -> GND
- IR-F1 pad 1: VCC-3V3-P -> VCC-3V3-REG
- IR-F2 pad 1: VCC-3V3-P -> VCC-3V3-REG
- L2 pad 2: VCC-3V3-P -> VCC-3V3
- LIGHT1 pad 1: VCC-3V3-P -> VCC-3V3-REG
- MAIN_FAN1 pad 2: Net-(Q1-D) -> /MAIN-FAN/MAIN-FAN-S-CTRL
- MCU_IO1 pad 1: /MCU-STM32/PB3 -> VCC-3V3-REG
- MCU_IO1 pad 2: /MCU-STM32/PA10 -> GND
- MCU_IO1 pad 4: /MCU-STM32/PB4 -> /MCU-STM32/PB6
- MCU_IO1 pad 6: /MCU-STM32/PB6 -> /MCU-STM32/PE15
- MCU_IO1 pad 7: /MCU-STM32/PC10 -> /MCU-STM32/PF2
- MCU_IO1 pad 8: /MCU-STM32/PE15 -> /MCU-STM32/PC13
- MIPI0 pad 15: VCC-3V3-P -> VCC-3V3-REG
- MIPI1 pad 15: VCC-3V3-P -> VCC-3V3-REG
- MOT_WHEEL_L1 pad 5: VCC-3V3-P -> VCC-3V3-REG
- MOT_WHEEL_R1 pad 5: VCC-3V3-P -> VCC-3V3-REG
- Module1 pad 19: Net-(Module1A-FAN_PWM) -> unconnected-(Module1A-FAN_PWM-Pad19)
- Module1 pad 40: /CM5-GPIO/GPIO9 -> /CM5-GPIO/PI_DONE
- Module1 pad 78: +3.3VP -> 3.3V-PI
- Module1 pad 84: +3.3VP -> 3.3V-PI
- Module1 pad 86: +3.3VP -> 3.3V-PI
- Q1 pad 1: VCC-3V3-P -> Net-(Q1-G)
- Q1 pad 2: /MAIN-FAN/MAIN-FAN-S-CTRL -> VM-VBAT
- Q1 pad 3: Net-(Q1-D) -> BAT-VCC
- Q4 pad 1: Net-(D39-A) -> Net-(Q4-G)
- Q4 pad 2: Net-(D39-K) -> VM-VBAT
- Q4 pad 3: Net-(D39-A) -> BAT-VCC
- Q8 pad 1: /MCU-STM32/WATER-PUMPU-CTRL -> Net-(Q8-G)
- R1 pad 1: VCC-3V3-P -> VCC-3V3-REG
- R120 pad 2: VCC-3V3-P -> VCC-3V3-REG
- R121 pad 2: VCC-3V3-P -> VCC-3V3-REG
- R13 pad 1: +3.3VP -> 3.3V-PI
- R132 pad 2: VCC-3V3-P -> VCC-3V3
- R142 pad 1: +3.3VP -> 3.3V-PI
- R144 pad 2: VCC-3V3-P -> VCC-3V3
- R16 pad 1: +3.3VP -> /POWER/POWER-EN
- R18 pad 1: VCC-3V3-P -> VCC-3V3-REG
- R21 pad 2: VCC-3V3-P -> VCC-3V3
- R23 pad 1: +3.3VP -> 3.3V-PI
- R31 pad 2: VCC-CHARG -> VCC-CHARGE
- R35 pad 2: VCC-3V3-P -> VCC-3V3-REG
- R36 pad 1: VCC-5V-REG -> Net-(Q19-D)
- R36 pad 2: Net-(Q1-D) -> Net-(Q1-G)
- R39 pad 2: VCC-3V3-P -> VCC-3V3-REG
- R42 pad 1: VCC-3V3-P -> Net-(Q19-D)
- R42 pad 2: /MAIN-FAN/MAIN-FAN-S-CTRL -> Net-(Q4-G)
- R44 pad 2: VCC-3V3-P -> VCC-3V3-REG
- R45 pad 1: /BUTTON-LED/POWER-BTN -> Net-(C126-Pad1)
- R48 pad 2: VCC-3V3-P -> VCC-3V3-REG
- R49 pad 1: VCC-3V3-P -> VCC-3V3-REG
- R5 pad 1: VCC-3V3-P -> VCC-3V3-REG
- R50 pad 1: VCC-3V3-P -> VCC-3V3-REG
- R51 pad 1: VCC-3V3-P -> VCC-3V3-REG
- R52 pad 1: VCC-3V3-P -> VCC-3V3-REG
- R53 pad 2: VCC-3V3-P -> VCC-3V3-REG
- R6 pad 1: VCC-3V3-P -> VCC-3V3-REG
- R61 pad 1: VCC-3V3-P -> VCC-3V3-REG
- R62 pad 1: VCC-3V3-P -> VCC-3V3-REG
- R64 pad 2: VCC-3V3-P -> VCC-3V3-REG
- R69 pad 1: VCC-3V3-P -> VCC-3V3-REG
- R7 pad 1: VCC-3V3-P -> VCC-3V3-REG
- R72 pad 1: VCC-3V3-P -> VCC-3V3-REG
- R73 pad 2: VCC-3V3-P -> VCC-3V3-REG
- R76 pad 1: Net-(D40-K) -> /MCU-STM32/WATER-PUMPU-CTRL
- R76 pad 2: Net-(U7-ACDRV1) -> VM-5V
- R85 pad 1: +3.3VP -> 3.3V-PI
- R87 pad 1: Net-(Module1A-FAN_PWM) -> /MCU-STM32/BOARD_FAN
- R92 pad 1: VCC-3V3-P -> VCC-3V3-REG
- R93 pad 1: VCC-3V3-P -> VCC-3V3-REG
- SIDE-L1 pad 1: VCC-3V3-P -> VCC-3V3-REG
- SIDE-R1 pad 1: VCC-3V3-P -> VCC-3V3-REG
- T1 pad 2: VCC-3V3-P -> VCC-3V3
- U10 pad 2: VCC-3V3-P -> VCC-3V3-REG
- U10 pad 5: VCC-3V3-P -> VCC-3V3-REG
- U13 pad 100: VCC-3V3-P -> VCC-3V3
- U13 pad 24: VCC-3V3-P -> VCC-3V3
- U13 pad 36: VCC-3V3-P -> VCC-3V3
- U13 pad 37: VCC-3V3-P -> VCC-3V3
- U13 pad 49: VCC-3V3-P -> VCC-3V3
- U13 pad 64: VCC-3V3-P -> VCC-3V3
- U13 pad 71: /MCU-STM32/PA10 -> /MCU-STM32/BOARD_FAN
- U13 pad 75: VCC-3V3-P -> VCC-3V3
- U13 pad 79: /MCU-STM32/PC10 -> /BATTERY-CHARGER/PWR_EN
- U13 pad 90: /MCU-STM32/PB3 -> /MCU-STM32/3.3V_EN
- U13 pad 91: /MCU-STM32/PB4 -> /MCU-STM32/5V_EN
- U13 pad 92: /MCU-STM32/PB5 -> /CM5-GPIO/PI_DONE
- U14 pad 4: VCC-3V3-P -> VCC-3V3-REG
- U15 pad 4: VCC-3V3-P -> VCC-3V3-REG
- U18 pad 4: VCC-3V3-P -> VCC-3V3-REG
- U19 pad 12: VCC-3V3-P -> VCC-3V3-REG
- U19 pad 5: VCC-3V3-P -> VCC-3V3-REG
- U19 pad 8: VCC-3V3-P -> VCC-3V3-REG
- U20 pad 4: VCC-3V3-P -> VCC-3V3-REG
- U21 pad 3: +3.3VP -> /POWER/POWER-EN
- U22 pad 3: /POWER/POWER-EN -> /MCU-STM32/5V_EN
- U3 pad 5: VCC-3V3-P -> VCC-3V3
- U6 pad 5: +3.3VP -> 3.3V-PI
- U7 pad 10: Net-(U7-ACDRV2) -> GND
- U7 pad 11: Net-(U7-ACDRV1) -> GND
- U7 pad 2: VCC-CHARG -> VCC-CHARGE
- U7 pad 25: Net-(U7-SYS) -> BAT-VCC
- U7 pad 3: VCC-CHARG -> VCC-CHARGE
- U7 pad 8: Net-(Q4-D2) -> VCC-CHARGE
- U7 pad 9: /BATTERY-CHARGER/VOUT_PD -> VCC-CHARGE
- U9 pad 5: VCC-3V3-P -> VCC-3V3-REG
- USB2 pad A5: /BATTERY-CHARGER/CC1 -> unconnected-(USB2-CC1-PadA5)
- USB2 pad B5: /BATTERY-CHARGER/CC2 -> unconnected-(USB2-CC2-PadB5)
- VL-L1 pad 1: Net-(C6-Pad1) -> VCC-3V3-REG
- VL-R1 pad 1: VCC-3V3-P -> VCC-3V3-REG
