File: kicad/main/Main.kicad_pcb (KiCad board)
At the start: 4 copper layers, 146.1 x 105.2 mm, 391 parts, among them CN1 91302-85-067RDM, CN2 EV2400, M2_ACT2 YLED0603B, Q1 AOD407_C6396162, Q10 AO3401, Q11 2N3904, Q12 2N3906_C49023424, Q13 2N3906_C49023424, Q14 2N3904, Q15 2N3904, Q16 AO3401, Q17 AO3401, Q19 2302V, Q2 2302V, Q20 AO3400, Q3 2302V, Q4 AOD407_C6396162, Q8 AO3401, Q9 2302V, T1 NTCG164KF104FT1, U10 ICS-43434_C5656610, U11 MAX98357AETE_T, U12 XRNR4030-10UH_M, U13 STM32G473VCT6, U14 DRV8870DDAR, U15 DRV8870DDAR, U16 HT7533-1_C14289, U18 DRV8870DDAR, U19 ICM-42607-P, U2 TMI6240, U20 DRV8870DDAR, U21 AP64501SP-13, U22 AP64501SP-13, U23 BV1HAL45EFJ-E2, U24 AP64501SP-13, U25 AP64501SP-13, U3 STWD100NYWY3F, U4 RS8422XK, U5 MT3608, U6 RT9742GGJ5, U7 BQ25792RQMR, U9 ICS-43434_C5656610, X1 ABM3-8_000MHZ-D2Y-T, X3 XKXEL89CII-SUAYLC-32_768K, Y2 ASEK-32.768KHZ-LRT

Commit message: LDR
Parts:
- removed MCU_IO1: HX_PM2_54-2X4P_WT, JLCImport:HX_PM2_54-2X4P_WT
- added R103: 10k, Resistor_SMD:R_0603_1608Metric, F.Cu at (154.6, 128.0)
- added R75: GL5537-1, JLCImport:GL5537-1, F.Cu at (154.6, 134.0)
Connections:
- CM_IO1 pad 1: /CM5-GPIO/GPIO10 -> GND
- Module1 pad 44: /CM5-GPIO/GPIO10 -> /CM5-GPIO/PI_SHUTDOWN
- U13 pad 5: /MCU-STM32/PE6 -> unconnected-(U13B-PE6-Pad5)
- U13 pad 51: /BUTTON-LED/LED-HOME -> Net-(U13A-PB12)
- U13 pad 7: /MCU-STM32/PC13 -> /BUTTON-LED/LED-HOME
- U13 pad 93: /MCU-STM32/PB6 -> /CM5-GPIO/PI_SHUTDOWN
