File: kicad/main/STM32G070RBT6.kicad_sch (KiCad schematic)
At the start: 33 parts, among them U13 STM32G473VCT6, X1 ABM3-8_000MHZ-D2Y-T, X3 XKXEL89CII-SUAYLC-32_768K

Commit message: Cliff/bumpers connector
Changed lines of the file:
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@@
 	(generator_version "10.0")
 	(paper "A2")
+	(rectangle
+		(start 403.86 232.41)
+		(end 406.4 254)
+		(stroke
+			(width 0)
+			(type solid)
+		)
+		(fill
+			(type color)
+			(color 72 0 0 1)
+		)
+	)
+	(rectangle
+		(start 478.79 232.41)
+		(end 481.33 254)
+		(stroke
+			(width 0)
+			(type solid)
+		)
+		(fill
+			(type color)
+			(color 72 0 0 1)
+		)
+	)
+	(rectangle
+		(start 361.95 233.68)
+		(end 364.49 255.27)
+		(stroke
+			(width 0)
+			(type solid)
+		)
+		(fill
+			(type color)
+			(color 72 0 0 1)
+		)
+	)
 	(text "Compatible with TTL-234X-3V3 smart cable"
 		(exclude_from_sim no)

Commit message: Second review round
Parts:
- removed MCU_IO1: HC-PM254-8_5H-2X12PS, JLCImport:HC-PM254-8_5H-2X12PS, symbol JLCImport:HC-PM254-8_5H-2X12PS
- removed R64, R73, R74: 10, Resistor_SMD:R_0603_1608Metric, symbol Device:R_US
- added IMU_IO1: HX_PM2_54-2X8P_WT, JLCImport:HX_PM2_54-2X8P_WT, symbol JLCImport:HX_PM2_54-2X8P_WT
Connections:
- net PE0 is gone; now on net WHEEL-M-LEFT-IN1: U13.97 (PE0)
- net PE1 is gone; now on net WHEEL-M-LEFT-IN2: U13.98 (PE1)
- net PE13 is gone; now on net WHEEL-M-LEFT-ENCODE-A: U13.44 (PE13)
- net PE14 is gone; now on net WHEEL-M-RIGHT-ENCODE-A: U13.45 (PE14)
- net PE7 is gone; now on net PWR-BTN-SENSE: U13.38 (PE7)
- net ~{JTAG_RST} is gone; now on net ~{STM32_RST}: JTAG1.12
- net GND: now also IMU_IO1.14, IMU_IO1.16
- net PC10: now also IMU_IO1.11
- net PC13: now also IMU_IO1.12
- net PD5: now also IMU_IO1.10
- net PE15: now also IMU_IO1.8
- net PE8: now also IMU_IO1.7; no longer U13.39 (PE8)
- net PF2: now also IMU_IO1.13, IMU_IO1.9
- net PMIC_PWRON: now also U13.39 (PE8); no longer U13.73 (PA12)
- net PWR-BTN-SENSE: no longer U13.72 (PA11)
- net VCC-3V3-P: now also IMU_IO1.15
- net WHEEL-M-LEFT-ENCODE-A: no longer U13.70 (PA9)
- net WHEEL-M-LEFT-IN1: no longer U13.69 (PA8)
- net WHEEL-M-LEFT-IN2: no longer U13.29 (PA7)
- net WHEEL-M-RIGHT-ENCODE-A: no longer U13.71 (PA10)
- net PB3: now reaches U13.90 (PB3)
- net PB3: now also IMU_IO1.3
- net PB4: now reaches U13.91 (PB4)
- net PB4: now also IMU_IO1.4
- net PB5: now reaches U13.92 (PB5)
- net PB5: now also IMU_IO1.5
- net 3.3V_JTG: now reaches D5.2 (A), JTAG1.03 (3)
- net IMU-SPI-CS renamed PB6
- net PB6: now also IMU_IO1.6
- net PE10 renamed CARPET-SENSOR-HI
- net PE11 renamed CARPET-SENSOR-LO
- net PE12 renamed CARPET-SENSOR-ECHO
- new net DM: U13.72 (PA11)
- new net DP: U13.73 (PA12)
- new net I2C2_SCL: U13.70 (PA9)
- new net I2C2_SDA: U13.69 (PA8)
- new net PA10: IMU_IO1.2, U13.71 (PA10)
- new net PA7: IMU_IO1.1, U13.29 (PA7)
- no-connect marks 12 -> 8

Commit message: Cliff/bumper connector reverse engineered
Parts:
- removed C14: 100nF/50V, Capacitor_SMD:C_0603_1608Metric, symbol Device:C_Small
- removed IMU_IO1: HX_PM2_54-2X8P_WT, JLCImport:HX_PM2_54-2X8P_WT, symbol JLCImport:HX_PM2_54-2X8P_WT
- added MCU_IO1: HX_PM2_54-2X6P_WT, JLCImport:HX_PM2_54-2X6P_WT, symbol JLCImport:HX_PM2_54-2X6P_WT
Connections:
- net PA7 is gone; now on net WATER-PUMP-SENSE-ADC: U13.29 (PA7)
- net GND: now also MCU_IO1.11
- net LED-PWR: now also U13.19 (PF2); no longer U13.28 (PA6)
- net MAIN-BRUSH-CURRENT-ADC: now also U13.28 (PA6); no longer U13.26 (PA4)
- net PA10: now also MCU_IO1.2
- net PB3: now also MCU_IO1.1
- net PB4: now also MCU_IO1.4
- net PB5: now also MCU_IO1.3
- net PB6: now also MCU_IO1.6
- net PC10: now also MCU_IO1.7
- net PC13: now also MCU_IO1.12
- net PD5: now also MCU_IO1.10
- net PE15: now also MCU_IO1.8
- net PE8: now also MCU_IO1.5
- net PF2: now also MCU_IO1.9; no longer U13.19 (PF2)
- net WATER-PUMP-SENSE-ADC: no longer U13.27 (PA5)
- net ANTI-FALL-LEFT-DOWN-ADC renamed RF-Q+
- net ANTI-FALL-LEFT-UP-ADC renamed RR-Q+
- net ANTI-FALL-RIGHT-DOWN-ADC renamed LF-Q+
- net ANTI-FALL-RIGHT-UP-ADC renamed LR-Q+
- new net BUMP-L-Q+: U13.26 (PA4)
- new net BUMP-R-Q+: U13.27 (PA5)
