File: kicad/main/WATER-PUMP .kicad_sch (KiCad schematic)
At the start: 10 parts, among them Q7 2302V, Q8 AO3401

Commit message: Second review round
Changed lines of the file:
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@@
 	(generator_version "10.0")
 	(paper "A2")
-	(rectangle
-		(start 149.86 173.99)
-		(end 279.4 198.12)
-		(stroke
-			(width 0)
-			(type solid)
-		)
-		(fill
-			(type color)
-			(color 72 0 0 1)
-		)
-	)
-	(rectangle
-		(start 170.18 123.19)
-		(end 386.08 261.62)
-		(stroke
-			(width 0)
-			(type solid)
-		)
-		(fill
-			(type color)
-			(color 0 72 0 1)
-		)
-	)
-	(rectangle
-		(start 308.61 114.3)
-		(end 312.42 180.34)
-		(stroke
-			(width 0)
-			(type solid)
-		)
-		(fill
-			(type color)
-			(color 72 0 0 1)
-		)
-	)
 	(text "5V MOTOR"
 		(exclude_from_sim no)

Commit message: Cliff/bumper connector reverse engineered
Parts:
- removed Q7: 2302V, JLCImport:2302V, symbol JLCImport:2302V
- removed R43: 100k, Resistor_SMD:R_0603_1608Metric, symbol Device:R_US
Connections:
- net WATER-PUMPU-CTRL: now also Q8.1 (G), R25.1
