File: kicad/main/WATER-PUMP .kicad_sch (KiCad schematic)
At the start: 8 parts, among them Q8 AO3401

Commit message: STM32 power rail switch
Parts:
- added Q10: AO3401, oomwoo_altium:SOT23-3D, symbol DesignLibrary:WATER-PUMP_1_mirrored_P-MOS-SOT23_DesignLibrary.SchLib
- added R76: 10k, Resistor_SMD:R_0603_1608Metric, symbol DesignLibrary:WATER-PUMP_2_Resistor-1_DesignLibrary.SchLib
- added R79, R88: 10, Resistor_SMD:R_0603_1608Metric, symbol Device:R_US
- C105: LCSC (none) -> C107075; VOLTAGERATE 10V -> (none)
- C133: value 10uF/25V -> 10uF/10V; LCSC C96446 -> C19702
- R25, R81: LCSC (none) -> C98220; VOLTAGERATE * -> (none)
- R47: LCSC (none) -> C2907011
Connections:
- net VM-5V: now also Q10.2 (S), R76.2
- net WATER-PUMPU-CTRL: now also R76.1, R79.1, R88.1; no longer Q8.1 (G)
- net at C105.2, C133.1, D6.2 (K)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: now also Q10.3 (D)
- new net: Q8.1 (G), R88.2
- new net: Q10.1 (G), R79.2
Other:
- moved on the sheet: R25
