File: kicad/main/BUTTON-LEDs .kicad_sch (KiCad schematic)
At the start: 9 parts, among them SW1 TC-6601-5_0-260-8_3, SW2 TC-6601-5_0-260-8_3, SW3 TC-6601-5_0-260-8_3

Commit message: Cliff/bumpers connector
Changed lines of the file:
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@@
 	(generator_version "10.0")
 	(paper "A2")
+	(rectangle
+		(start 212.09 132.08)
+		(end 394.97 257.81)
+		(stroke
+			(width 0)
+			(type solid)
+		)
+		(fill
+			(type color)
+			(color 0 72 0 1)
+		)
+	)
 	(text "LEDs AND BUTTONs"
 		(exclude_from_sim no)

Commit message: Second review round
Parts:
- removed SW1, SW2, SW3: TC-6601-5_0-260-8_3, JLCImport:TC-6601-5_0-260-8_3, symbol JLCImport:TC-6601-5_0-260-8_3
- added SW_CLEAN1, SW_HOME1, SW_PWR1: TS-1187A-B-A-B, JLCImport:TS-1187A-B-A-B, symbol JLCImport:TS-1187A-B-A-B
Connections:
- net CLEAN-BTN: now also SW_CLEAN1.3 (C), SW_CLEAN1.4 (D)
- net GND: now also SW_CLEAN1.1 (A), SW_CLEAN1.2 (B), SW_HOME1.1 (A), SW_HOME1.2 (B), SW_PWR1.1 (A), SW_PWR1.2 (B)
- net HOME-BTN: now also SW_HOME1.3 (C), SW_HOME1.4 (D)
- net POWER-BTN: now also SW_PWR1.3 (C), SW_PWR1.4 (D)

Commit message: STM32 power rail switch
Parts:
- R120, R121: LCSC (none) -> C2907113; VOLTAGERATE * -> (none)
- R77, R78: LCSC (none) -> C2907113
Connections:
- net VCC-3V3-P renamed VCC-3V3-REG
