File: kicad/main/Front Sensors.kicad_sch (KiCad schematic)
At the start: 18 parts, among them Q2 2302V

Commit message: STM32 power rail switch
Parts:
- C19, C6, C90, C91: value 10uF/25V -> 10uF/6.3V; LCSC C96446 -> C1691
- R2, R61, R62, R7: LCSC (none) -> C2907042
- R5, R6: LCSC (none) -> C2907005
- R54: LCSC (none) -> C2907088
Connections:
- net VCC-3V3-P is gone; now on net VCC-3V3-REG: C19.1, C90.1, C91.1, IR-F1.1, IR-F2.1, LIGHT1.1, R5.1, R6.1, R61.1, R62.1, R7.1, VL-R1.1
- net VCC-3V3-REG: now reaches C6.1, VL-L1.1
Other:
- moved on the sheet: C90, C91, IR-F1, IR-F2
