File: kicad/main/MAIN-BRUSH-MOTOR .kicad_sch (KiCad schematic)
At the start: 7 parts, among them U20 DRV8870DDAR

Commit message: Cliff/bumpers connector
Changed lines of the file:
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@@
 	(generator_version "10.0")
 	(paper "A2")
+	(rectangle
+		(start 156.21 123.19)
+		(end 335.28 207.01)
+		(stroke
+			(width 0)
+			(type solid)
+		)
+		(fill
+			(type color)
+			(color 0 72 0 1)
+		)
+	)
+	(rectangle
+		(start 252.73 171.45)
+		(end 261.62 240.03)
+		(stroke
+			(width 0)
+			(type solid)
+		)
+		(fill
+			(type color)
+			(color 72 0 0 1)
+		)
+	)
 	(text "MAIN BUSH MOTOR CONTROL"
 		(exclude_from_sim no)

Commit message: Second review round
Parts:
- removed R112: 0.2R/10W, Resistor_SMD:R_2512_6332Metric, symbol DesignLibrary:WHEEL MOTOR_1_Resistor-1_DesignLibrary.SchLib
- added R84: RLH12FTCR110, JLCImport:RLH12FTCR110, symbol JLCImport:RLH12FTCR110
Connections:
- net GND: now also R84.1
- net MAIN-BRUSH-CURRENT-ADC: now also R84.2

Commit message: STM32 power rail switch
Parts:
- C103: value 100nF/50V -> 100nF/25V; LCSC C1591 -> C1590; VOLTAGERATE 50V -> (none)
- R3, R4: LCSC (none) -> C2907088
Connections:
- net VCC-3V3-P renamed VCC-3V3-REG
