File: kicad/main/SIDE-BRUSH-MOTORs .kicad_sch (KiCad schematic)
At the start: 9 parts, among them U18 DRV8870DDAR

Commit message: Cliff/bumpers connector
Changed lines of the file:
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@@
 	(generator_version "10.0")
 	(paper "A2")
+	(rectangle
+		(start 140.97 106.68)
+		(end 347.98 213.36)
+		(stroke
+			(width 0)
+			(type solid)
+		)
+		(fill
+			(type color)
+			(color 0 72 0 1)
+		)
+	)
+	(rectangle
+		(start 199.39 176.53)
+		(end 227.33 222.25)
+		(stroke
+			(width 0)
+			(type solid)
+		)
+		(fill
+			(type color)
+			(color 72 0 0 1)
+		)
+	)
+	(rectangle
+		(start 256.54 158.75)
+		(end 265.43 228.6)
+		(stroke
+			(width 0)
+			(type solid)
+		)
+		(fill
+			(type color)
+			(color 72 0 0 1)
+		)
+	)
 	(text "SIDE-BRUSH MOTOR CONTROL"
 		(exclude_from_sim no)

Commit message: Second review round
Parts:
- removed D22: 1N4007, oomwoo_altium:SOD123, symbol DesignLibrary:WHEEL MOTOR_3_DIODE-1_DesignLibrary.SchLib
- removed R110: 10k, Resistor_SMD:R_0603_1608Metric, symbol DesignLibrary:WHEEL MOTOR_0_Resistor-1_DesignLibrary.SchLib
- removed R88: 0.2R/10W, Resistor_SMD:R_2512_6332Metric, symbol DesignLibrary:WHEEL MOTOR_1_Resistor-1_DesignLibrary.SchLib
- added R83: RL12FTNR300, JLCImport:RL12FTNR300, symbol JLCImport:RL12FTNR300
Connections:
- net GND: now also R83.1
- net SIDE-BRUSH-CURRENT-ADC: now also U18.7 (ISEN), R83.2

Commit message: STM32 power rail switch
Parts:
- C92: value 100nF/50V -> 100nF/25V; LCSC C1591 -> C1590; VOLTAGERATE 50V -> (none)
- R55, R57: LCSC (none) -> C2907088
Connections:
- net VCC-3V3-P renamed VCC-3V3-REG
