File: kicad/main/SPEAKER-MIC.kicad_sch (KiCad schematic)
At the start: 15 parts, among them Q9 2302V, U10 ICS-43434_C5656610, U11 MAX98357AETE_T, U9 ICS-43434_C5656610

Commit message: STM32 power rail switch
Parts:
- C10: value 100nF/50V -> 100nF/10V; LCSC C1591 -> C36911391
- C11: value 10uF/25V -> 10uF/10V; LCSC C96446 -> C19702
- C5, C9: value 100nF/50V -> 100nF/6.3V; LCSC C1591 -> C5356672
- R12, R9: LCSC (none) -> C2906974
- R13, R8: LCSC (none) -> C2907088
Connections:
- net +3.3VP renamed 3.3V-PI
- net VCC-3V3-P renamed VCC-3V3-REG
