File: kicad/main/WHEEL-MOTORs .kicad_sch (KiCad schematic)
At the start: 20 parts, among them U14 DRV8870DDAR, U15 DRV8870DDAR

Commit message: Cliff/bumpers connector
Changed lines of the file:
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@@
 	(generator_version "10.0")
 	(paper "A2")
+	(rectangle
+		(start 270.51 236.22)
+		(end 278.13 248.92)
+		(stroke
+			(width 0)
+			(type solid)
+		)
+		(fill
+			(type color)
+			(color 72 0 0 1)
+		)
+	)
+	(rectangle
+		(start 151.13 106.68)
+		(end 415.29 278.13)
+		(stroke
+			(width 0)
+			(type solid)
+		)
+		(fill
+			(type color)
+			(color 0 72 0 1)
+		)
+	)
+	(rectangle
+		(start 267.97 151.13)
+		(end 275.59 161.29)
+		(stroke
+			(width 0)
+			(type solid)
+		)
+		(fill
+			(type color)
+			(color 72 0 0 1)
+		)
+	)
 	(text "WHEEL MOTOR CONTROL"
 		(exclude_from_sim no)

Commit message: Second review round
Parts:
- removed R83, R84: 0.2R/10W, Resistor_SMD:R_2512_6332Metric, symbol DesignLibrary:WHEEL MOTOR_1_Resistor-1_DesignLibrary.SchLib
- added R15, R65: RL12FTNR250, JLCImport:RL12FTNR250, symbol JLCImport:RL12FTNR250
Connections:
- net GND: now also R15.1, R65.1
- net WHEEL-M-L-F-ADC: now also R65.2
- net WHEEL-M-R-F-ADC: now also R15.2

Commit message: STM32 power rail switch
Parts:
- C142, C143: value 100nF/50V -> 100nF/6.3V; LCSC C1591 -> C5356672; Manufacturer_Part_Number CL10B104KB8NNNC -> (none)
- C84, C88: value 100nF/50V -> 100nF/25V; LCSC C1591 -> C1590; VOLTAGERATE 50V -> (none)
- R11, R17, R20, R27: LCSC (none) -> C2907088
- R49, R50, R51, R52: LCSC (none) -> C98220
Connections:
- net VCC-3V3-P renamed VCC-3V3-REG
