File: kicad/main/CM5-Highspeed.kicad_sch (KiCad schematic)
At the start: 5 parts

Commit message: Cliff/bumpers connector
Changed lines of the file:
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@@
 	(generator_version "10.0")
 	(paper "A2")
+	(rectangle
+		(start 341.63 76.2)
+		(end 403.86 224.79)
+		(stroke
+			(width 0)
+			(type solid)
+		)
+		(fill
+			(type color)
+			(color 0 72 0 1)
+		)
+	)
+	(rectangle
+		(start 359.41 92.71)
+		(end 367.03 95.25)
+		(stroke
+			(width 0)
+			(type solid)
+		)
+		(fill
+			(type color)
+			(color 132 0 0 1)
+		)
+	)
+	(rectangle
+		(start 233.68 76.2)
+		(end 321.31 224.79)
+		(stroke
+			(width 0)
+			(type solid)
+		)
+		(fill
+			(type color)
+			(color 0 72 0 1)
+		)
+	)
+	(rectangle
+		(start 358.14 151.13)
+		(end 361.95 171.45)
+		(stroke
+			(width 0)
+			(type solid)
+		)
+		(fill
+			(type color)
+			(color 132 0 0 1)
+		)
+	)
+	(rectangle
+		(start 358.14 80.01)
+		(end 365.76 82.55)
+		(stroke
+			(width 0)
+			(type solid)
+		)
+		(fill
+			(type color)
+			(color 132 0 0 1)
+		)
+	)
+	(rectangle
+		(start 373.38 81.28)
+		(end 389.89 88.9)
+		(stroke
+			(width 0)
+			(type solid)
+		)
+		(fill
+			(type color)
+			(color 132 0 0 1)
+		)
+	)
 	(junction
 		(at 291.465 96.52)

Commit message: Second review round
Parts:
- removed R101, R96: 10, Resistor_SMD:R_0603_1608Metric, symbol Device:R_US
- added D35: TPD2EUSB30DRTR, TPD2EUSB30DRTR:SOTFL35P100X50-3N, symbol TPD2EUSB30DRTR:TPD2EUSB30DRTR
- added USB_BOOT1: USB4215-03-A_REVA, USB4215-03-A_REVA:GCT_USB4215-03-A_REVA, symbol USB4215-03-A_REVA:USB4215-03-A_REVA
Connections:
- net GND: now also D35.3 (GND), USB_BOOT1.A1_B12 (GND_A), USB_BOOT1.B1_A12 (GND_B), USB_BOOT1.SH1 (SHIELD), USB_BOOT1.SH2 (SHIELD__1), USB_BOOT1.SH3 (SHIELD__2), USB_BOOT1.SH4 (SHIELD__3)
- net D-: now reaches Module1.103 (USB2_N)
- net D-: now also D35.2 (D-), USB_BOOT1.A7 (DN1), USB_BOOT1.B7 (DN2)
- net D+: now reaches Module1.105 (USB2_P)
- net D+: now also D35.1 (D+), USB_BOOT1.A6 (DP1), USB_BOOT1.B6 (DP2)
- new net: USB_BOOT1.A4_B9 (VBUS_A), USB_BOOT1.B4_A9 (VBUS_B)
- new net CC1: USB_BOOT1.A5 (CC1)
- new net CC2: USB_BOOT1.B5 (CC2)
- no-connect marks 40 -> 42
Other:
- moved on the sheet: JP1, JP2, Module1B

Commit message: Update Power Control sch, Charger sch, Speaker + Mic, JTAG and Watch Dog
**Power Control:** Replaced the BJT with a MOSFET. The MCU hang condition is not covered yet.
Parts:
- removed D35: TPD2EUSB30DRTR, TPD2EUSB30DRTR:SOTFL35P100X50-3N, symbol TPD2EUSB30DRTR:TPD2EUSB30DRTR
- removed USB_BOOT1: USB4215-03-A_REVA, USB4215-03-A_REVA:GCT_USB4215-03-A_REVA, symbol USB4215-03-A_REVA:USB4215-03-A_REVA
- added D3: USBLC6-2SC6_C2687116, JLCImport:USBLC6-2SC6_C2687116, symbol JLCImport:USBLC6-2SC6_C2687116
- added F2: SMD0603-050, JLCImport:SMD0603-050, symbol JLCImport:SMD0603-050
- added USB1: HC-GH-4PWT, JLCImport:HC-GH-4PWT, symbol JLCImport:HC-GH-4PWT
Connections:
- net GND: now also D3.2 (GND), USB1.4, USB1.5, USB1.6
- net D+: no longer names the net of Module1.105 (USB2_P)
- net D+: now also D3.3 (I/O2), D3.4 (I/O2), USB1.3
- net D-: no longer names the net of Module1.103 (USB2_N)
- net D-: now also D3.1 (I/O1), D3.6 (I/O1), USB1.2
- new net: F2.1, USB1.1
- new net VCC-5V-REG: D3.5 (VBUS), F2.2
- no-connect marks 42 -> 40
