File: kicad/main/SPEAKER.kicad_sch (KiCad schematic)
At the start: 11 parts, among them Q9 2302V, U8 NS4168_C910588

Commit message: Change N-MOSFET part
Parts:
- Q9: value 2302V -> AO3400; footprint JLCImport:2302V -> JLCImport:AO3400; symbol JLCImport:2302V -> JLCImport:AO3400; LCSC C7431443 -> C20628874; Manufacturer HL -> FOSAN; Manufacturer Part 2302V -> AO3400
Changed lines of the file:
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@@
 	)
 	(symbol
-		(lib_id "JLCImport:2302V")
+		(lib_id "JLCImport:AO3400")
 		(at 122.555 241.3 0)
 		(unit 1)
@@
 			)
 		)
-		(property "Value" "2302V"
+		(property "Value" "AO3400"
 			(at 117.475 236.22 0)
 			(show_name no)
@@
 			)
 		)
-		(property "Footprint" "JLCImport:2302V"
+		(property "Footprint" "JLCImport:AO3400"
 			(at 122.555 241.3 0)
 			(hide yes)
@@
 			)
 		)
-		(property "Datasheet" "https://wmsc.lcsc.com/wmsc/upload/file/pdf/v2/lcsc/2306211455_HL-2302V_C7431443.pdf"
+		(property "Datasheet" "https://wmsc.lcsc.com/wmsc/upload/file/pdf/v2/lcsc/2403011756_FOSAN-AO3400_C20628874.pdf"
 			(at 122.555 241.3 0)
 			(hide yes)
@@
 			)
 		)
-		(property "Description" "-55℃~+150℃ 1 N-channel 184pF 20V 28pF 3A 400mV 43mΩ 850mW SOT-23 MOSFETs ROHS"
+		(property "Description" "30V 5.8A N-channel MOSFET, 25mOhm@4.5V, Vgs +/-12V, Vth 0.65-1.5V, SOT-23"
 			(at 122.555 241.3 0)
 			(hide yes)
@@
 			)
 		)
-		(property "LCSC" "C7431443"
+		(property "LCSC" "C20628874"
 			(at 122.555 241.3 0)
 			(hide yes)
@@
 			)
 		)
-		(property "Manufacturer" "HL"
+		(property "Manufacturer" "FOSAN"
 			(at 122.555 241.3 0)
 			(hide yes)
@@
 			)
 		)
-		(property "Manufacturer Part" "2302V"
+		(property "Manufacturer Part" "AO3400"
 			(at 122.555 241.3 0)
 			(hide yes)
