File: kicad/main/STM32G473.kicad_sch (KiCad schematic)
At the start: 32 parts, among them T1 NTCG164KF104FT1, U13 STM32G473VCT6, X1 ABM3-8_000MHZ-D2Y-T, X3 XKXEL89CII-SUAYLC-32_768K

Commit message: STM32 power rail switch
Parts:
- removed MCU_IO1: HX_PM2_54-2X6P_WT, JLCImport:HX_PM2_54-2X6P_WT, symbol JLCImport:HX_PM2_54-2X6P_WT
- added D9: SS34_C8678, JLCImport:SS34_C8678, symbol JLCImport:SS34_C8678
- added FAN1: S2B-ZR-SM4A-TF_LF_SN, JLCImport:S2B-ZR-SM4A-TF_LF_SN, symbol JLCImport:S2B-ZR-SM4A-TF_LF_SN
- added MCU_IO1: HX_PM2_54-2X4P_WT, JLCImport:HX_PM2_54-2X4P_WT, symbol JLCImport:HX_PM2_54-2X4P_WT
- added Q3: 2302V, JLCImport:2302V, symbol JLCImport:2302V
- added R87: 1k, Resistor_SMD:R_0603_1608Metric, symbol Device:R_US
- C12, C13, C15, C16, C30, C32, C36, C37: value 100nF/50V -> 100nF/6.3V; LCSC C1591 -> C5356672
- C17, C31, C33: value 10uF/25V -> 10uF/6.3V; LCSC C96446 -> C1691
- C34, C35: LCSC (none) -> C1653
- C39, C42: value 18pF/10V -> 18pF/50V; LCSC (none) -> C107040
- R113: LCSC (none) -> C2907113
- R117, R80, R94, R95: LCSC (none) -> C2907091
- R19: LCSC (none) -> C2906974
- R21, R22: LCSC (none) -> C98220
- R38: LCSC (none) -> C2907088
Connections:
- net GND: now also FAN1.0, MCU_IO1.2, Q3.2 (S)
- net PB5: now also MCU_IO1.3; no longer U13.92 (PB5)
- net PB6: now also MCU_IO1.4
- net PC13: now also MCU_IO1.8
- net PE15: now also MCU_IO1.6
- net PE8: now also MCU_IO1.5
- net PF2: now also MCU_IO1.7
- net PA10 renamed BOARD_FAN
- net BOARD_FAN: now also R87.1
- net PB3 renamed 3.3V_EN
- net PB4 renamed 5V_EN
- net PC10 renamed USB_PWR_EN
- net VCC-3V3-P renamed VCC-3V3
- new net: Q3.1 (G), R87.2
- new net: D9.2 (A), FAN1.2, Q3.3 (D)
- new net PI_DONE: U13.92 (PB5)
- new net VCC-3V3-REG: MCU_IO1.1
- new net VCC-5V-REG: D9.1 (K), FAN1.1
Other:
- moved on the sheet: C12, C13, C15, C16, C17, C30, C31, C32, C33, C34, C35, C36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

Commit message: LDR
Parts:
- removed MCU_IO1: HX_PM2_54-2X4P_WT, JLCImport:HX_PM2_54-2X4P_WT, symbol JLCImport:HX_PM2_54-2X4P_WT
- added R103: 10k, Resistor_SMD:R_0603_1608Metric, symbol Device:R_US
- added R75: GL5537-1, JLCImport:GL5537-1, symbol JLCImport:GL5537-1
Connections:
- net PC13 is gone; now on net LED-HOME: U13.7 (PC13)
- net GND: now also R103.1
- net LED-HOME: no longer U13.51 (PB12)
- net VCC-3V3-REG: now also R75.2
- net PB6 renamed PI_SHUTDOWN
- net PE6: no longer names the net of U13.5 (PE6)
- new net: R103.2, R75.1, U13.51 (PB12)
- no-connect marks 8 -> 9

Commit message: Update Power Control sch, Charger sch, Speaker + Mic, JTAG and Watch Dog
**Power Control:** Replaced the BJT with a MOSFET. The MCU hang condition is not covered yet.
Parts:
- removed D5: SS34, Diode_SMD:D_SMA, symbol Diode:SS34
- removed D9: SS34_C8678, JLCImport:SS34_C8678, symbol JLCImport:SS34_C8678
- removed JTAG1: STLINK-V3MINIE, JLCImport:FTSH-107-01-L-DV-K-A, symbol JLCImport:FTSH-107-01-L-DV-K-A
- added D17: SS56, JLCImport:SS56, symbol JLCImport:SS56
- added JTAG1: 5AIW2-3520-207-W5, JLCImport:5AIW2-3520-207-W5, symbol JLCImport:5AIW2-3520-207-W5
- added Q25: 2302V, JLCImport:2302V, symbol JLCImport:2302V
- added R40, R45, R69: 100k, Resistor_SMD:R_0603_1608Metric, symbol Device:R_US
Connections:
- net PB10 is gone; now on net 3.3V_EN: U13.47 (PB10)
- net 3.3V_EN: no longer U13.90 (PB3)
- net GND: now also JTAG1.5, JTAG1.7, Q25.2 (S)
- net STM32-RX: now also JTAG1.13
- net STM32-TX: now also JTAG1.14
- net VCC-3V3: now also R40.1, R45.1, R69.1
- net VCC-5V-REG: now also D17.1 (K)
- net ~{STM32_RST}: now also JTAG1.12
- net BOOT: now reaches R22.2, U13.95 (PB8-BOOT0)
- net at FAN1.2, Q3.3 (D): now also D17.2 (A)
- net I2C3_SCL: no longer names the net of U13.67 (PC8)
- net I2C3_SDA: no longer names the net of U13.68 (PC9)
- net STM32-SWCLK renamed SWCLK
- net SWCLK: now also JTAG1.6
- net STM32-SWDIO renamed SWDIO
- net SWDIO: now also JTAG1.4
- net ~{CHG_INT}: no longer names the net of U13.54 (PB15)
- new net: JTAG1.11, Q25.1 (G), R45.2
- new net: JTAG1.3, R40.2
- new net JTAG_PRESENCE: Q25.3 (D), R69.2
- new net STM32-SWO: JTAG1.8, U13.90 (PB3)
- no-connect marks 9 -> 10

Commit message: Reassigned CARPET-SENSOR-HI to VM-VBAT-EN
Parts:
- Q25, Q3: value 2302V -> AO3400; footprint JLCImport:2302V -> JLCImport:AO3400; symbol JLCImport:2302V -> JLCImport:AO3400; LCSC C7431443 -> C20628874; Manufacturer HL -> FOSAN; Manufacturer Part 2302V -> AO3400
Connections:
- net CARPET-SENSOR-HI renamed ~{VM-VBAT-EN}
Changed lines of the file:
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@@
 	(generator_version "10.0")
 	(paper "A2")
+	(rectangle
+		(start 336.55 116.205)
+		(end 377.825 118.745)
+		(stroke
+			(width 0)
+			(type solid)
+		)
+		(fill
+			(type color)
+			(color 0 72 0 1)
+		)
+	)
 	(text "Compatible with TTL-234X-3V3 smart cable"
 		(exclude_from_sim no)
@@
 		)
 	)
-	(hierarchical_label "CARPET-SENSOR-HI"
+	(hierarchical_label "~{VM-VBAT-EN}"
 		(shape output)
 		(at 365.76 118.11 180)
@@
 	)
 	(symbol
-		(lib_id "JLCImport:2302V")
+		(lib_id "JLCImport:AO3400")
 		(at 300.99 311.785 0)
 		(unit 1)
@@
 			)
 		)
-		(property "Value" "2302V"
+		(property "Value" "AO3400"
 			(at 308.61 311.785 0)
 			(show_name no)
@@
 			)
 		)
-		(property "Footprint" "JLCImport:2302V"
+		(property "Footprint" "JLCImport:AO3400"
 			(at 300.99 311.785 0)
 			(hide yes)
@@
 			)
 		)
-		(property "Datasheet" "https://wmsc.lcsc.com/wmsc/upload/file/pdf/v2/lcsc/2306211455_HL-2302V_C7431443.pdf"
+		(property "Datasheet" "https://wmsc.lcsc.com/wmsc/upload/file/pdf/v2/lcsc/2403011756_FOSAN-AO3400_C20628874.pdf"
 			(at 300.99 311.785 0)
 			(hide yes)
@@
 			)
 		)
-		(property "Description" "-55℃~+150℃ 1 N-channel 184pF 20V 28pF 3A 400mV 43mΩ 850mW SOT-23 MOSFETs ROHS"
+		(property "Description" "30V 5.8A N-channel MOSFET, 25mOhm@4.5V, Vgs +/-12V, Vth 0.65-1.5V, SOT-23"
 			(at 300.99 311.785 0)
 			(hide yes)
@@
 			)
 		)
-		(property "LCSC" "C7431443"
+		(property "LCSC" "C20628874"
 			(at 300.99 311.785 0)
 			(hide yes)
@@
 			)
 		)
-		(property "Manufacturer" "HL"
+		(property "Manufacturer" "FOSAN"
 			(at 300.99 311.785 0)
 			(hide yes)
@@
 			)
 		)
-		(property "Manufacturer Part" "2302V"
+		(property "Manufacturer Part" "AO3400"
 			(at 300.99 311.785 0)
 			(hide yes)
@@
 	)
 	(symbol
-		(lib_id "JLCImport:2302V")
+		(lib_id "JLCImport:AO3400")
 		(at 412.115 287.02 0)
 		(unit 1)
@@
 			)
 		)
-		(property "Value" "2302V"
+		(property "Value" "AO3400"
 			(at 420.37 287.02 90)
 			(show_name no)
@@
 			)
 		)
-		(property "Footprint" "JLCImport:2302V"
+		(property "Footprint" "JLCImport:AO3400"
 			(at 412.115 287.02 0)
 			(hide yes)
@@
 			)
 		)
-		(property "Datasheet" "https://wmsc.lcsc.com/wmsc/upload/file/pdf/v2/lcsc/2306211455_HL-2302V_C7431443.pdf"
+		(property "Datasheet" "https://wmsc.lcsc.com/wmsc/upload/file/pdf/v2/lcsc/2403011756_FOSAN-AO3400_C20628874.pdf"
 			(at 412.115 287.02 0)
 			(hide yes)
@@
 			)
 		)
-		(property "Description" "-55℃~+150℃ 1 N-channel 184pF 20V 28pF 3A 400mV 43mΩ 850mW SOT-23 MOSFETs ROHS"
+		(property "Description" "30V 5.8A N-channel MOSFET, 25mOhm@4.5V, Vgs +/-12V, Vth 0.65-1.5V, SOT-23"
 			(at 412.115 287.02 0)
 			(hide yes)
@@
 			)
 		)
-		(property "LCSC" "C7431443"
+		(property "LCSC" "C20628874"
 			(at 412.115 287.02 0)
 			(hide yes)
@@
 			)
 		)
-		(property "Manufacturer" "HL"
+		(property "Manufacturer" "FOSAN"
 			(at 412.115 287.02 0)
 			(hide yes)
@@
 			)
 		)
-		(property "Manufacturer Part" "2302V"
+		(property "Manufacturer Part" "AO3400"
 			(at 412.115 287.02 0)
 			(hide yes)

Commit message: Cleanup; renamed WDO to WDI
Parts:
- removed Q25: AO3400, JLCImport:AO3400, symbol JLCImport:AO3400
- removed R45, R69: 100k, Resistor_SMD:R_0603_1608Metric, symbol Device:R_US
Connections:
- net WDO renamed WDI
- no-connect marks 10 -> 11
Other:
- note added: "Compatible with STDC14 Pin 11 (GNDDetect) can detect JTAG cable presence using a 100k pull-up plus a spare GPIO The watchdog shuts off motors when not petted JTAG, SWD, BOOT0 do NOT disable the watchdog So, using JTAG/SWD/flash-over-UART stops motors"
