File: kicad/main/STM32G473.kicad_sch (KiCad schematic)
At the start: 37 parts, among them Q3 AO3400, T1 NTCG164KF104FT1, U13 STM32G473VCT6, X1 ABM3-8_000MHZ-D2Y-T, X3 XKXEL89CII-SUAYLC-32_768K

Commit message: Add main-phone: v1 board with a smartphone as the compute
kicad/main-phone is a fork of the Pi carrier for the first board: an
Android phone talks to the STM32 over USB-C, no Pi, cameras, M.2, SD,
speaker or mopping. The Pi board (kicad/main) stays in the plans.

v1 board:
- USB-C CC1/CC2 to the STM32 UCPD; reverse-block FETs for the TMI6240
- front ToF on I2C4; LiDAR UART TX/RX unswapped
- power control: charger rail-hold, ~4-9 s hardware off timer
- 20 V input: SMAJ22A TVS, 50 V DC_IN caps, DC_IN sense to PB15
- low-profile DC-044A-20A barrel jack (footprint + 3D model added)
- on-board ITR9606 bumpers in parallel with the harness bumpers
- carpet drive AC-coupled; right-angle 1x5 for LiDAR and debug headers
- spare I/O pads (2x6), pull-up/series fixes, BOM consolidation

Also: README and SPEC updated (v1 sections, STM32G473), LiDAR UART
net names on the Pi board.

Co-Authored-By: Claude Opus 5.5 (1M context) <noreply@anthropic.com>
Connections:
- net UART5_RX renamed LIDAR_TX
- net UART5_TX renamed LIDAR_RX
Changed lines of the file:
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@@
 		)
 	)
-	(hierarchical_label "UART5_RX"
+	(hierarchical_label "LIDAR_TX"
 		(shape input)
 		(at 297.18 144.78 0)
@@
 		)
 	)
-	(hierarchical_label "UART5_TX"
+	(hierarchical_label "LIDAR_RX"
 		(shape output)
 		(at 297.18 127 0)
