File: kicad/main/Battery-Charger.kicad_sch (KiCad schematic)
At the start: 68 parts, among them CN2 EV2400, IC5 TPS25730DREFR, Q21 SQJ844AEP-T1_GE3, Q4 SQJ844AEP-T1_GE3, U7 BQ25792RQMR

Commit message: Add master fuse
Parts:
- added F1: JFC1206-2200FS, JLCImport:JFC1206-2200FS, symbol JLCImport:JFC1206-2200FS
- R100, R75, R76: footprint Resistor_SMD:R_0805_2012Metric -> Resistor_SMD:R_0603_1608Metric
Connections:
- net BAT-VCC: now also F1.2; no longer C100.2, C83.1, C96.2, C97.2, C98.2, C99.2, U7.25 (SYS)
- new net: C100.2, C83.1, C96.2, C97.2, C98.2, C99.2, F1.1, U7.25 (SYS)
Other:
- moved on the sheet: D3

Commit message: STM32 power rail switch
Parts:
- removed C125, C126: 1nF/50V, Capacitor_SMD:C_0603_1608Metric, symbol Device:C
- removed C47, C58: 330pF/25V, Capacitor_SMD:C_0603_1608Metric, symbol Device:C
- removed C59, C61, C64, C65, C73: 100nF/50V, Capacitor_SMD:C_0603_1608Metric, symbol Device:C
- removed C60, C66, C71, C72, C74, C76, C94: 10uF/25V, Capacitor_SMD:C_0603_1608Metric, symbol Device:C
- removed D1, D2: TVS2200DRVR, JLCImport:TVS2200DRVR, symbol JLCImport:TVS2200DRVR
- removed D39, D40: BZT52C12T-7, JLCImport:BZT52C12T-7, symbol JLCImport:BZT52C12T-7
- removed IC5: TPS25730DREFR, LIB_TPS25730DREFR:TPS25730DREFR, symbol SamacSys_Parts:TPS25730DREFR
- removed Q21, Q4: SQJ844AEP-T1_GE3, JLCImport:SQJ844AEP-T1_GE3, symbol JLCImport:SQJ844AEP-T1_GE3
- removed R128, R130, R133, R138, R139: 100k, Resistor_SMD:R_0603_1608Metric, symbol Device:R_US
- removed R131: 20k, Resistor_SMD:R_0603_1608Metric, symbol Device:R_US
- removed R136, R137: 5.24k, Resistor_SMD:R_0603_1608Metric, symbol Device:R_US
- removed R140: 1k, Resistor_SMD:R_0603_1608Metric, symbol Device:R_US
- removed R75, R76: 100, Resistor_SMD:R_0603_1608Metric, symbol Device:R_US
- added C125: 10uF/50V, Capacitor_SMD:C_0805_2012Metric, symbol Library:C_0603
- added C139, C154: 10uF/25V, Capacitor_SMD:C_0603_1608Metric, symbol JLCImport:CL21A106KBYQNNE
- added C155, C156, C157: 100nF/25V, Capacitor_SMD:C_0603_1608Metric, symbol Library:C_0603
- added C159, C160, C161: 10uF/6.3V, Capacitor_SMD:C_0603_1608Metric, symbol JLCImport:CL21A106KBYQNNE
- added C162, C85: 1.2nF/50V, Capacitor_SMD:C_0603_1608Metric, symbol Library:C_0603
- added C163: 100nF/10V, Capacitor_SMD:C_0603_1608Metric, symbol Library:C_0603
- added D1: SMBJ24A_C908801, JLCImport:SMBJ24A_C908801, symbol JLCImport:SMBJ24A_C908801
- added D10: SS34, Diode_SMD:D_SMA, symbol DesignLibrary:WATER-PUMP_1_DIODE-2_DesignLibrary.SchLib
- added DC1: DC-005-5A-2_0, JLCImport:DC-005-5A-2_0, symbol JLCImport:DC-005-5A-2_0
- added L5: CYA0630-3_3UH, JLCImport:CYA0630-3_3UH, symbol JLCImport:CYA0630-3_3UH
- added R101: 215k, Resistor_SMD:R_0603_1608Metric, symbol Device:R_US
- added R161: 10, Resistor_SMD:R_0603_1608Metric, symbol Device:R_US
- added R162: 20k, Resistor_SMD:R_0603_1608Metric, symbol Device:R_US
- added R163: 12k, Resistor_SMD:R_0603_1608Metric, symbol Device:R_US
- added R164: 2.2k, Resistor_SMD:R_0603_1608Metric, symbol Device:R_US
- added R41, R43: 100k, Resistor_SMD:R_0603_1608Metric, symbol Device:R_US
- added U2: TMI6240, JLCImport:TMI6240, symbol JLCImport:TMI6240
- added U25: AP64501SP-13, JLCImport:AP64501SP-13, symbol JLCImport:AP64501SP-13
- C67, C68, C69, C78, C80, C81, C82: value 10uF/25V -> 10uF/50V; footprint Capacitor_SMD:C_0603_1608Metric -> Capacitor_SMD:C_0805_2012Metric; LCSC C96446 -> C22367830
- C70: value 10uF/25V -> 4.7uF/10V; LCSC C96446 -> C2826877
- C75, C79: LCSC (none) -> C1622
- C77: LCSC (none) -> C14442
- R100: LCSC (none) -> C2906981
- R115: LCSC (none) -> C2907088
- R132: LCSC (none) -> C98220
- R37: LCSC (none) -> C2907113; VOLTAGERATE * -> (none)
Connections:
- net VCC-CHARG is gone; now on net VCC-CHARGE: C67.2, C68.2, C69.1, U7.2 (VBUS), U7.3 (VBUS)
- net VOUT_PD is gone; now on net VCC-CHARGE: U7.9 (VAC1)
- net BAT-VCC: now also C100.2, C83.1, C96.2, C97.2, C98.2, C99.2, U7.25 (SYS), C139.1, C154.1, C155.1, U25.2 (VIN); no longer F1.2
- net GND: now also U7.10 (ACDRV2), U7.11 (ACDRV1), C125.2, C139.2, C154.2, C155.2, C156.2, C159.2, C160.2, C161.2, C162.2, C163.2, C85.2, D1.2, D10.1 (A), DC1.2, R164.1, R41.2, R43.2, U2.2 (GND), U25.7 (GND), U25.9 (EP); no longer CONTACT_CHGR1.1, CONTACT_CHGR1.2
- net P+/C+: now also F1.1; no longer BAT2.1
- net VBUS: now also C163.1, D10.2 (K), U2.5 (VOUT)
- net VCC-CHARGE: now reaches CONTACT_CHGR1.3, CONTACT_CHGR1.4, U7.8 (VAC2)
- net VCC-CHARGE: now also C125.1, D1.1, DC1.1
- net CC1: no longer names the net of USB2.A5 (CC1)
- net CC2: no longer names the net of USB2.B5 (CC2)
- net VCC-3V3-P renamed VCC-3V3
- new net: R163.1, R164.2, U25.5 (FB)
- new net: C159.1, C160.1, C161.1, L5.2, R101.2, R163.2, U2.1 (VIN)
- new net: R101.1, R41.1, U2.3 (EN)
- new net: C85.1, R162.1
- new net: R162.2, U25.6 (COMP)
- new net: L5.1, R161.2, U25.8 (SW)
- new net: BAT2.1, F1.2
- new net: C157.1, R161.1
- new net: C157.2, U25.1 (BST)
- new net: CONTACT_CHGR1.1, CONTACT_CHGR1.2, DC1.3
- new net: C162.1, U2.4 (SS)
- new net: C156.1, U25.4 (SS)
- new net PWR_EN: R43.1, U25.3 (EN)
- no-connect marks 14 -> 8
Other:
- note removed: ".I2C Address = 0x20 .Min Voltage= 5V .Max Voltage= 20V .Op Current= 1A .Max Current= 5A"
- note removed: "NOTE : D+ , D_ are connected to CM4/5"
- note removed: "NOTE : SDA,SCL,nINT are connected to MCU"
- note removed: "POWER DELIVERY"
- moved on the sheet: CONTACT_CHGR1, D34, USB2

Commit message: Update Power Control sch, Charger sch, Speaker + Mic, JTAG and Watch Dog
**Power Control:** Replaced the BJT with a MOSFET. The MCU hang condition is not covered yet.
Parts:
- removed C100, C83, C96, C97, C98, C99: 10uF/25V, Capacitor_SMD:C_0603_1608Metric, symbol Device:C
- removed C125: 10uF/50V, Capacitor_SMD:C_0805_2012Metric, symbol Library:C_0603
- removed C67, C68, C69, C78, C80, C81, C82: 10uF/50V, Capacitor_SMD:C_0805_2012Metric, symbol Device:C
- removed C70: 4.7uF/10V, Capacitor_SMD:C_0603_1608Metric, symbol Device:C
- removed C75, C79: 47nF/50V, Capacitor_SMD:C_0603_1608Metric, symbol Device:C
- removed C77: 1nF/50V, Capacitor_SMD:C_0603_1608Metric, symbol Device:C
- removed CN2: EV2400, JLCImport:A2543WV-4P, symbol JLCImport:A2543WV-4P
- removed D1: SMBJ24A_C908801, JLCImport:SMBJ24A_C908801, symbol JLCImport:SMBJ24A_C908801
- removed D10: SS34, Diode_SMD:D_SMA, symbol DesignLibrary:WATER-PUMP_1_DIODE-2_DesignLibrary.SchLib
- removed D29: 3V3-STAT, oomwoo_altium:LED0603-B, symbol DesignLibrary:POWER_0_LED-SMD_DesignLibrary.SchLib
- removed D3: SMAJ18A_C148219, JLCImport:SMAJ18A_C148219, symbol JLCImport:SMAJ18A_C148219
- removed D34: TPD2EUSB30DRTR, TPD2EUSB30DRTR:SOTFL35P100X50-3N, symbol TPD2EUSB30DRTR:TPD2EUSB30DRTR
- removed L7: 1uH, JLCImport:GSM0420-1R0-M, symbol JLCImport:GSM0420-1R0-M
- removed R100: 100, Resistor_SMD:R_0603_1608Metric, symbol Device:R_US
- removed R115: 100k, Resistor_SMD:R_0603_1608Metric, symbol Device:R_US
- removed R127: 5.24k, Resistor_SMD:R_0603_1608Metric, symbol Device:R_US
- removed R129: 17.4k, Resistor_SMD:R_0603_1608Metric, symbol Device:R_US
- removed R132: 10k, Resistor_SMD:R_0603_1608Metric, symbol Device:R_US
- removed R37: 1k, Resistor_SMD:R_0603_1608Metric, symbol DesignLibrary:POWER_2_Resistor-1_DesignLibrary.SchLib
- removed R60: 30.31k, Resistor_SMD:R_0603_1608Metric, symbol Device:R_US
- removed R99: 215k, Resistor_SMD:R_0603_1608Metric, symbol Device:R_US
- removed U7: BQ25792RQMR, JLCImport:BQ25792RQMR, symbol JLCImport:BQ25792RQMR
- added C158, C167: 100nF/25V, Capacitor_SMD:C_0603_1608Metric, symbol Library:C_0603
- added C164, C165, C166, C168: 10uF/25V, Capacitor_SMD:C_0603_1608Metric, symbol JLCImport:CL21A106KBYQNNE
- added C8: 220nF, symbol Device:C_Small
- added D1: USBLC6-2SC6_C2687116, JLCImport:USBLC6-2SC6_C2687116, symbol JLCImport:USBLC6-2SC6_C2687116
- added D12, D13, D14, D15: SS56, JLCImport:SS56, symbol JLCImport:SS56
- added L1: SMMS0630-100M, JLCImport:SMMS0630-100M, symbol JLCImport:SMMS0630-100M
- added LED_CHG1, LED_STDBY1: (no value), oomwoo_altium:LED0603-B, symbol DesignLibrary:POWER_0_LED-SMD_DesignLibrary.SchLib
- added Q12, Q14: AOD407_C6396162, JLCImport:AOD407_C6396162, symbol JLCImport:AOD407_C6396162
- added R104, R105, R107: 10k, Resistor_SMD:R_0603_1608Metric, symbol Device:R_US
- added R106: RE1206F1R050, JLCImport:RE1206F1R050, symbol JLCImport:RE1206F1R050
- added R175: 100k, Resistor_SMD:R_0603_1608Metric, symbol Device:R_US
- added R37: 120 Ohm, symbol Device:R_US
- added R59: FRC0805J1R0TS, JLCImport:FRC0805J1R0TS, symbol JLCImport:FRC0805J1R0TS
- added U1: SLM6900, JLCImport:SLM6900, symbol JLCImport:SLM6900
Connections:
- net BAT-VCC: now also D14.1 (K), Q14.3 (S)
- net D+: now also D1.3 (I/O2), D1.4 (I/O2)
- net D-: now also D1.1 (I/O1), D1.6 (I/O1)
- net GND: now also C158.2, C164.2, C165.2, C168.2, C8.2, D1.2 (GND), D13.2 (A), D15.2 (A), R175.2, R59.2, U1.12 (GND), U1.13 (PGND)
- net NTC: now also U1.6 (NTC)
- net P+/C+: now also C168.1, Q14.2 (D), R106.2, R107.2, U1.10 (ISN)
- net VBUS: now also D1.5 (VBUS), D15.1 (K)
- net VCC-CHARGE renamed DC_IN
- net DC_IN: now also C158.1, C164.1, C165.1, C166.1, C167.1, D14.2 (A), LED_CHG1.1, LED_STDBY1.1, Q12.3 (S), Q14.1 (G), R175.1, U1.2 (PVCC), U1.3 (VCC), U1.7 (SEL)
- new net: D12.1 (K), L1.1
- new net: L1.2, R106.1, U1.11 (ISP)
- new net: R37.1, U1.8 (COMP)
- new net: C8.1, R37.2
- new net: C166.2, R59.1
- new net: Q12.1 (G), U1.1 (DRV)
- new net: D12.2 (A), D13.1 (K), Q12.2 (D)
- new net: R107.1, U1.9 (FB)
- new net: LED_CHG1.2, R105.1
- new net: LED_STDBY1.2, R104.1
- new net: R104.2, U1.5 (NSTDBY)
- new net: C167.2, U1.14 (GVC)
- new net: R105.2, U1.4 (NCHRG)
- no-connect marks 8 -> 4
Other:
- note added: "2.2 - 2.6 Amp"
- note added: "configured as 4S"
- note removed: "4S/1Amp"
- note removed: "Freq=1.5MHz"
- note removed: "I Limit = 5 Amp"
- note removed: "OPTIONAL"
- note removed: "Put the MCU into RESET mode if use EV2400 to debug the charger"

Commit message: Assigned footprints
Parts:
- C8: value 220nF -> 220nF/25V; footprint (none) -> Capacitor_SMD:C_0603_1608Metric
- R37: footprint (none) -> Resistor_SMD:R_0603_1608Metric
Changed lines of the file:
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@@
 			)
 		)
-		(property "Footprint" ""
+		(property "Footprint" "Resistor_SMD:R_0603_1608Metric"
 			(at 228.854 352.679 90)
 			(hide yes)
@@
 			)
 		)
-		(property "Value" "220nF"
+		(property "Value" "220nF/25V"
 			(at 240.665 359.41 90)
 			(show_name no)
@@
 			)
 		)
-		(property "Footprint" ""
+		(property "Footprint" "Capacitor_SMD:C_0603_1608Metric"
 			(at 240.665 353.695 0)
 			(hide yes)
