File: kicad/main-phone/Front-Sensors.kicad_sch (KiCad schematic)
At the start: 15 parts

Commit message: Front sensors rev 2: IR receivers onto main-phone, ToF board x2 on JST SH
- main-phone FRONT SENSORS: IR-F1/IR-F2 connectors replaced by two
  side-looking IRM-V838M3-C receivers on the board (U7501 left, U7502
  right) with 100R + 10uF filters; IRM-H638T is top-looking
- VL-L1/VL-R1: ZX-SH1.0-7PWT (JST SH compatible), same pinout
- kicad/front-sensors: one VL53L7 breakout fitted twice, refs 83xx, no
  pull-ups (main board has them), RSVD6 47k, ferrite to AVDD; the sensor
  is hand-placed (not in the JLC BOM/CPL); uses the shared ../main libs
- shared JLCImport: VL53L7, BLM18PG121SN1D, IRM-V838M3-C, ZX-SH1_0-7PWT
- docs: SPEC, READMEs, new front-sensors README

Co-Authored-By: Claude Opus 5.5 (1M context) <noreply@anthropic.com>
Parts:
- removed IR-F1, IR-F2: ZX-ZH1_5-4PWT, JLCImport:ZX-ZH1_5-4PWT, symbol JLCImport:ZX-ZH1_5-4PWT
- added R7501, R7502: 100, Resistor_SMD:R_0603_1608Metric, symbol Device:R_US
- added U7501, U7502: IRM-V838M3-C/TR1, JLCImport:IRM-V838M3-C, symbol JLCImport:IRM-V838M3-C
- VL-L1, VL-R1: value ZX-ZH1_5-7PWT -> ZX-SH1_0-7PWT; footprint JLCImport:ZX-ZH1_5-7PWT -> JLCImport:ZX-SH1_0-7PWT; symbol JLCImport:ZX-ZH1_5-7PWT -> JLCImport:ZX-SH1_0-7PWT; LCSC C19272410 -> C7430449; Manufacturer Part ZX-ZH1.5-7PWT -> ZX-SH1.0-7PWT
Connections:
- net GND: now also U7501.1 (GND), U7501.4 (GND), U7502.1 (GND), U7502.4 (GND)
- net IR-F-RX1: now also U7501.3 (OUT)
- net IR-F-RX2: now also U7502.3 (OUT)
- net VCC-3V3-REG: now also R7501.1, R7502.1; no longer C90.1, C91.1
- new net: C90.1, R7502.2, U7502.2 (VCC)
- new net: C91.1, R7501.2, U7501.2 (VCC)
Other:
- note added: "2x VL53L7 ToF BOARDS"
- note added: "U7501 left, U7502 right (robot view). Side-looking: put both at the board front edge, lenses facing forward, ~10 mm apart, with a baffle between them in the bumper window."
- note removed: "2x VL53L7CX"
- note removed: "RECEIVER"

Commit message: main-phone: free MCU pins; 2x11 spare header with UART and I2C
- LiDAR rail enable joins ~VM-VBAT-EN (PE10); PD9 freed
- IMU FSYNC/INT2 go to J7301 instead of the MCU; FSYNC 100k pull-down (R7601); PD4/PD7 freed
- one open-drain ToF interrupt (PD12) for both VL53L7s and the side VL53L0X; PC8/PE2 freed
- right VL53L7 LPn held up by R7307, no MCU pin; PE8 freed
- IMU moved from I2C2 to I2C4 (R18/R72 not fitted); PA8/PA9 freed;
  R7315 keeps PA9 (UCPD DBCC1) pulled up for dead-battery Rd on CC1
- PWR_EN moved PC10 -> PD7; PC10/PC11 are a spare UART
- J7301 2x6 -> 2x11: 3.3 V, 5 V, I2C4, UART, 12 spare GPIO, IMU FSYNC/INT2, GND
- docs: SPEC, main-phone and side-sensor READMEs

Co-Authored-By: Claude Opus 5.5 <noreply@anthropic.com>
Changed lines of the file:
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@@
 		)
 	)
-	(hierarchical_label "VL-R-LPn"
-		(shape input)
+	(label "VL-R-LPn"
 		(at 46.355 88.9 180)
 		(effects
@@
 				(size 1.27 1.27)
 			)
-			(justify right)
+			(justify right bottom)
 		)
 	)
