File: kicad/main-phone/Front-Sensors.kicad_sch (KiCad schematic)
At the start: 17 parts, among them U7501 IRM-V838M3-C/TR1, U7502 IRM-V838M3-C/TR1

Commit message: LiDAR header, shunt, holes, Hall connector, INT pullup fix
Parts:
- removed R7: 47k, Resistor_SMD:R_0603_1608Metric, symbol Device:R_US
