File: kicad/main-phone/Front-Sensors.kicad_sch (KiCad schematic)
At the start: 16 parts, among them U7501 IRM-V838M3-C/TR1, U7502 IRM-V838M3-C/TR1

Commit message: Per-board reference ranges, J1 spare header, IMU AD0 pull-down, BOM outputs
- reference ranges: main-phone 1-999, dock 1000s, front ToF 2000s, side 3000s,
  cliff 4000s, rear IR 5000s, Hall 6000s (main-phone 7xxx parts renumbered
  below 1000; sensor boards and dock moved from 8xxx)
- main-phone: J7301 -> J1, a fitted 2x7 0.1" header with spares only
  (3.3 V, 5 V, I2C4, UART PC10/PC11, PA8-PA10, PD4, PE2, PE6, GND)
- IMU: AP_AD0 pulled low by R217 (address 0x68); INT2 on test pad TP1;
  FSYNC reachable on R211; R18/R72 removed
- tools/export.py replaces export_pdfs.py: schematic PDF and JLC-style BOM in
  each board's output/ folder; --pcb adds Gerbers, placement and STEP
- cliff and rear IR projects: fix top-level sheet left over from a copy
- Hall board: visual tidy-up

Co-Authored-By: Claude Opus 5.5 <noreply@anthropic.com>
Parts:
- renumbered R7307 to R196, R7501 to R209, R7502 to R210, U7501 to U24, U7502 to U25
Other:
- note added: "U24 left, U25 right (robot view). Side-looking: put both at the board front edge, lenses facing forward, ~10 mm apart, with a baffle between them in the bumper window."
- note removed: "U7501 left, U7502 right (robot view). Side-looking: put both at the board front edge, lenses facing forward, ~10 mm apart, with a baffle between them in the bumper window."
Changed lines of the file:
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@@
 			)
 		)
-		(property "Description" "JST SH compatible 1.0 mm 1x7P, SMD right angle; to a front ToF board (J8301)"
+		(property "Description" "JST SH compatible 1.0 mm 1x7P, SMD right angle; to a front ToF board (J2001)"
 			(at 100.965 81.28 0)
 			(hide yes)
@@
 			)
 		)
-		(property "Description" "JST SH compatible 1.0 mm 1x7P, SMD right angle; to a front ToF board (J8301)"
+		(property "Description" "JST SH compatible 1.0 mm 1x7P, SMD right angle; to a front ToF board (J2001)"
 			(at 100.965 111.76 0)
 			(hide yes)
@@
 		(in_pos_files yes)
 		(dnp no)
-		(property "Reference" "R7307"
+		(property "Reference" "R196"
 			(at 53.975 92.075 0)
 			(show_name no)
@@
 			(project "Main"
 				(path "/dbcfb655-8d45-4808-9a74-2a0eb03372e8/bbba09df-157d-4294-b403-7dc3ed0c5481"
-					(reference "R7307")
+					(reference "R196")
 					(unit 1)
 				)
@@
 		(in_pos_files yes)
 		(dnp no)
-		(property "Reference" "R7501"
+		(property "Reference" "R209"
 			(at 196.85 63.5 90)
 			(show_name no)
@@
 			(project "Main"
 				(path "/dbcfb655-8d45-4808-9a74-2a0eb03372e8/bbba09df-157d-4294-b403-7dc3ed0c5481"
-					(reference "R7501")
+					(reference "R209")
 					(unit 1)
 				)
@@
 		(in_pos_files yes)
 		(dnp no)
-		(property "Reference" "U7501"
+		(property "Reference" "U24"
 			(at 227.33 74.93 0)
 			(show_name no)
@@
 			(project "Main"
 				(path "/dbcfb655-8d45-4808-9a74-2a0eb03372e8/bbba09df-157d-4294-b403-7dc3ed0c5481"
-					(reference "U7501")
+					(reference "U24")
 					(unit 1)
 				)
@@
 		(in_pos_files yes)
 		(dnp no)
-		(property "Reference" "R7502"
+		(property "Reference" "R210"
 			(at 196.85 119.38 90)
 			(show_name no)
@@
 			(project "Main"
 				(path "/dbcfb655-8d45-4808-9a74-2a0eb03372e8/bbba09df-157d-4294-b403-7dc3ed0c5481"
-					(reference "R7502")
+					(reference "R210")
 					(unit 1)
 				)
@@
 		(in_pos_files yes)
 		(dnp no)
-		(property "Reference" "U7502"
+		(property "Reference" "U25"
 			(at 227.33 130.81 0)
 			(show_name no)
@@
 			(project "Main"
 				(path "/dbcfb655-8d45-4808-9a74-2a0eb03372e8/bbba09df-157d-4294-b403-7dc3ed0c5481"
-					(reference "U7502")
+					(reference "U25")
 					(unit 1)
 				)
@@
 		)
 	)
-	(text "U7501 left, U7502 right (robot view). Side-looking: put both at the board front edge,\nlenses facing forward, ~10 mm apart, with a baffle between them in the bumper window."
+	(text "U24 left, U25 right (robot view). Side-looking: put both at the board front edge,\nlenses facing forward, ~10 mm apart, with a baffle between them in the bumper window."
 		(exclude_from_sim no)
 		(at 154.94 54.61 0)
