File: kicad/main-phone/CLIFF.kicad_sch (KiCad schematic)
At the start: 21 parts, among them Q7304 AO3400, Q7701 AO3400

Commit message: LiDAR header, shunt, holes, Hall connector, INT pullup fix
Connections:
- net GND: now also CLIFF-LF1.5, CLIFF-LF1.6, CLIFF-LM1.5, CLIFF-LM1.6, CLIFF-LR1.5, CLIFF-LR1.6, CLIFF-RF1.5, CLIFF-RF1.6, CLIFF-RM1.5, CLIFF-RM1.6, CLIFF-RR1.5, CLIFF-RR1.6
- no-connect marks 12 -> 0
