File: kicad/main-phone/CLIFF.kicad_sch (KiCad schematic)
At the start: 21 parts, among them Q7304 AO3400, Q7701 AO3400

Commit message: Per-board reference ranges, J1 spare header, IMU AD0 pull-down, BOM outputs
- reference ranges: main-phone 1-999, dock 1000s, front ToF 2000s, side 3000s,
  cliff 4000s, rear IR 5000s, Hall 6000s (main-phone 7xxx parts renumbered
  below 1000; sensor boards and dock moved from 8xxx)
- main-phone: J7301 -> J1, a fitted 2x7 0.1" header with spares only
  (3.3 V, 5 V, I2C4, UART PC10/PC11, PA8-PA10, PD4, PE2, PE6, GND)
- IMU: AP_AD0 pulled low by R217 (address 0x68); INT2 on test pad TP1;
  FSYNC reachable on R211; R18/R72 removed
- tools/export.py replaces export_pdfs.py: schematic PDF and JLC-style BOM in
  each board's output/ folder; --pcb adds Gerbers, placement and STEP
- cliff and rear IR projects: fix top-level sheet left over from a copy
- Hall board: visual tidy-up

Co-Authored-By: Claude Opus 5.5 <noreply@anthropic.com>
Parts:
- renumbered Q7304 to Q32, Q7701 to Q35, R7308 to R197, R7309 to R198, R7701 to R212, R7702 to R213, R7703 to R214
Other:
- note added: "Cliff sensors: 6 boards (kicad/cliff-sensor), SH 4-pin vertical: 1 VCC-5V-REG (LED, 150R on the board), 2 CLIFF-LED-K (Q35 sinks all 6 LEDs), 3 phototransistor collector (47k pull-up), 4 GND. Modulate CLIFF_LED_EN and read each channel LED-on minus LED-off to cancel ambient light. ADC: LF PA3, RF PA1, LR PA2, RR PA0, LM PD9, RM PE8 (LM/RM via global labels)."
- note removed: "Cliff sensors: 6 boards (kicad/cliff-sensor), SH 4-pin vertical: 1 VCC-5V-REG (LED, 150R on the board), 2 CLIFF-LED-K (Q7701 sinks all 6 LEDs), 3 phototransistor collector (47k pull-up), 4 GND. Modulate CLIFF_LED_EN and read each channel LED-on minus LED-off to cancel ambient light. ADC: LF PA3, RF PA1, LR PA2, RR PA0, LM PD9, RM PE8 (LM/RM via global labels)."
Changed lines of the file:
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@@
 		(in_pos_files yes)
 		(dnp no)
-		(property "Reference" "R7308"
+		(property "Reference" "R197"
 			(at 181.61 102.235 0)
 			(show_name no)
@@
 			(project "Main"
 				(path "/dbcfb655-8d45-4808-9a74-2a0eb03372e8/eb65cbe8-a43a-448e-bb05-c96139672d5e"
-					(reference "R7308")
+					(reference "R197")
 					(unit 1)
 				)
@@
 		(in_pos_files yes)
 		(dnp no)
-		(property "Reference" "Q7304"
+		(property "Reference" "Q32"
 			(at 193.04 144.78 0)
 			(show_name no)
@@
 			(project "Main"
 				(path "/dbcfb655-8d45-4808-9a74-2a0eb03372e8/eb65cbe8-a43a-448e-bb05-c96139672d5e"
-					(reference "Q7304")
+					(reference "Q32")
 					(unit 1)
 				)
@@
 		(in_pos_files yes)
 		(dnp no)
-		(property "Reference" "R7309"
+		(property "Reference" "R198"
 			(at 172.72 150.495 0)
 			(show_name no)
@@
 			(project "Main"
 				(path "/dbcfb655-8d45-4808-9a74-2a0eb03372e8/eb65cbe8-a43a-448e-bb05-c96139672d5e"
-					(reference "R7309")
+					(reference "R198")
 					(unit 1)
 				)
@@
 			)
 		)
-		(property "Description" "JST SH compatible 1.0 mm 1x4P, SMD vertical; to a cliff sensor board (J8501)"
+		(property "Description" "JST SH compatible 1.0 mm 1x4P, SMD vertical; to a cliff sensor board (J4001)"
 			(at 38.1 88.9 0)
 			(hide yes)
@@
 			)
 		)
-		(property "Description" "JST SH compatible 1.0 mm 1x4P, SMD vertical; to a cliff sensor board (J8501)"
+		(property "Description" "JST SH compatible 1.0 mm 1x4P, SMD vertical; to a cliff sensor board (J4001)"
 			(at 38.1 116.84 0)
 			(hide yes)
@@
 			)
 		)
-		(property "Description" "JST SH compatible 1.0 mm 1x4P, SMD vertical; to a cliff sensor board (J8501)"
+		(property "Description" "JST SH compatible 1.0 mm 1x4P, SMD vertical; to a cliff sensor board (J4001)"
 			(at 38.1 144.78 0)
 			(hide yes)
@@
 			)
 		)
-		(property "Description" "JST SH compatible 1.0 mm 1x4P, SMD vertical; to a cliff sensor board (J8501)"
+		(property "Description" "JST SH compatible 1.0 mm 1x4P, SMD vertical; to a cliff sensor board (J4001)"
 			(at 88.9 88.9 0)
 			(hide yes)
@@
 			)
 		)
-		(property "Description" "JST SH compatible 1.0 mm 1x4P, SMD vertical; to a cliff sensor board (J8501)"
+		(property "Description" "JST SH compatible 1.0 mm 1x4P, SMD vertical; to a cliff sensor board (J4001)"
 			(at 88.9 116.84 0)
 			(hide yes)
@@
 			)
 		)
-		(property "Description" "JST SH compatible 1.0 mm 1x4P, SMD vertical; to a cliff sensor board (J8501)"
+		(property "Description" "JST SH compatible 1.0 mm 1x4P, SMD vertical; to a cliff sensor board (J4001)"
 			(at 88.9 144.78 0)
 			(hide yes)
@@
 		(in_pos_files yes)
 		(dnp no)
-		(property "Reference" "R7701"
+		(property "Reference" "R212"
 			(at 153.035 99.695 90)
 			(show_name no)
@@
 			(project "Main"
 				(path "/dbcfb655-8d45-4808-9a74-2a0eb03372e8/eb65cbe8-a43a-448e-bb05-c96139672d5e"
-					(reference "R7701")
+					(reference "R212")
 					(unit 1)
 				)
@@
 		(in_pos_files yes)
 		(dnp no)
-		(property "Reference" "R7702"
+		(property "Reference" "R213"
 			(at 159.385 99.695 90)
 			(show_name no)
@@
 			(project "Main"
 				(path "/dbcfb655-8d45-4808-9a74-2a0eb03372e8/eb65cbe8-a43a-448e-bb05-c96139672d5e"
-					(reference "R7702")
+					(reference "R213")
 					(unit 1)
 				)
@@
 		(in_pos_files yes)
 		(dnp no)
-		(property "Reference" "Q7701"
+		(property "Reference" "Q35"
 			(at 156.21 156.21 0)
 			(show_name no)
@@
 			(project "Main"
 				(path "/dbcfb655-8d45-4808-9a74-2a0eb03372e8/eb65cbe8-a43a-448e-bb05-c96139672d5e"
-					(reference "Q7701")
+					(reference "Q35")
 					(unit 1)
 				)
@@
 		(in_pos_files yes)
 		(dnp no)
-		(property "Reference" "R7703"
+		(property "Reference" "R214"
 			(at 135.89 161.29 0)
 			(show_name no)
@@
 			(project "Main"
 				(path "/dbcfb655-8d45-4808-9a74-2a0eb03372e8/eb65cbe8-a43a-448e-bb05-c96139672d5e"
-					(reference "R7703")
+					(reference "R214")
 					(unit 1)
 				)
@@
 		)
 	)
-	(text "Cliff sensors: 6 boards (kicad/cliff-sensor), SH 4-pin vertical: 1 VCC-5V-REG (LED, 150R on the board),\n2 CLIFF-LED-K (Q7701 sinks all 6 LEDs), 3 phototransistor collector (47k pull-up), 4 GND.\nModulate CLIFF_LED_EN and read each channel LED-on minus LED-off to cancel ambient light.\nADC: LF PA3, RF PA1, LR PA2, RR PA0, LM PD9, RM PE8 (LM/RM via global labels)."
+	(text "Cliff sensors: 6 boards (kicad/cliff-sensor), SH 4-pin vertical: 1 VCC-5V-REG (LED, 150R on the board),\n2 CLIFF-LED-K (Q35 sinks all 6 LEDs), 3 phototransistor collector (47k pull-up), 4 GND.\nModulate CLIFF_LED_EN and read each channel LED-on minus LED-off to cancel ambient light.\nADC: LF PA3, RF PA1, LR PA2, RR PA0, LM PD9, RM PE8 (LM/RM via global labels)."
 		(exclude_from_sim no)
 		(at 25.4 182.88 0)
