File: kicad/main-phone/LIDAR.kicad_sch (KiCad schematic)
At the start: 15 parts, among them Q20 AO3400, Q7002 AO3401, Q7003 AO3400

Commit message: LiDAR header, shunt, holes, Hall connector, INT pullup fix
Parts:
- removed LIDAR2: PZ254R-11-05P, Connector_PinHeader_2.54mm:PinHeader_1x05_P2.54mm_Horizontal, symbol Connector:Conn_01x05_Pin
- added LIDAR2: LIDAR-ALT (DNP), Connector_PinHeader_2.54mm:PinHeader_2x03_P2.54mm_Vertical, symbol Connector_Generic:Conn_02x03_Odd_Even
- added R113: 100, Resistor_SMD:R_0603_1608Metric, symbol Device:R_US
- R66, R7008: value 1k -> 100; LCSC C2907113 -> C2906981
Connections:
- net GND: now also LIDAR2.2 (Pin_2)
- net LiDAR-MOT-: now also LIDAR2.3 (Pin_3)
- net LiDAR-TXD: now also R113.1; no longer LIDAR1.3
- net VM-5V-LIDAR: now also LIDAR2.4 (Pin_4), LIDAR2.6 (Pin_6)
- net at R66.2: now also LIDAR2.1 (Pin_1)
- new net LiDAR-TX-J: LIDAR1.3, LIDAR2.5 (Pin_5), R113.2
- no-connect marks 1 -> 0
Other:
- note added: "R66, R113, R7008: 100R series resistors on the LiDAR signals. Only one LiDAR is fitted: LIDAR1 (LD14P) or a header/cable on LIDAR2."
- note added: "VM-5V-LIDAR powers the whole LiDAR (laser included) for any model. On only while WD_OK is high AND LiDAR-EN is low (Q7003 source-switched AND). R7006/C7003: ~1.5 ms soft start, ~30 ms soft stop. LIDAR2: 2x3 0.1in through-hole pads (not fitted) for other LiDARs. Pin 6 = VM-5V-LIDAR for LiDARs that need a separate motor supply (motor between pins 6 and 3). Pin 5 = the LiDAR TX, shared with LIDAR1 p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"
- note removed: "LIDAR2 and STM32_DEBUG1 use the same right-angle 1x5 0.1in header (PZ254R-11-05P), one BOM line. LIDAR2 pin 5 is unused."
- note removed: "VM-5V-LIDAR powers the whole LiDAR (laser included) for any model. On only while WD_OK is high AND LiDAR-EN is low (Q7003 source-switched AND). R7006/C7003: ~1.5 ms soft start, ~30 ms soft stop. LIDAR2: 0.1in header for other LiDARs (pin 2 now GND)."
