File: kicad/main-phone/LIDAR.kicad_sch (KiCad schematic)
At the start: 16 parts, among them Q20 AO3400, Q7002 AO3401, Q7003 AO3400

Commit message: Per-board reference ranges, J1 spare header, IMU AD0 pull-down, BOM outputs
- reference ranges: main-phone 1-999, dock 1000s, front ToF 2000s, side 3000s,
  cliff 4000s, rear IR 5000s, Hall 6000s (main-phone 7xxx parts renumbered
  below 1000; sensor boards and dock moved from 8xxx)
- main-phone: J7301 -> J1, a fitted 2x7 0.1" header with spares only
  (3.3 V, 5 V, I2C4, UART PC10/PC11, PA8-PA10, PD4, PE2, PE6, GND)
- IMU: AP_AD0 pulled low by R217 (address 0x68); INT2 on test pad TP1;
  FSYNC reachable on R211; R18/R72 removed
- tools/export.py replaces export_pdfs.py: schematic PDF and JLC-style BOM in
  each board's output/ folder; --pcb adds Gerbers, placement and STEP
- cliff and rear IR projects: fix top-level sheet left over from a copy
- Hall board: visual tidy-up

Co-Authored-By: Claude Opus 5.5 <noreply@anthropic.com>
Parts:
- renumbered C7003 to C171, Q7002 to Q25, Q7003 to Q26, R7005 to R180, R7006 to R181, R7007 to R182, R7008 to R183
Other:
- note added: "R66, R113, R183: 100R series resistors on the LiDAR signals. Only one LiDAR is fitted: LIDAR1 (LD14P) or a header/cable on LIDAR2."
- note added: "VM-5V-LIDAR powers the whole LiDAR (laser included) for any model. On only while WD_OK is high AND LiDAR-EN is low (Q26 source-switched AND). R181/C171: ~1.5 ms soft start, ~30 ms soft stop. LIDAR2: 2x3 0.1in through-hole pads (not fitted) for other LiDARs. Pin 6 = VM-5V-LIDAR for LiDARs that need a separate motor supply (motor between pins 6 and 3). Pin 5 = the LiDAR TX, shared with LIDAR1 pin 3."
- note removed: "R66, R113, R7008: 100R series resistors on the LiDAR signals. Only one LiDAR is fitted: LIDAR1 (LD14P) or a header/cable on LIDAR2."
- note removed: "VM-5V-LIDAR powers the whole LiDAR (laser included) for any model. On only while WD_OK is high AND LiDAR-EN is low (Q7003 source-switched AND). R7006/C7003: ~1.5 ms soft start, ~30 ms soft stop. LIDAR2: 2x3 0.1in through-hole pads (not fitted) for other LiDARs. Pin 6 = VM-5V-LIDAR for LiDARs that need a separate motor supply (motor between pins 6 and 3). Pin 5 = the LiDAR TX, shared with LIDAR1 p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"
Changed lines of the file:
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@@
 		)
 	)
-	(text "VM-5V-LIDAR powers the whole LiDAR (laser included) for any model. On only while WD_OK is high\nAND LiDAR-EN is low (Q7003 source-switched AND). R7006/C7003: ~1.5 ms soft start, ~30 ms soft stop.\nLIDAR2: 2x3 0.1in through-hole pads (not fitted) for other LiDARs. Pin 6 = VM-5V-LIDAR for LiDARs\nthat need a separate motor supply (motor between pins 6 and 3). Pin 5 = the LiDAR TX, shared with LIDAR1 pin 3."
+	(text "VM-5V-LIDAR powers the whole LiDAR (laser included) for any model. On only while WD_OK is high\nAND LiDAR-EN is low (Q26 source-switched AND). R181/C171: ~1.5 ms soft start, ~30 ms soft stop.\nLIDAR2: 2x3 0.1in through-hole pads (not fitted) for other LiDARs. Pin 6 = VM-5V-LIDAR for LiDARs\nthat need a separate motor supply (motor between pins 6 and 3). Pin 5 = the LiDAR TX, shared with LIDAR1 pin 3."
 		(exclude_from_sim no)
 		(at 60.325 35.56 0)
@@
 		)
 	)
-	(text "R66, R113, R7008: 100R series resistors on the LiDAR signals. Only one LiDAR is fitted:\nLIDAR1 (LD14P) or a header/cable on LIDAR2."
+	(text "R66, R113, R183: 100R series resistors on the LiDAR signals. Only one LiDAR is fitted:\nLIDAR1 (LD14P) or a header/cable on LIDAR2."
 		(exclude_from_sim no)
 		(at 190.5 172.72 0)
@@
 		(in_pos_files yes)
 		(dnp no)
-		(property "Reference" "R7006"
+		(property "Reference" "R181"
 			(at 80.645 108.585 0)
 			(show_name no)
@@
 			)
 		)
-		(property "Description" "Soft-start: with C7003 about 1.5 ms turn-on ramp"
+		(property "Description" "Soft-start: with C171 about 1.5 ms turn-on ramp"
 			(at 86.36 109.22 0)
 			(hide yes)
@@
 			(project "Main"
 				(path "/dbcfb655-8d45-4808-9a74-2a0eb03372e8/994d55da-8e8c-4fe8-9877-f2e4533982e7"
-					(reference "R7006")
+					(reference "R181")
 					(unit 1)
 				)
@@
 		(in_pos_files yes)
 		(dnp no)
-		(property "Reference" "Q7003"
+		(property "Reference" "Q26"
 			(at 88.9 117.475 0)
 			(show_name no)
@@
 			(project "Main"
 				(path "/dbcfb655-8d45-4808-9a74-2a0eb03372e8/994d55da-8e8c-4fe8-9877-f2e4533982e7"
-					(reference "Q7003")
+					(reference "Q26")
 					(unit 1)
 				)
@@
 		(in_pos_files yes)
 		(dnp no)
-		(property "Reference" "R7008"
+		(property "Reference" "R183"
 			(at 139.065 60.96 90)
 			(show_name no)
@@
 			(project "Main"
 				(path "/dbcfb655-8d45-4808-9a74-2a0eb03372e8/994d55da-8e8c-4fe8-9877-f2e4533982e7"
-					(reference "R7008")
+					(reference "R183")
 					(unit 1)
 				)
@@
 		(in_pos_files yes)
 		(dnp no)
-		(property "Reference" "Q7002"
+		(property "Reference" "Q25"
 			(at 101.6 100.965 0)
 			(show_name no)
@@
 			(project "Main"
 				(path "/dbcfb655-8d45-4808-9a74-2a0eb03372e8/994d55da-8e8c-4fe8-9877-f2e4533982e7"
-					(reference "Q7002")
+					(reference "Q25")
 					(unit 1)
 				)
@@
 		(in_pos_files yes)
 		(dnp no)
-		(property "Reference" "R7007"
+		(property "Reference" "R182"
 			(at 81.915 128.905 0)
 			(show_name no)
@@
 			(project "Main"
 				(path "/dbcfb655-8d45-4808-9a74-2a0eb03372e8/994d55da-8e8c-4fe8-9877-f2e4533982e7"
-					(reference "R7007")
+					(reference "R182")
 					(unit 1)
 				)
@@
 		(in_pos_files yes)
 		(dnp no)
-		(property "Reference" "C7003"
+		(property "Reference" "C171"
 			(at 93.345 114.3 90)
 			(show_name no)
@@
 			(project "Main"
 				(path "/dbcfb655-8d45-4808-9a74-2a0eb03372e8/994d55da-8e8c-4fe8-9877-f2e4533982e7"
-					(reference "C7003")
+					(reference "C171")
 					(unit 1)
 				)
@@
 		(in_pos_files yes)
 		(dnp no)
-		(property "Reference" "R7005"
+		(property "Reference" "R180"
 			(at 85.725 94.615 0)
 			(show_name no)
@@
 			)
 		)
-		(property "Description" "Q7002 gate-source pull-up (off by default)"
+		(property "Description" "Q25 gate-source pull-up (off by default)"
 			(at 91.44 95.25 0)
 			(hide yes)
@@
 			(project "Main"
 				(path "/dbcfb655-8d45-4808-9a74-2a0eb03372e8/994d55da-8e8c-4fe8-9877-f2e4533982e7"
-					(reference "R7005")
+					(reference "R180")
 					(unit 1)
 				)
