File: kicad/main-phone/MAIN-BRUSH-MOTOR .kicad_sch (KiCad schematic)
At the start: 7 parts, among them U20 DRV8870DDAR

Commit message: LiDAR header, shunt, holes, Hall connector, INT pullup fix
Parts:
- R84: value RLH12FTCR110 -> LRBK25EFER110; footprint JLCImport:RLH12FTCR110 -> Resistor_SMD:R_2512_6332Metric; LCSC C22464898 -> C5121166; Manufacturer TA-I Tech -> NCT; Manufacturer Part RLH12FTCR110 -> LRBK25EFER110
Changed lines of the file:
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@@
 			)
 		)
-		(property "Value" "RLH12FTCR110"
+		(property "Value" "LRBK25EFER110"
 			(at 161.29 119.3799 90)
 			(show_name no)
@@
 			)
 		)
-		(property "Footprint" "JLCImport:RLH12FTCR110"
+		(property "Footprint" "Resistor_SMD:R_2512_6332Metric"
 			(at 158.115 118.11 0)
 			(hide yes)
@@
 			)
 		)
-		(property "Datasheet" "https://www.lcsc.com/datasheet/lcsc_datasheet_2406141138_TA-I-Tech-RLH12FTCR110_C22464898.pdf"
+		(property "Datasheet" "https://www.lcsc.com/product-detail/C5121166.html"
 			(at 158.115 118.11 0)
 			(hide yes)
@@
 			)
 		)
-		(property "Description" "110mΩ 1W Current Sense Resistor Surface Mount ±1% ±100ppm/℃ 1206 Current Sense Resistors / Shunt Resistors ROHS"
+		(property "Description" "110mOhm 2W current sense resistor, 2512, 1%"
 			(at 158.115 118.11 0)
 			(hide yes)
@@
 			)
 		)
-		(property "LCSC" "C22464898"
+		(property "LCSC" "C5121166"
 			(at 158.115 118.11 0)
 			(hide yes)
@@
 			)
 		)
-		(property "Manufacturer" "TA-I Tech"
+		(property "Manufacturer" "NCT"
 			(at 158.115 118.11 0)
 			(hide yes)
@@
 			)
 		)
-		(property "Manufacturer Part" "RLH12FTCR110"
+		(property "Manufacturer Part" "LRBK25EFER110"
 			(at 158.115 118.11 0)
 			(hide yes)
