File: kicad/main-phone/SIDE-BRUSH-MOTORs .kicad_sch (KiCad schematic)
At the start: 7 parts, among them U18 DRV8870DDAR

Commit message: LiDAR header, shunt, holes, Hall connector, INT pullup fix
Parts:
- R83: value RL12FTNR300 -> RLH12FTCR300; footprint JLCImport:RL12FTNR300 -> Resistor_SMD:R_1206_3216Metric; LCSC C160919 -> C22464904; Manufacturer Part RL12FTNR300 -> RLH12FTCR300
Changed lines of the file:
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@@
 			)
 		)
-		(property "Value" "RL12FTNR300"
+		(property "Value" "RLH12FTCR300"
 			(at 156.21 126.9999 90)
 			(show_name no)
@@
 			)
 		)
-		(property "Footprint" "JLCImport:RL12FTNR300"
+		(property "Footprint" "Resistor_SMD:R_1206_3216Metric"
 			(at 153.67 125.73 0)
 			(hide yes)
@@
 			)
 		)
-		(property "Datasheet" "https://www.lcsc.com/datasheet/lcsc_datasheet_2304140030_TA-I-Tech-RL12FTNR300_C160919.pdf"
+		(property "Datasheet" "https://www.lcsc.com/product-detail/C22464904.html"
 			(at 153.67 125.73 0)
 			(hide yes)
@@
 			)
 		)
-		(property "Description" "300mΩ 500mW Metal Film Resistor SMD ±1% ±200ppm/℃ 1206 Current Sense Resistors / Shunt Resistors ROHS"
+		(property "Description" "300mOhm 1W current sense resistor, 1206, 1%, 100ppm/C"
 			(at 153.67 125.73 0)
 			(hide yes)
@@
 			)
 		)
-		(property "LCSC" "C160919"
+		(property "LCSC" "C22464904"
 			(at 153.67 125.73 0)
 			(hide yes)
@@
 			)
 		)
-		(property "Manufacturer Part" "RL12FTNR300"
+		(property "Manufacturer Part" "RLH12FTCR300"
 			(at 153.67 125.73 0)
 			(hide yes)
