File: kicad/main-phone/SIDE-PROXIMITY-IR-SENSOR .kicad_sch (KiCad schematic)
At the start: 6 parts

Commit message: LiDAR header, shunt, holes, Hall connector, INT pullup fix
Parts:
- removed HALL-BIN1, HALL-TOWER1: ZX-SH1_0-4PLT, JLCImport:ZX-SH1_0-4PLT, symbol JLCImport:ZX-SH1_0-4PLT
- added HALL-BIN1, HALL-TOWER1: ZX-SH1_0-3PLT, JLCImport:ZX-SH1_0-3PLT, symbol JLCImport:ZX-SH1_0-3PLT
Connections:
- net GND: now also REAR-IR1.5, REAR-IR1.6, HALL-BIN1.3, HALL-BIN1.4, HALL-BIN1.5, HALL-TOWER1.3, HALL-TOWER1.4, HALL-TOWER1.5
- net HALL-BIN: now also HALL-BIN1.2
- net HALL-TOWER: now also HALL-TOWER1.2
- net VCC-3V3-REG: now also HALL-BIN1.1, HALL-TOWER1.1
- no-connect marks 8 -> 0
Other:
- note added: "REAR-IR1: rear docking IR board, 1 3.3 V, 2 IR_L (PC8, TIM3_CH3), 3 IR_R (PC9, TIM3_CH4), 4 GND. HALL-BIN1 / HALL-TOWER1: Hall boards, SH 3-pin (ZX-SH1.0-3PLT, so a Hall cable cannot go into a 4-pin socket): 1 3.3 V, 2 OUT (PE4 / PE5, low = magnet near), 3 GND. All mounting pads to GND."
- note removed: "REAR-IR1: rear docking IR board, 1 3.3 V, 2 IR_L (PC8, TIM3_CH3), 3 IR_R (PC9, TIM3_CH4), 4 GND. HALL-BIN1 / HALL-TOWER1: Hall boards, 1 3.3 V, 2 OUT (PE4 / PE5, low = magnet near), 3 NC, 4 GND. Same connector part as the cliff sensors (ZX-SH1.0-4PLT)."
