File: kicad/main-phone/SIDE-PROXIMITY-IR-SENSOR .kicad_sch (KiCad schematic)
At the start: 6 parts

Commit message: Per-board reference ranges, J1 spare header, IMU AD0 pull-down, BOM outputs
- reference ranges: main-phone 1-999, dock 1000s, front ToF 2000s, side 3000s,
  cliff 4000s, rear IR 5000s, Hall 6000s (main-phone 7xxx parts renumbered
  below 1000; sensor boards and dock moved from 8xxx)
- main-phone: J7301 -> J1, a fitted 2x7 0.1" header with spares only
  (3.3 V, 5 V, I2C4, UART PC10/PC11, PA8-PA10, PD4, PE2, PE6, GND)
- IMU: AP_AD0 pulled low by R217 (address 0x68); INT2 on test pad TP1;
  FSYNC reachable on R211; R18/R72 removed
- tools/export.py replaces export_pdfs.py: schematic PDF and JLC-style BOM in
  each board's output/ folder; --pcb adds Gerbers, placement and STEP
- cliff and rear IR projects: fix top-level sheet left over from a copy
- Hall board: visual tidy-up

Co-Authored-By: Claude Opus 5.5 <noreply@anthropic.com>
Parts:
- renumbered R7801 to R215, R7802 to R216
Changed lines of the file:
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@@
 			)
 		)
-		(property "Description" "JST SH compatible 1.0 mm 1x7P, SMD right angle; to the side sensor board (J8401)"
+		(property "Description" "JST SH compatible 1.0 mm 1x7P, SMD right angle; to the side sensor board (J3001)"
 			(at 134.62 80.01 0)
 			(hide yes)
@@
 			)
 		)
-		(property "Description" "JST SH compatible 1.0 mm 1x4P, SMD vertical; to the rear docking IR board (J8601)"
+		(property "Description" "JST SH compatible 1.0 mm 1x4P, SMD vertical; to the rear docking IR board (J5001)"
 			(at 50.8 137.16 0)
 			(hide yes)
@@
 		(in_pos_files yes)
 		(dnp no)
-		(property "Reference" "R7801"
+		(property "Reference" "R215"
 			(at 116.205 135.89 0)
 			(show_name no)
@@
 			(project "Main"
 				(path "/dbcfb655-8d45-4808-9a74-2a0eb03372e8/5e1370fc-da76-42ab-8a06-17e0cb799727"
-					(reference "R7801")
+					(reference "R215")
 					(unit 1)
 				)
@@
 		(in_pos_files yes)
 		(dnp no)
-		(property "Reference" "R7802"
+		(property "Reference" "R216"
 			(at 128.905 135.89 0)
 			(show_name no)
@@
 			(project "Main"
 				(path "/dbcfb655-8d45-4808-9a74-2a0eb03372e8/5e1370fc-da76-42ab-8a06-17e0cb799727"
-					(reference "R7802")
+					(reference "R216")
 					(unit 1)
 				)
