File: kicad/main-phone/STM32G473.kicad_sch (KiCad schematic)
At the start: 34 parts, among them J7301 SPARE-IO (DNP), T1 NTCG164KF104FT1, U13 STM32G473VCT6, X1 ABM3-8_000MHZ-D2Y-T, X3 XKXEL89CII-SUAYLC-32_768K

Commit message: LiDAR header, shunt, holes, Hall connector, INT pullup fix
Parts:
- removed R113: 1k, Resistor_SMD:R_0603_1608Metric, symbol Device:R_US
- removed R117: 10, Resistor_SMD:R_0603_1608Metric, symbol Device:R_US
Connections:
- net LIDAR_RX: now also U13.81 (PC12)
- net LIDAR_TX: now also U13.84 (PD2)
- net NTC: now reaches R38.1, T1.1, U13.34 (PB2)
- net LDR: now reaches R103.2, R75.1, U13.51 (PB12)
