File: kicad/main-phone/STM32G473.kicad_sch (KiCad schematic)
At the start: 32 parts, among them J7301 SPARE-IO (DNP), T1 NTCG164KF104FT1, U13 STM32G473VCT6, X1 ABM3-8_000MHZ-D2Y-T, X3 XKXEL89CII-SUAYLC-32_768K

Commit message: Per-board reference ranges, J1 spare header, IMU AD0 pull-down, BOM outputs
- reference ranges: main-phone 1-999, dock 1000s, front ToF 2000s, side 3000s,
  cliff 4000s, rear IR 5000s, Hall 6000s (main-phone 7xxx parts renumbered
  below 1000; sensor boards and dock moved from 8xxx)
- main-phone: J7301 -> J1, a fitted 2x7 0.1" header with spares only
  (3.3 V, 5 V, I2C4, UART PC10/PC11, PA8-PA10, PD4, PE2, PE6, GND)
- IMU: AP_AD0 pulled low by R217 (address 0x68); INT2 on test pad TP1;
  FSYNC reachable on R211; R18/R72 removed
- tools/export.py replaces export_pdfs.py: schematic PDF and JLC-style BOM in
  each board's output/ folder; --pcb adds Gerbers, placement and STEP
- cliff and rear IR projects: fix top-level sheet left over from a copy
- Hall board: visual tidy-up

Co-Authored-By: Claude Opus 5.5 <noreply@anthropic.com>
Parts:
- removed J7301: SPARE-IO (DNP), Connector_PinHeader_2.54mm:PinHeader_2x11_P2.54mm_Vertical, symbol Connector_Generic:Conn_02x11_Odd_Even
- added J1: SPARE-IO, Connector_PinHeader_2.54mm:PinHeader_2x07_P2.54mm_Vertical, symbol Connector_Generic:Conn_02x07_Odd_Even
- renumbered R7306 to R195, R7315 to R204
Connections:
- net GND: now also J1.13 (Pin_13), J1.14 (Pin_14)
- net I2C4_SCL: now also J1.3 (Pin_3)
- net I2C4_SDA: now also J1.4 (Pin_4)
- net SPARE-PA10: now also J1.7 (Pin_7)
- net SPARE-PA8: now also J1.9 (Pin_9)
- net SPARE-PA9: now also J1.10 (Pin_10)
- net SPARE-PC10-TX: now also J1.5 (Pin_5)
- net SPARE-PC11-RX: now also J1.6 (Pin_6)
- net SPARE-PD4: now also J1.11 (Pin_11)
- net SPARE-PE2: now also J1.12 (Pin_12)
- net SPARE-PE6: now also J1.8 (Pin_8)
- net VCC-3V3-REG: now also J1.1 (Pin_1)
- net VCC-5V-REG: now also J1.2 (Pin_2)
Other:
- note added: "J1 spare I/O: 0.1in 2x7 header (fitted). 1 VCC-3V3-REG (sensor rail), 2 VCC-5V-REG, 13/14 GND. 3/4 I2C4 SCL/SDA (shared with the ToF, side sensor and IMU; 2.2k pull-ups). 5/6 UART PC10 TX / PC11 RX (UART4 or USART3). 7 PA10, 8 PE6, 9 PA8, 10 PA9 (10k pull-up), 11 PD4, 12 PE2. IMU AD0/INT2/FSYNC are test pads on the IMU sheet. SWO (PB3) on JTAG1 is a spare when not tracing."
- note added: "R204: PA9 = UCPD DBCC1. High during reset turns on the dead-battery Rd on CC1 (PB6)."
- note removed: "J7301 spare I/O: 0.1in 2x11 pads, do not fit (zero height). 1 VCC-3V3-REG (sensor rail), 2 VCC-5V-REG, 21/22 GND. 3/4 I2C4 SCL/SDA (shared with the ToF, side sensor and IMU; 2.2k pull-ups). 5/6 UART PC10 TX / PC11 RX (UART4 or USART3). 7-18 spare GPIO, except 9/17 rear IR R/L, 10/11 Hall bin/tower, 12/13 cliff LM/RM. 19/20 IMU FSYNC/INT2 (FSYNC: 100k pull-down on the IMU sheet). SWO (PB3) on JTAG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"
- note removed: "R7315: PA9 = UCPD DBCC1. High during reset turns on the dead-battery Rd on CC1 (PB6)."
