File: kicad/main-phone/WHEEL-MOTORs .kicad_sch (KiCad schematic)
At the start: 20 parts, among them U14 DRV8870DDAR, U15 DRV8870DDAR

Commit message: LiDAR header, shunt, holes, Hall connector, INT pullup fix
Parts:
- R15, R65: value RL12FTNR250 -> RLH12FTCR250; footprint JLCImport:RL12FTNR250 -> Resistor_SMD:R_1206_3216Metric; LCSC C160921 -> C22464902; Manufacturer Part RL12FTNR250 -> RLH12FTCR250
Changed lines of the file:
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@@
 			)
 		)
-		(property "Value" "RL12FTNR250"
+		(property "Value" "RLH12FTCR250"
 			(at 127 62.2299 90)
 			(show_name no)
@@
 			)
 		)
-		(property "Footprint" "JLCImport:RL12FTNR250"
+		(property "Footprint" "Resistor_SMD:R_1206_3216Metric"
 			(at 125.095 60.96 0)
 			(hide yes)
@@
 			)
 		)
-		(property "Datasheet" "https://www.lcsc.com/datasheet/lcsc_datasheet_2304140030_TA-I-Tech-RL12FTNR250_C160921.pdf"
+		(property "Datasheet" "https://www.lcsc.com/product-detail/C22464902.html"
 			(at 125.095 60.96 0)
 			(hide yes)
@@
 			)
 		)
-		(property "Description" "250mΩ 500mW Metal Film Resistor SMD ±1% ±200ppm/℃ 1206 Current Sense Resistors / Shunt Resistors ROHS"
+		(property "Description" "250mOhm 1W current sense resistor, 1206, 1%, 100ppm/C"
 			(at 125.095 60.96 0)
 			(hide yes)
@@
 			)
 		)
-		(property "LCSC" "C160921"
+		(property "LCSC" "C22464902"
 			(at 125.095 60.96 0)
 			(hide yes)
@@
 			)
 		)
-		(property "Manufacturer Part" "RL12FTNR250"
+		(property "Manufacturer Part" "RLH12FTCR250"
 			(at 125.095 60.96 0)
 			(hide yes)
@@
 			)
 		)
-		(property "Value" "RL12FTNR250"
+		(property "Value" "RLH12FTCR250"
 			(at 129.54 148.5899 90)
 			(show_name no)
@@
 			)
 		)
-		(property "Footprint" "JLCImport:RL12FTNR250"
+		(property "Footprint" "Resistor_SMD:R_1206_3216Metric"
 			(at 127.635 147.32 0)
 			(hide yes)
@@
 			)
 		)
-		(property "Datasheet" "https://www.lcsc.com/datasheet/lcsc_datasheet_2304140030_TA-I-Tech-RL12FTNR250_C160921.pdf"
+		(property "Datasheet" "https://www.lcsc.com/product-detail/C22464902.html"
 			(at 127.635 147.32 0)
 			(hide yes)
@@
 			)
 		)
-		(property "Description" "250mΩ 500mW Metal Film Resistor SMD ±1% ±200ppm/℃ 1206 Current Sense Resistors / Shunt Resistors ROHS"
+		(property "Description" "250mOhm 1W current sense resistor, 1206, 1%, 100ppm/C"
 			(at 127.635 147.32 0)
 			(hide yes)
@@
 			)
 		)
-		(property "LCSC" "C160921"
+		(property "LCSC" "C22464902"
 			(at 127.635 147.32 0)
 			(hide yes)
@@
 			)
 		)
-		(property "Manufacturer Part" "RL12FTNR250"
+		(property "Manufacturer Part" "RLH12FTCR250"
 			(at 127.635 147.32 0)
 			(hide yes)
