File: kicad/main-phone/Battery-Charger.kicad_sch (KiCad schematic)
At the start: 49 parts, among them Q12 AOD407_C6396162, Q14 AOD407_C6396162, Q7101 AO3401, Q7102 AO3400, Q7303 AO3400, U1 SLM6900, U2 TMI6240

Commit message: main-phone: VBUS lockout, 2x6 spare I/O header
- VBUS lockout (Q7305, Q7306, R7312-R7314): PWR_EN reaches the TMI6240
  and Q7102 as PWR_EN_G, held low while VBUS is present, latched once on.
  The robot can no longer drive VBUS against a phone that sources it.
- spare I/O pads J7301: 2x7 -> 2x6 (PB15 is now DC_IN sense)

Co-Authored-By: Claude Opus 5.5 (1M context) <noreply@anthropic.com>
Parts:
- added Q7305, Q7306: AO3400, JLCImport:AO3400, symbol JLCImport:AO3400
- added R7312: 10k, Resistor_SMD:R_0603_1608Metric, symbol Device:R_US
- added R7313, R7314: 100k, Resistor_SMD:R_0603_1608Metric, symbol Device:R_US
Connections:
- net GND: now also Q7305.2 (S), Q7306.2 (S), R7314.2
- net PWR_EN: now also R7312.1; no longer Q7102.1 (G), R41.1, U2.3 (EN)
- net VBUS: now also R7313.1
- new net: Q7305.1 (G), Q7306.3 (D), R7313.2, R7314.1
- new net PWR_EN_G: Q7102.1 (G), Q7305.3 (D), Q7306.1 (G), R41.1, R7312.2, U2.3 (EN)
Other:
- note added: "VBUS lockout: the robot 5 V (TMI6240 + Q7101) can only turn on while VBUS is ~0 V. Q7305 holds PWR_EN_G low if a phone already sources VBUS; once on, Q7306 latches it."

Commit message: Per-board reference ranges, J1 spare header, IMU AD0 pull-down, BOM outputs
- reference ranges: main-phone 1-999, dock 1000s, front ToF 2000s, side 3000s,
  cliff 4000s, rear IR 5000s, Hall 6000s (main-phone 7xxx parts renumbered
  below 1000; sensor boards and dock moved from 8xxx)
- main-phone: J7301 -> J1, a fitted 2x7 0.1" header with spares only
  (3.3 V, 5 V, I2C4, UART PC10/PC11, PA8-PA10, PD4, PE2, PE6, GND)
- IMU: AP_AD0 pulled low by R217 (address 0x68); INT2 on test pad TP1;
  FSYNC reachable on R211; R18/R72 removed
- tools/export.py replaces export_pdfs.py: schematic PDF and JLC-style BOM in
  each board's output/ folder; --pcb adds Gerbers, placement and STEP
- cliff and rear IR projects: fix top-level sheet left over from a copy
- Hall board: visual tidy-up

Co-Authored-By: Claude Opus 5.5 <noreply@anthropic.com>
Parts:
- renumbered C7304 to C175, D7101 to D40, D7301 to D41, Q7101 to Q27, Q7102 to Q28, Q7303 to Q31, Q7305 to Q33, Q7306 to Q34, R7101 to R187, R7102 to R188, R7103 to R189, R7305 to R194, R7310 to R199, R7311 to R200, R7312 to R201, R7313 to R202, R7314 to R203
Other:
- note added: "DC_IN: 20 V brick or dock. With the battery disconnected (Q14 off) BAT-VCC = DC_IN - 0.4 V, so the SLM6900 (95% max duty) needs >= ~18.5 V to finish a 4S charge. Keep DC_IN <= 22 V (D41, Q13 Vgs)."
- note added: "Rail-hold: charger power (dock or barrel jack) turns the MCU rail on and keeps it on. DC_IN to GND ~130k (R175+R194 || R199+R200) = dock presence signature."
- note added: "USB-C (phone): phone is the USB host. CC1/CC2 go to the STM32 UCPD (PB6/PB4): Rd by default, PD power-role swap lets the robot charge the phone while it stays host. Q27 blocks the phone's VBUS from back-feeding the robot 5 V (the TMI6240 body diode conducts VOUT->VIN); PWR_EN turns on TMI6240 and Q27 together. TMI6240 now runs from VCC-5V-REG (U25 buck removed)."
- note added: "VBUS lockout: the robot 5 V (TMI6240 + Q27) can only turn on while VBUS is ~0 V. Q33 holds PWR_EN_G low if a phone already sources VBUS; once on, Q34 latches it."
- note removed: "DC_IN: 20 V brick or dock. With the battery disconnected (Q14 off) BAT-VCC = DC_IN - 0.4 V, so the SLM6900 (95% max duty) needs >= ~18.5 V to finish a 4S charge. Keep DC_IN <= 22 V (D7301, Q13 Vgs)."
- note removed: "Rail-hold: charger power (dock or barrel jack) turns the MCU rail on and keeps it on. DC_IN to GND ~130k (R175+R7305 || R7310+R7311) = dock presence signature."
- note removed: "USB-C (phone): phone is the USB host. CC1/CC2 go to the STM32 UCPD (PB6/PB4): Rd by default, PD power-role swap lets the robot charge the phone while it stays host. Q7101 blocks the phone's VBUS from back-feeding the robot 5 V (the TMI6240 body diode conducts VOUT->VIN); PWR_EN turns on TMI6240 and Q7101 together. TMI6240 now runs from VCC-5V-REG (U25 buck removed)."
- note removed: "VBUS lockout: the robot 5 V (TMI6240 + Q7101) can only turn on while VBUS is ~0 V. Q7305 holds PWR_EN_G low if a phone already sources VBUS; once on, Q7306 latches it."
Changed lines of the file:
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@@
 		)
 	)
-	(text "USB-C (phone): phone is the USB host. CC1/CC2 go to the STM32 UCPD (PB6/PB4): Rd by default,\nPD power-role swap lets the robot charge the phone while it stays host. Q7101 blocks the phone's\nVBUS from back-feeding the robot 5 V (the TMI6240 body diode conducts VOUT->VIN); PWR_EN turns\non TMI6240 and Q7101 together. TMI6240 now runs from VCC-5V-REG (U25 buck removed)."
+	(text "USB-C (phone): phone is the USB host. CC1/CC2 go to the STM32 UCPD (PB6/PB4): Rd by default,\nPD power-role swap lets the robot charge the phone while it stays host. Q27 blocks the phone's\nVBUS from back-feeding the robot 5 V (the TMI6240 body diode conducts VOUT->VIN); PWR_EN turns\non TMI6240 and Q27 together. TMI6240 now runs from VCC-5V-REG (U25 buck removed)."
 		(exclude_from_sim no)
 		(at 300.99 60.96 0)
@@
 			)
 		)
-		(property "Description" "Rail-hold divider top (with R7305); with the DC_IN sense divider, ~130k to GND is the dock presence signature"
+		(property "Description" "Rail-hold divider top (with R194); with the DC_IN sense divider, ~130k to GND is the dock presence signature"
 			(at 316.865 314.325 0)
 			(hide yes)
@@
 		(in_pos_files yes)
 		(dnp no)
-		(property "Reference" "Q7101"
+		(property "Reference" "Q27"
 			(at 327.66 68.58 0)
 			(show_name no)
@@
 			(project "Main"
 				(path "/dbcfb655-8d45-4808-9a74-2a0eb03372e8/ef1147df-ce85-4822-98ae-5614ce438d97"
-					(reference "Q7101")
+					(reference "Q27")
 					(unit 1)
 				)
@@
 		(dnp no)
 		(fields_autoplaced yes)
-		(property "Reference" "R7103"
+		(property "Reference" "R189"
 			(at 347.472 86.3599 0)
 			(show_name no)
@@
 			(project "Main"
 				(path "/dbcfb655-8d45-4808-9a74-2a0eb03372e8/ef1147df-ce85-4822-98ae-5614ce438d97"
-					(reference "R7103")
+					(reference "R189")
 					(unit 1)
 				)
@@
 		(dnp no)
 		(fields_autoplaced yes)
-		(property "Reference" "R7102"
+		(property "Reference" "R188"
 			(at 347.472 78.7399 0)
 			(show_name no)
@@
 			(project "Main"
 				(path "/dbcfb655-8d45-4808-9a74-2a0eb03372e8/ef1147df-ce85-4822-98ae-5614ce438d97"
-					(reference "R7102")
+					(reference "R188")
 					(unit 1)
 				)
@@
 		(dnp no)
 		(fields_autoplaced yes)
-		(property "Reference" "R7101"
+		(property "Reference" "R187"
 			(at 341.122 76.1999 0)
 			(show_name no)
@@
 			)
 		)
-		(property "Description" "Q7101 gate-source pull-up: robot 5 V stays off the USB-C VBUS unless PWR_EN is high"
+		(property "Description" "Q27 gate-source pull-up: robot 5 V stays off the USB-C VBUS unless PWR_EN is high"
 			(at 339.09 77.47 0)
 			(hide yes)
@@
 			(project "Main"
 				(path "/dbcfb655-8d45-4808-9a74-2a0eb03372e8/ef1147df-ce85-4822-98ae-5614ce438d97"
-					(reference "R7101")
+					(reference "R187")
 					(unit 1)
 				)
@@
 		(in_pos_files yes)
 		(dnp no)
-		(property "Reference" "Q7102"
+		(property "Reference" "Q28"
 			(at 332.74 86.995 0)
 			(show_name no)
@@
 			(project "Main"
 				(path "/dbcfb655-8d45-4808-9a74-2a0eb03372e8/ef1147df-ce85-4822-98ae-5614ce438d97"
-					(reference "Q7102")
+					(reference "Q28")
 					(unit 1)
 				)
@@
 		(in_pos_files yes)
 		(dnp no)
-		(property "Reference" "D7101"
+		(property "Reference" "D40"
 			(at 374.65 169.545 90)
 			(show_name no)
@@
 			(project "Main"
 				(path "/dbcfb655-8d45-4808-9a74-2a0eb03372e8/ef1147df-ce85-4822-98ae-5614ce438d97"
-					(reference "D7101")
+					(reference "D40")
 					(unit 1)
 				)
@@
 		(in_pos_files yes)
 		(dnp no)
-		(property "Reference" "R7305"
+		(property "Reference" "R194"
 			(at 328.93 316.865 0)
 			(show_name no)
@@
 			(project "Main"
 				(path "/dbcfb655-8d45-4808-9a74-2a0eb03372e8/ef1147df-ce85-4822-98ae-5614ce438d97"
-					(reference "R7305")
+					(reference "R194")
 					(unit 1)
 				)
@@
 		(in_pos_files yes)
 		(dnp no)
-		(property "Reference" "Q7303"
+		(property "Reference" "Q31"
 			(at 339.09 313.055 0)
 			(show_name no)
@@
 			(project "Main"
 				(path "/dbcfb655-8d45-4808-9a74-2a0eb03372e8/ef1147df-ce85-4822-98ae-5614ce438d97"
-					(reference "Q7303")
+					(reference "Q31")
 					(unit 1)
 				)
@@
 		)
 	)
-	(text "Rail-hold: charger power (dock or barrel jack)\nturns the MCU rail on and keeps it on.\nDC_IN to GND ~130k (R175+R7305 || R7310+R7311)\n= dock presence signature."
+	(text "Rail-hold: charger power (dock or barrel jack)\nturns the MCU rail on and keeps it on.\nDC_IN to GND ~130k (R175+R194 || R199+R200)\n= dock presence signature."
 		(exclude_from_sim no)
 		(at 311.15 332.74 0)
@@
 		(in_pos_files yes)
 		(dnp no)
-		(property "Reference" "D7301"
+		(property "Reference" "D41"
 			(at 111.125 287.655 90)
 			(show_name no)
@@
 			(project "Main"
 				(path "/dbcfb655-8d45-4808-9a74-2a0eb03372e8/ef1147df-ce85-4822-98ae-5614ce438d97"
-					(reference "D7301")
+					(reference "D41")
 					(unit 1)
 				)
@@
 		)
 	)
-	(text "DC_IN: 20 V brick or dock. With the battery disconnected (Q14 off) BAT-VCC = DC_IN - 0.4 V,\nso the SLM6900 (95% max duty) needs >= ~18.5 V to finish a 4S charge. Keep DC_IN <= 22 V (D7301, Q13 Vgs)."
+	(text "DC_IN: 20 V brick or dock. With the battery disconnected (Q14 off) BAT-VCC = DC_IN - 0.4 V,\nso the SLM6900 (95% max duty) needs >= ~18.5 V to finish a 4S charge. Keep DC_IN <= 22 V (D41, Q13 Vgs)."
 		(exclude_from_sim no)
 		(at 63.5 276.86 0)
@@
 		(in_pos_files yes)
 		(dnp no)
-		(property "Reference" "R7310"
+		(property "Reference" "R199"
 			(at 69.85 304.165 0)
 			(show_name no)
@@
 			(project "Main"
 				(path "/dbcfb655-8d45-4808-9a74-2a0eb03372e8/ef1147df-ce85-4822-98ae-5614ce438d97"
-					(reference "R7310")
+					(reference "R199")
 					(unit 1)
 				)
@@
 		(in_pos_files yes)
 		(dnp no)
-		(property "Reference" "R7311"
+		(property "Reference" "R200"
 			(at 68.58 311.785 0)
 			(show_name no)
@@
 			(project "Main"
 				(path "/dbcfb655-8d45-4808-9a74-2a0eb03372e8/ef1147df-ce85-4822-98ae-5614ce438d97"
-					(reference "R7311")
+					(reference "R200")
 					(unit 1)
 				)
@@
 		(in_pos_files yes)
 		(dnp no)
-		(property "Reference" "C7304"
+		(property "Reference" "C175"
 			(at 85.725 313.055 0)
 			(show_name no)
@@
 			(project "Main"
 				(path "/dbcfb655-8d45-4808-9a74-2a0eb03372e8/ef1147df-ce85-4822-98ae-5614ce438d97"
-					(reference "C7304")
+					(reference "C175")
 					(unit 1)
 				)
@@
 		(in_pos_files yes)
 		(dnp no)
-		(property "Reference" "R7312"
+		(property "Reference" "R201"
 			(at 208.28 54.61 90)
 			(show_name no)
@@
 			)
 		)
-		(property "Description" "PWR_EN series: Q7305 can hold PWR_EN_G low against the MCU"
+		(property "Description" "PWR_EN series: Q33 can hold PWR_EN_G low against the MCU"
 			(at 208.28 58.42 0)
 			(hide yes)
@@
 			(project "Main"
 				(path "/dbcfb655-8d45-4808-9a74-2a0eb03372e8/ef1147df-ce85-4822-98ae-5614ce438d97"
-					(reference "R7312")
+					(reference "R201")
 					(unit 1)
 				)
@@
 		(in_pos_files yes)
 		(dnp no)
-		(property "Reference" "Q7305"
+		(property "Reference" "Q33"
 			(at 236.22 64.77 0)
 			(show_name no)
@@
 			(project "Main"
 				(path "/dbcfb655-8d45-4808-9a74-2a0eb03372e8/ef1147df-ce85-4822-98ae-5614ce438d97"
-					(reference "Q7305")
+					(reference "Q33")
 					(unit 1)
 				)
@@
 		(in_pos_files yes)
 		(dnp no)
-		(property "Reference" "R7313"
+		(property "Reference" "R202"
 			(at 194.31 62.23 90)
 			(show_name no)
@@
 			(project "Main"
 				(path "/dbcfb655-8d45-4808-9a74-2a0eb03372e8/ef1147df-ce85-4822-98ae-5614ce438d97"
-					(reference "R7313")
+					(reference "R202")
 					(unit 1)
 				)
@@
 		(in_pos_files yes)
 		(dnp no)
-		(property "Reference" "R7314"
+		(property "Reference" "R203"
 			(at 196.85 69.215 0)
 			(show_name no)
@@
 			(project "Main"
 				(path "/dbcfb655-8d45-4808-9a74-2a0eb03372e8/ef1147df-ce85-4822-98ae-5614ce438d97"
-					(reference "R7314")
+					(reference "R203")
 					(unit 1)
 				)
@@
 		(in_pos_files yes)
 		(dnp no)
-		(property "Reference" "Q7306"
+		(property "Reference" "Q34"
 			(at 218.44 69.85 0)
 			(show_name no)
@@
 			)
 		)
-		(property "Description" "VBUS lockout latch: once PWR_EN_G is on, keeps Q7305 off"
+		(property "Description" "VBUS lockout latch: once PWR_EN_G is on, keeps Q33 off"
 			(at 215.9 71.12 0)
 			(hide yes)
@@
 			(project "Main"
 				(path "/dbcfb655-8d45-4808-9a74-2a0eb03372e8/ef1147df-ce85-4822-98ae-5614ce438d97"
-					(reference "Q7306")
+					(reference "Q34")
 					(unit 1)
 				)
@@
 		)
 	)
-	(text "VBUS lockout: the robot 5 V (TMI6240 + Q7101) can only\nturn on while VBUS is ~0 V. Q7305 holds PWR_EN_G low if a\nphone already sources VBUS; once on, Q7306 latches it."
+	(text "VBUS lockout: the robot 5 V (TMI6240 + Q27) can only\nturn on while VBUS is ~0 V. Q33 holds PWR_EN_G low if a\nphone already sources VBUS; once on, Q34 latches it."
 		(exclude_from_sim no)
 		(at 238.76 80.01 0)
