File: kicad/main-phone/Carpet-sensor.kicad_sch (KiCad schematic)
At the start: 12 parts, among them Q18 AO3400

Commit message: Per-board reference ranges, J1 spare header, IMU AD0 pull-down, BOM outputs
- reference ranges: main-phone 1-999, dock 1000s, front ToF 2000s, side 3000s,
  cliff 4000s, rear IR 5000s, Hall 6000s (main-phone 7xxx parts renumbered
  below 1000; sensor boards and dock moved from 8xxx)
- main-phone: J7301 -> J1, a fitted 2x7 0.1" header with spares only
  (3.3 V, 5 V, I2C4, UART PC10/PC11, PA8-PA10, PD4, PE2, PE6, GND)
- IMU: AP_AD0 pulled low by R217 (address 0x68); INT2 on test pad TP1;
  FSYNC reachable on R211; R18/R72 removed
- tools/export.py replaces export_pdfs.py: schematic PDF and JLC-style BOM in
  each board's output/ folder; --pcb adds Gerbers, placement and STEP
- cliff and rear IR projects: fix top-level sheet left over from a copy
- Hall board: visual tidy-up

Co-Authored-By: Claude Opus 5.5 <noreply@anthropic.com>
Parts:
- renumbered C7303 to C174, R7011 to R185, R7012 to R186
Other:
- note added: "C174 AC-couples LO to the Q18 gate: if LO sticks high, the gate decays through R186 (~10 ms) and Q18 turns off, so R185 is never stressed by firmware holding LO high."
- note added: "Carpet driver: one low-side AO3400 + 330R pull-up from VUS (14.4 V). The P-FET half-bridge was removed: its 100k gate pull-up could not turn it off at 290 kHz (shoot-through). R186 holds LO low in reset/flash. Drive LO in short bursts only: LO stuck high puts 0.63 W into R185."
- note removed: "C7303 AC-couples LO to the Q18 gate: if LO sticks high, the gate decays through R7012 (~10 ms) and Q18 turns off, so R7011 is never stressed by firmware holding LO high."
- note removed: "Carpet driver: one low-side AO3400 + 330R pull-up from VUS (14.4 V). The P-FET half-bridge was removed: its 100k gate pull-up could not turn it off at 290 kHz (shoot-through). R7012 holds LO low in reset/flash. Drive LO in short bursts only: LO stuck high puts 0.63 W into R7011."
Changed lines of the file:
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@@
 	(generator_version "10.0")
 	(paper "USLetter")
-	(text "Carpet driver: one low-side AO3400 + 330R pull-up from VUS (14.4 V). The P-FET half-bridge was removed:\nits 100k gate pull-up could not turn it off at 290 kHz (shoot-through). R7012 holds LO low in reset/flash.\nDrive LO in short bursts only: LO stuck high puts 0.63 W into R7011."
+	(text "Carpet driver: one low-side AO3400 + 330R pull-up from VUS (14.4 V). The P-FET half-bridge was removed:\nits 100k gate pull-up could not turn it off at 290 kHz (shoot-through). R186 holds LO low in reset/flash.\nDrive LO in short bursts only: LO stuck high puts 0.63 W into R185."
 		(exclude_from_sim no)
 		(at 98.425 40.005 0)
@@
 		)
 	)
-	(text "C7303 AC-couples LO to the Q18 gate: if LO sticks high, the gate decays through R7012 (~10 ms)\nand Q18 turns off, so R7011 is never stressed by firmware holding LO high."
+	(text "C174 AC-couples LO to the Q18 gate: if LO sticks high, the gate decays through R186 (~10 ms)\nand Q18 turns off, so R185 is never stressed by firmware holding LO high."
 		(exclude_from_sim no)
 		(at 209.55 75.057 0)
@@
 		(in_pos_files yes)
 		(dnp no)
-		(property "Reference" "R7011"
+		(property "Reference" "R185"
 			(at 93.98 45.72 0)
 			(show_name no)
@@
 			(project "Main"
 				(path "/dbcfb655-8d45-4808-9a74-2a0eb03372e8/b8feb78a-8098-4bc8-81b4-34551e1a6113"
-					(reference "R7011")
+					(reference "R185")
 					(unit 1)
 				)
@@
 		(in_pos_files yes)
 		(dnp no)
-		(property "Reference" "R7012"
+		(property "Reference" "R186"
 			(at 78.74 80.645 0)
 			(show_name no)
@@
 			(project "Main"
 				(path "/dbcfb655-8d45-4808-9a74-2a0eb03372e8/b8feb78a-8098-4bc8-81b4-34551e1a6113"
-					(reference "R7012")
+					(reference "R186")
 					(unit 1)
 				)
@@
 		(in_pos_files yes)
 		(dnp no)
-		(property "Reference" "C7303"
+		(property "Reference" "C174"
 			(at 76.2 72.39 90)
 			(show_name no)
@@
 			(project "Main"
 				(path "/dbcfb655-8d45-4808-9a74-2a0eb03372e8/b8feb78a-8098-4bc8-81b4-34551e1a6113"
-					(reference "C7303")
+					(reference "C174")
 					(unit 1)
 				)
