File: kicad/main-phone/SYSTEM-POWER.kicad_sch (KiCad schematic)
At the start: 90 parts, among them Q1 AO4407C, Q13 AO4407C, Q16 AO3401, Q17 AO3401, Q19 AO3400, Q23 AO3400, Q7301 AO3400, Q7302 AO3400, U12 XRNR4030-10UH_M, U16 HT7533-1_C14289, U21 AP64501SP-13, U22 AP64501SP-13, U5 MT3608, U7301 74LVC1G17

Commit message: Charging dock rev 2; main-phone bucks AP64501 -> TPS54560B
Charging dock (kicad/charging-dock), redesigned:
- CH32V003F4P6 control (Arduino core, ch32fun, PlatformIO)
- robot detection: resistance-signature probe before DOCK+ goes live
- AO4407C soft-start output switch, 50 mOhm + INA180A1 current sense
- NEC IR beacon: two 3x TSAL6200 strings, AC-coupled gates
- 20 V input: DC-044A-20A, 5 A fuse, SMAJ22A, HT7533-1
- refs 8xxx for the one-panel plan; uses the shared ../main libraries
- removed the orphan sheets, the old local library copy and an unrelated PDF
- README with pin map, detection math, firmware rules, layout notes

main-phone: U21/U22 TPS54560B (AP64501 out of stock) with SS56 catch
diodes, 232k RT, 4.7k + 47nF compensation, U21 EN divider; BAT-VCC input
caps 10uF/50V 1206. SPEC and READMEs updated.

Co-Authored-By: Claude Opus 5.5 (1M context) <noreply@anthropic.com>
Parts:
- removed C107, C118: 100nF/50V, Capacitor_SMD:C_0603_1608Metric, symbol Library:C_0603
- added D7401, D7402: SS56, JLCImport:SS56, symbol JLCImport:SS56
- added R7401, R7402: 232k, Resistor_SMD:R_0603_1608Metric, symbol Device:R_US
- added R7403: 100k, Resistor_SMD:R_0603_1608Metric, symbol Device:R_US
- added R7404: 22.1k, Resistor_SMD:R_0603_1608Metric, symbol Device:R_US
- C106, C115, C116, C95: value 10uF/25V -> 10uF/50V; footprint Capacitor_SMD:C_0603_1608Metric -> Capacitor_SMD:C_1206_3216Metric; LCSC C96446 -> C13585
- C112, C120: value 1.2nF/50V -> 47nF/50V; LCSC C107073 -> C1622
- R143: value 12k -> 4.7k; LCSC C2930069 -> C2907034
- R147: value 20k -> 4.7k; LCSC C2907011 -> C2907034
- U21, U22: value AP64501SP-13 -> TPS54560BDDAR; footprint JLCImport:AP64501SP-13 -> Package_SO:Texas_R-PDSO-G8_EP2.95x4.9mm_Mask2.4x3.1mm_ThermalVias; symbol JLCImport:AP64501SP-13 -> JLCImport:TPS54560BDDAR; LCSC C2071517 -> C1850354
Connections:
- net GND: now also D7401.2 (A), D7402.2 (A), R7401.2, R7402.2, R7404.2
- net POWER-EN: now also R7403.1; no longer U21.3 (EN)
- net at U22.4 (RT/CLK): now also R7402.1
- net at L2.1, R141.2, U21.8 (SW): now also D7401.1 (K)
- net at U21.4 (RT/CLK): now also R7401.1
- net at L3.1, R146.2, U22.8 (SW): now also D7402.1 (K)
- new net: R7403.2, R7404.1, U21.3 (EN)
Other:
- note added: "TPS54560B (U21, U22): non-synchronous, SS56 catch diode; fsw 418 kHz (RT 232k); COMP 4.7k + 47nF (all-ceramic Cout, no pole cap). EN abs max 8.4 V: R7403/R7404 on U21."

Commit message: Per-board reference ranges, J1 spare header, IMU AD0 pull-down, BOM outputs
- reference ranges: main-phone 1-999, dock 1000s, front ToF 2000s, side 3000s,
  cliff 4000s, rear IR 5000s, Hall 6000s (main-phone 7xxx parts renumbered
  below 1000; sensor boards and dock moved from 8xxx)
- main-phone: J7301 -> J1, a fitted 2x7 0.1" header with spares only
  (3.3 V, 5 V, I2C4, UART PC10/PC11, PA8-PA10, PD4, PE2, PE6, GND)
- IMU: AP_AD0 pulled low by R217 (address 0x68); INT2 on test pad TP1;
  FSYNC reachable on R211; R18/R72 removed
- tools/export.py replaces export_pdfs.py: schematic PDF and JLC-style BOM in
  each board's output/ folder; --pcb adds Gerbers, placement and STEP
- cliff and rear IR projects: fix top-level sheet left over from a copy
- Hall board: visual tidy-up

Co-Authored-By: Claude Opus 5.5 <noreply@anthropic.com>
Parts:
- renumbered C7301 to C172, C7302 to C173, D7401 to D42, D7402 to D43, Q7301 to Q29, Q7302 to Q30, R7010 to R184, R7301 to R190, R7302 to R191, R7303 to R192, R7304 to R193, R7401 to R205, R7402 to R206, R7403 to R207, R7404 to R208, U7301 to U23
Other:
- note added: "Hardware off timer: holding the power button for ~4-9 s turns the MCU rail off even if the firmware hangs (Q29 releases C172, U23 trips, Q30 pulls PWR-LATCH low). Firmware turns off at 3 s. While charging, the rail-hold (Q31 on BATTERY-CHARGER, from DC_IN) keeps the MCU rail on regardless, and charger power alone turns the MCU rail on (Q31 pulls PWR-SW-G low)."
- note added: "TPS54560B (U21, U22): non-synchronous, SS56 catch diode; fsw 418 kHz (RT 232k); COMP 4.7k + 47nF (all-ceramic Cout, no pole cap). EN abs max 8.4 V: R207/R208 on U21."
- note added: "VM-VBAT (motors, fan) is on only while WD_OK is high (RC watchdog fed) AND ~{VM-VBAT-EN} is low. Q19 source-switched AND: GPIO low = on. R184 keeps it off in reset/flash. AO4407C: Vgs +/-25 V, no gate divider needed."
- note removed: "Hardware off timer: holding the power button for ~4-9 s turns the MCU rail off even if the firmware hangs (Q7301 releases C7301, U7301 trips, Q7302 pulls PWR-LATCH low). Firmware turns off at 3 s. While charging, the rail-hold (Q7303 on BATTERY-CHARGER, from DC_IN) keeps the MCU rail on regardless, and charger power alone turns the MCU rail on (Q7303 pulls PWR-SW-G low)."
- note removed: "TPS54560B (U21, U22): non-synchronous, SS56 catch diode; fsw 418 kHz (RT 232k); COMP 4.7k + 47nF (all-ceramic Cout, no pole cap). EN abs max 8.4 V: R7403/R7404 on U21."
- note removed: "VM-VBAT (motors, fan) is on only while WD_OK is high (RC watchdog fed) AND ~{VM-VBAT-EN} is low. Q19 source-switched AND: GPIO low = on. R7010 keeps it off in reset/flash. AO4407C: Vgs +/-25 V, no gate divider needed."
Changed lines of the file:
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@@
 		)
 	)
-	(text "VM-VBAT (motors, fan) is on only while WD_OK is high (RC watchdog fed) AND ~{VM-VBAT-EN} is low.\nQ19 source-switched AND: GPIO low = on. R7010 keeps it off in reset/flash. AO4407C: Vgs +/-25 V, no gate divider needed."
+	(text "VM-VBAT (motors, fan) is on only while WD_OK is high (RC watchdog fed) AND ~{VM-VBAT-EN} is low.\nQ19 source-switched AND: GPIO low = on. R184 keeps it off in reset/flash. AO4407C: Vgs +/-25 V, no gate divider needed."
 		(exclude_from_sim no)
 		(at 283.21 182.88 0)
@@
 		(in_pos_files yes)
 		(dnp no)
-		(property "Reference" "R7010"
+		(property "Reference" "R184"
 			(at 311.15 156.21 0)
 			(show_name no)
@@
 			(project "Main"
 				(path "/dbcfb655-8d45-4808-9a74-2a0eb03372e8/35c833ed-33c3-4a72-8fc9-e035e67a6b75"
-					(reference "R7010")
+					(reference "R184")
 					(unit 1)
 				)
@@
 		(in_pos_files yes)
 		(dnp no)
-		(property "Reference" "R7301"
+		(property "Reference" "R190"
 			(at 386.08 338.455 90)
 			(show_name no)
@@
 			)
 		)
-		(property "Description" "PA15 series: lets Q7302 (5 s off timer) override a high PA15"
+		(property "Description" "PA15 series: lets Q30 (5 s off timer) override a high PA15"
 			(at 381.635 341.63 0)
 			(hide yes)
@@
 			(project "Main"
 				(path "/dbcfb655-8d45-4808-9a74-2a0eb03372e8/35c833ed-33c3-4a72-8fc9-e035e67a6b75"
-					(reference "R7301")
+					(reference "R190")
 					(unit 1)
 				)
@@
 		(in_pos_files yes)
 		(dnp no)
-		(property "Reference" "R7302"
+		(property "Reference" "R191"
 			(at 445.77 360.68 0)
 			(show_name no)
@@
 			)
 		)
-		(property "Description" "Power button divider: Q7301 on while the button is up"
+		(property "Description" "Power button divider: Q29 on while the button is up"
 			(at 443.23 361.95 0)
 			(hide yes)
@@
 			(project "Main"
 				(path "/dbcfb655-8d45-4808-9a74-2a0eb03372e8/35c833ed-33c3-4a72-8fc9-e035e67a6b75"
-					(reference "R7302")
+					(reference "R191")
 					(unit 1)
 				)
@@
 		(in_pos_files yes)
 		(dnp no)
-		(property "Reference" "R7303"
+		(property "Reference" "R192"
 			(at 445.77 368.3 0)
 			(show_name no)
@@
 			(project "Main"
 				(path "/dbcfb655-8d45-4808-9a74-2a0eb03372e8/35c833ed-33c3-4a72-8fc9-e035e67a6b75"
-					(reference "R7303")
+					(reference "R192")
 					(unit 1)
 				)
@@
 		(in_pos_files yes)
 		(dnp no)
-		(property "Reference" "Q7301"
+		(property "Reference" "Q29"
 			(at 458.47 364.49 0)
 			(show_name no)
@@
 			(project "Main"
 				(path "/dbcfb655-8d45-4808-9a74-2a0eb03372e8/35c833ed-33c3-4a72-8fc9-e035e67a6b75"
-					(reference "Q7301")
+					(reference "Q29")
 					(unit 1)
 				)
@@
 		(in_pos_files yes)
 		(dnp no)
-		(property "Reference" "R7304"
+		(property "Reference" "R193"
 			(at 458.47 350.52 0)
 			(show_name no)
@@
 			(project "Main"
 				(path "/dbcfb655-8d45-4808-9a74-2a0eb03372e8/35c833ed-33c3-4a72-8fc9-e035e67a6b75"
-					(reference "R7304")
+					(reference "R193")
 					(unit 1)
 				)
@@
 		(in_pos_files yes)
 		(dnp no)
-		(property "Reference" "C7301"
+		(property "Reference" "C172"
 			(at 466.09 358.14 0)
 			(show_name no)
@@
 			(project "Main"
 				(path "/dbcfb655-8d45-4808-9a74-2a0eb03372e8/35c833ed-33c3-4a72-8fc9-e035e67a6b75"
-					(reference "C7301")
+					(reference "C172")
 					(unit 1)
 				)
@@
 		(in_pos_files yes)
 		(dnp no)
-		(property "Reference" "U7301"
+		(property "Reference" "U23"
 			(at 484.505 369.57 0)
 			(show_name no)
@@
 			(project "Main"
 				(path "/dbcfb655-8d45-4808-9a74-2a0eb03372e8/35c833ed-33c3-4a72-8fc9-e035e67a6b75"
-					(reference "U7301")
+					(reference "U23")
 					(unit 1)
 				)
@@
 		(in_pos_files yes)
 		(dnp no)
-		(property "Reference" "C7302"
+		(property "Reference" "C173"
 			(at 498.475 343.535 0)
 			(show_name no)
@@
 			(project "Main"
 				(path "/dbcfb655-8d45-4808-9a74-2a0eb03372e8/35c833ed-33c3-4a72-8fc9-e035e67a6b75"
-					(reference "C7302")
+					(reference "C173")
 					(unit 1)
 				)
@@
 		(in_pos_files yes)
 		(dnp no)
-		(property "Reference" "Q7302"
+		(property "Reference" "Q30"
 			(at 509.27 354.33 0)
 			(show_name no)
@@
 			(project "Main"
 				(path "/dbcfb655-8d45-4808-9a74-2a0eb03372e8/35c833ed-33c3-4a72-8fc9-e035e67a6b75"
-					(reference "Q7302")
+					(reference "Q30")
 					(unit 1)
 				)
@@
 		)
 	)
-	(text "Hardware off timer: holding the power button for ~4-9 s turns the MCU rail off even if the firmware hangs\n(Q7301 releases C7301, U7301 trips, Q7302 pulls PWR-LATCH low). Firmware turns off at 3 s.\nWhile charging, the rail-hold (Q7303 on BATTERY-CHARGER, from DC_IN) keeps the MCU rail on regardless,\nand charger power alone turns the MCU rail on (Q7303 pulls PWR-SW-G low)."
+	(text "Hardware off timer: holding the power button for ~4-9 s turns the MCU rail off even if the firmware hangs\n(Q29 releases C172, U23 trips, Q30 pulls PWR-LATCH low). Firmware turns off at 3 s.\nWhile charging, the rail-hold (Q31 on BATTERY-CHARGER, from DC_IN) keeps the MCU rail on regardless,\nand charger power alone turns the MCU rail on (Q31 pulls PWR-SW-G low)."
 		(exclude_from_sim no)
 		(at 434.34 389.89 0)
@@
 		(in_pos_files yes)
 		(dnp no)
-		(property "Reference" "R7401"
+		(property "Reference" "R205"
 			(at 72.39 293.37 0)
 			(show_name no)
@@
 			(project "Main"
 				(path "/dbcfb655-8d45-4808-9a74-2a0eb03372e8/35c833ed-33c3-4a72-8fc9-e035e67a6b75"
-					(reference "R7401")
+					(reference "R205")
 					(unit 1)
 				)
@@
 		(in_pos_files yes)
 		(dnp no)
-		(property "Reference" "R7402"
+		(property "Reference" "R206"
 			(at 57.785 117.475 0)
 			(show_name no)
@@
 			(project "Main"
 				(path "/dbcfb655-8d45-4808-9a74-2a0eb03372e8/35c833ed-33c3-4a72-8fc9-e035e67a6b75"
-					(reference "R7402")
+					(reference "R206")
 					(unit 1)
 				)
@@
 		(in_pos_files yes)
 		(dnp no)
-		(property "Reference" "D7401"
+		(property "Reference" "D42"
 			(at 135.255 280.035 90)
 			(show_name no)
@@
 			(project "Main"
 				(path "/dbcfb655-8d45-4808-9a74-2a0eb03372e8/35c833ed-33c3-4a72-8fc9-e035e67a6b75"
-					(reference "D7401")
+					(reference "D42")
 					(unit 1)
 				)
@@
 		(in_pos_files yes)
 		(dnp no)
-		(property "Reference" "D7402"
+		(property "Reference" "D43"
 			(at 135.255 104.14 90)
 			(show_name no)
@@
 			(project "Main"
 				(path "/dbcfb655-8d45-4808-9a74-2a0eb03372e8/35c833ed-33c3-4a72-8fc9-e035e67a6b75"
-					(reference "D7402")
+					(reference "D43")
 					(unit 1)
 				)
@@
 		(in_pos_files yes)
 		(dnp no)
-		(property "Reference" "R7403"
+		(property "Reference" "R207"
 			(at 27.94 276.86 90)
 			(show_name no)
@@
 			(project "Main"
 				(path "/dbcfb655-8d45-4808-9a74-2a0eb03372e8/35c833ed-33c3-4a72-8fc9-e035e67a6b75"
-					(reference "R7403")
+					(reference "R207")
 					(unit 1)
 				)
@@
 		(in_pos_files yes)
 		(dnp no)
-		(property "Reference" "R7404"
+		(property "Reference" "R208"
 			(at 38.735 284.48 0)
 			(show_name no)
@@
 			(project "Main"
 				(path "/dbcfb655-8d45-4808-9a74-2a0eb03372e8/35c833ed-33c3-4a72-8fc9-e035e67a6b75"
-					(reference "R7404")
+					(reference "R208")
 					(unit 1)
 				)
@@
 		)
 	)
-	(text "TPS54560B (U21, U22): non-synchronous,\nSS56 catch diode; fsw 418 kHz (RT 232k);\nCOMP 4.7k + 47nF (all-ceramic Cout, no pole cap).\nEN abs max 8.4 V: R7403/R7404 on U21."
+	(text "TPS54560B (U21, U22): non-synchronous,\nSS56 catch diode; fsw 418 kHz (RT 232k);\nCOMP 4.7k + 47nF (all-ceramic Cout, no pole cap).\nEN abs max 8.4 V: R207/R208 on U21."
 		(exclude_from_sim no)
 		(at 15.24 250.19 0)
