File: kicad/main-phone/WATCHDOG.kicad_sch (KiCad schematic)
At the start: 7 parts, among them Q7001 AO3401

Commit message: Per-board reference ranges, J1 spare header, IMU AD0 pull-down, BOM outputs
- reference ranges: main-phone 1-999, dock 1000s, front ToF 2000s, side 3000s,
  cliff 4000s, rear IR 5000s, Hall 6000s (main-phone 7xxx parts renumbered
  below 1000; sensor boards and dock moved from 8xxx)
- main-phone: J7301 -> J1, a fitted 2x7 0.1" header with spares only
  (3.3 V, 5 V, I2C4, UART PC10/PC11, PA8-PA10, PD4, PE2, PE6, GND)
- IMU: AP_AD0 pulled low by R217 (address 0x68); INT2 on test pad TP1;
  FSYNC reachable on R211; R18/R72 removed
- tools/export.py replaces export_pdfs.py: schematic PDF and JLC-style BOM in
  each board's output/ folder; --pcb adds Gerbers, placement and STEP
- cliff and rear IR projects: fix top-level sheet left over from a copy
- Hall board: visual tidy-up

Co-Authored-By: Claude Opus 5.5 <noreply@anthropic.com>
Parts:
- renumbered C7001 to C169, C7002 to C170, Q7001 to Q24, R7001 to R176, R7002 to R177, R7003 to R178, R7004 to R179
Other:
- note added: "Firmware toggles WDI in software (50-1000 Hz, ~50% duty) only while the control loop is healthy. Never drive WDI from a timer/PWM: a timer keeps running after the CPU hangs. Each falling edge on WDI pulls the Q24 gate low through C169 and tops up C170 via R178. WD_OK ~2.7 V while toggling. WDI stuck high, low or floating: <1 V in ~100 ms, <0.4 V in ~190 ms (10 uF nominal; DC-bias derating shorten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"
- note removed: "Firmware toggles WDI in software (50-1000 Hz, ~50% duty) only while the control loop is healthy. Never drive WDI from a timer/PWM: a timer keeps running after the CPU hangs. Each falling edge on WDI pulls the Q7001 gate low through C7001 and tops up C7002 via R7003. WD_OK ~2.7 V while toggling. WDI stuck high, low or floating: <1 V in ~100 ms, <0.4 V in ~190 ms (10 uF nominal; DC-bias derating sh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"
Changed lines of the file:
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@@
 		)
 	)
-	(text "Firmware toggles WDI in software (50-1000 Hz, ~50% duty) only while the control loop is healthy.\nNever drive WDI from a timer/PWM: a timer keeps running after the CPU hangs.\nEach falling edge on WDI pulls the Q7001 gate low through C7001 and tops up C7002 via R7003.\nWD_OK ~2.7 V while toggling. WDI stuck high, low or floating: <1 V in ~100 ms, <0.4 V in ~190 ms\n(10 uF nominal; DC-bias derating shortens this). WD_OK starts at 0 V at power-up (fail-safe).\nWD_OK drives N-FET gates only (14.4 V rail switch, water pump, LiDAR incl. laser): no resistive loads.\nWDI pin: high-Z at reset, no pull-down. All parts reuse existing BOM lines."
+	(text "Firmware toggles WDI in software (50-1000 Hz, ~50% duty) only while the control loop is healthy.\nNever drive WDI from a timer/PWM: a timer keeps running after the CPU hangs.\nEach falling edge on WDI pulls the Q24 gate low through C169 and tops up C170 via R178.\nWD_OK ~2.7 V while toggling. WDI stuck high, low or floating: <1 V in ~100 ms, <0.4 V in ~190 ms\n(10 uF nominal; DC-bias derating shortens this). WD_OK starts at 0 V at power-up (fail-safe).\nWD_OK drives N-FET gates only (14.4 V rail switch, water pump, LiDAR incl. laser): no resistive loads.\nWDI pin: high-Z at reset, no pull-down. All parts reuse existing BOM lines."
 		(exclude_from_sim no)
 		(at 69.85 140.97 0)
@@
 		(in_pos_files yes)
 		(dnp no)
-		(property "Reference" "R7002"
+		(property "Reference" "R177"
 			(at 87.63 81.915 0)
 			(show_name no)
@@
 			(project "Main"
 				(path "/dbcfb655-8d45-4808-9a74-2a0eb03372e8/7f043eef-851b-4fc7-bc1b-c170004bfbd9"
-					(reference "R7002")
+					(reference "R177")
 					(unit 1)
 				)
@@
 		(in_pos_files yes)
 		(dnp no)
-		(property "Reference" "R7003"
+		(property "Reference" "R178"
 			(at 105.41 100.965 0)
 			(show_name no)
@@
 			)
 		)
-		(property "Description" "Charge current limit into C7002"
+		(property "Description" "Charge current limit into C170"
 			(at 102.87 101.6 0)
 			(hide yes)
@@
 			(project "Main"
 				(path "/dbcfb655-8d45-4808-9a74-2a0eb03372e8/7f043eef-851b-4fc7-bc1b-c170004bfbd9"
-					(reference "R7003")
+					(reference "R178")
 					(unit 1)
 				)
@@
 		(in_pos_files yes)
 		(dnp no)
-		(property "Reference" "C7002"
+		(property "Reference" "C170"
 			(at 112.395 112.395 0)
 			(show_name no)
@@
 			)
 		)
-		(property "Description" "Hold capacitor: sets timeout with R7004"
+		(property "Description" "Hold capacitor: sets timeout with R179"
 			(at 110.49 113.03 0)
 			(hide yes)
@@
 			(project "Main"
 				(path "/dbcfb655-8d45-4808-9a74-2a0eb03372e8/7f043eef-851b-4fc7-bc1b-c170004bfbd9"
-					(reference "C7002")
+					(reference "C170")
 					(unit 1)
 				)
@@
 		(in_pos_files yes)
 		(dnp no)
-		(property "Reference" "C7001"
+		(property "Reference" "C169"
 			(at 84.455 95.25 90)
 			(show_name no)
@@
 			(project "Main"
 				(path "/dbcfb655-8d45-4808-9a74-2a0eb03372e8/7f043eef-851b-4fc7-bc1b-c170004bfbd9"
-					(reference "C7001")
+					(reference "C169")
 					(unit 1)
 				)
@@
 		(in_pos_files yes)
 		(dnp no)
-		(property "Reference" "Q7001"
+		(property "Reference" "Q24"
 			(at 109.22 90.805 0)
 			(show_name no)
@@
 			(project "Main"
 				(path "/dbcfb655-8d45-4808-9a74-2a0eb03372e8/7f043eef-851b-4fc7-bc1b-c170004bfbd9"
-					(reference "Q7001")
+					(reference "Q24")
 					(unit 1)
 				)
@@
 		(in_pos_files yes)
 		(dnp no)
-		(property "Reference" "R7004"
+		(property "Reference" "R179"
 			(at 128.27 112.395 0)
 			(show_name no)
@@
 			(project "Main"
 				(path "/dbcfb655-8d45-4808-9a74-2a0eb03372e8/7f043eef-851b-4fc7-bc1b-c170004bfbd9"
-					(reference "R7004")
+					(reference "R179")
 					(unit 1)
 				)
@@
 		(in_pos_files yes)
 		(dnp no)
-		(property "Reference" "R7001"
+		(property "Reference" "R176"
 			(at 74.295 95.25 90)
 			(show_name no)
@@
 			)
 		)
-		(property "Description" "Series R: limits GPIO edge current into C7001"
+		(property "Description" "Series R: limits GPIO edge current into C169"
 			(at 77.47 91.44 0)
 			(hide yes)
@@
 			(project "Main"
 				(path "/dbcfb655-8d45-4808-9a74-2a0eb03372e8/7f043eef-851b-4fc7-bc1b-c170004bfbd9"
-					(reference "R7001")
+					(reference "R176")
 					(unit 1)
 				)
