File: kicad/charging-dock/Control.kicad_sch (KiCad schematic)
At the start: 9 parts, among them J8201 DEBUG (DNP), U8201 CH32V003F4P6, U8202 IRM-H638T (DNP)

Commit message: Side sensor board rev 2 (VL53L0X + IRM-H638T, JST SH); mounting holes on dock and sensor boards
- kicad/side-sensors: VL53L0X (C91199) replaces the NRND VL6180 and its 2.8 V LDO;
  top-looking IRM-H638T replaces the TSOP38238; ZX-SH1.0-7PWT connector, same pinout;
  10k XSHUT/GPIO1 pull-ups, no local I2C pull-ups; refs 84xx; libs from ../main
- main-phone SIDE-R1: ZX-ZH1.5-7PWT -> ZX-SH1.0-7PWT
- mounting holes: dock 4x M3 (H8201-H8204), ToF board 2x M2 (H8301/H8302),
  side board 2x M2 (H8401/H8402)
- JLCImport: VL53L0CXV0DH_1 symbol, footprint, 3D model
- docs: side board README, SPEC, READMEs; IRM-H638T pinout confirmed

Co-Authored-By: Claude Opus 5.5 (1M context) <noreply@anthropic.com>
Parts:
- added H8201, H8202, H8203, H8204: M3, MountingHole:MountingHole_3.2mm_M3_Pad, symbol Mechanical:MountingHole_Pad
Connections:
- net GND: now also H8201.1, H8202.1, H8203.1, H8204.1
Other:
- note added: "Mounting: 4x M3 (pads to GND)"

Commit message: Per-board reference ranges, J1 spare header, IMU AD0 pull-down, BOM outputs
- reference ranges: main-phone 1-999, dock 1000s, front ToF 2000s, side 3000s,
  cliff 4000s, rear IR 5000s, Hall 6000s (main-phone 7xxx parts renumbered
  below 1000; sensor boards and dock moved from 8xxx)
- main-phone: J7301 -> J1, a fitted 2x7 0.1" header with spares only
  (3.3 V, 5 V, I2C4, UART PC10/PC11, PA8-PA10, PD4, PE2, PE6, GND)
- IMU: AP_AD0 pulled low by R217 (address 0x68); INT2 on test pad TP1;
  FSYNC reachable on R211; R18/R72 removed
- tools/export.py replaces export_pdfs.py: schematic PDF and JLC-style BOM in
  each board's output/ folder; --pcb adds Gerbers, placement and STEP
- cliff and rear IR projects: fix top-level sheet left over from a copy
- Hall board: visual tidy-up

Co-Authored-By: Claude Opus 5.5 <noreply@anthropic.com>
Parts:
- renumbered C8201 to C1201, C8202 to C1202, C8203 to C1203, D8201 to D1201, H8201 to H1201, H8202 to H1202, H8203 to H1203, H8204 to H1204, J8201 to J1201, R8201 to R1201, R8202 to R1202, U8201 to U1201, U8202 to U1202
Changed lines of the file:
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@@
 		(in_pos_files yes)
 		(dnp no)
-		(property "Reference" "U8201"
+		(property "Reference" "U1201"
 			(at 142.24 73.66 0)
 			(show_name no)
@@
 			(project "Charging Dock"
 				(path "/b1780c3e-7100-4df4-97c9-2fd6186fb125/98be3a95-74c8-4a8a-bf9d-07f6f90f1855"
-					(reference "U8201")
+					(reference "U1201")
 					(unit 1)
 				)
@@
 		(in_pos_files yes)
 		(dnp no)
-		(property "Reference" "C8201"
+		(property "Reference" "C1201"
 			(at 171.45 71.12 0)
 			(show_name no)
@@
 			(project "Charging Dock"
 				(path "/b1780c3e-7100-4df4-97c9-2fd6186fb125/98be3a95-74c8-4a8a-bf9d-07f6f90f1855"
-					(reference "C8201")
+					(reference "C1201")
 					(unit 1)
 				)
@@
 		(in_pos_files yes)
 		(dnp no)
-		(property "Reference" "C8202"
+		(property "Reference" "C1202"
 			(at 186.69 71.12 0)
 			(show_name no)
@@
 			(project "Charging Dock"
 				(path "/b1780c3e-7100-4df4-97c9-2fd6186fb125/98be3a95-74c8-4a8a-bf9d-07f6f90f1855"
-					(reference "C8202")
+					(reference "C1202")
 					(unit 1)
 				)
@@
 		(in_pos_files yes)
 		(dnp no)
-		(property "Reference" "R8201"
+		(property "Reference" "R1201"
 			(at 60.96 46.99 90)
 			(show_name no)
@@
 			(project "Charging Dock"
 				(path "/b1780c3e-7100-4df4-97c9-2fd6186fb125/98be3a95-74c8-4a8a-bf9d-07f6f90f1855"
-					(reference "R8201")
+					(reference "R1201")
 					(unit 1)
 				)
@@
 		(in_pos_files yes)
 		(dnp no)
-		(property "Reference" "D8201"
+		(property "Reference" "D1201"
 			(at 72.39 44.45 0)
 			(show_name no)
@@
 			(project "Charging Dock"
 				(path "/b1780c3e-7100-4df4-97c9-2fd6186fb125/98be3a95-74c8-4a8a-bf9d-07f6f90f1855"
-					(reference "D8201")
+					(reference "D1201")
 					(unit 1)
 				)
@@
 		(in_pos_files yes)
 		(dnp yes)
-		(property "Reference" "J8201"
+		(property "Reference" "J1201"
 			(at 45.72 123.19 0)
 			(show_name no)
@@
 			(project "Charging Dock"
 				(path "/b1780c3e-7100-4df4-97c9-2fd6186fb125/98be3a95-74c8-4a8a-bf9d-07f6f90f1855"
-					(reference "J8201")
+					(reference "J1201")
 					(unit 1)
 				)
@@
 		(in_pos_files yes)
 		(dnp yes)
-		(property "Reference" "U8202"
+		(property "Reference" "U1202"
 			(at 226.06 123.19 0)
 			(show_name no)
@@
 			(project "Charging Dock"
 				(path "/b1780c3e-7100-4df4-97c9-2fd6186fb125/98be3a95-74c8-4a8a-bf9d-07f6f90f1855"
-					(reference "U8202")
+					(reference "U1202")
 					(unit 1)
 				)
@@
 		(in_pos_files yes)
 		(dnp yes)
-		(property "Reference" "R8202"
+		(property "Reference" "R1202"
 			(at 203.2 140.97 90)
 			(show_name no)
@@
 			(project "Charging Dock"
 				(path "/b1780c3e-7100-4df4-97c9-2fd6186fb125/98be3a95-74c8-4a8a-bf9d-07f6f90f1855"
-					(reference "R8202")
+					(reference "R1202")
 					(unit 1)
 				)
@@
 		(in_pos_files yes)
 		(dnp yes)
-		(property "Reference" "C8203"
+		(property "Reference" "C1203"
 			(at 214.63 142.24 0)
 			(show_name no)
@@
 			(project "Charging Dock"
 				(path "/b1780c3e-7100-4df4-97c9-2fd6186fb125/98be3a95-74c8-4a8a-bf9d-07f6f90f1855"
-					(reference "C8203")
+					(reference "C1203")
 					(unit 1)
 				)
@@
 		(in_pos_files no)
 		(dnp no)
-		(property "Reference" "H8201"
+		(property "Reference" "H1201"
 			(at 213.36 40.64 0)
 			(show_name no)
@@
 			(project "Charging Dock"
 				(path "C:/Program Files/Git/b1780c3e-7100-4df4-97c9-2fd6186fb125/98be3a95-74c8-4a8a-bf9d-07f6f90f1855"
-					(reference "H8201")
+					(reference "H1201")
 					(unit 1)
 				)
@@
 		(in_pos_files no)
 		(dnp no)
-		(property "Reference" "H8202"
+		(property "Reference" "H1202"
 			(at 228.6 40.64 0)
 			(show_name no)
@@
 			(project "Charging Dock"
 				(path "C:/Program Files/Git/b1780c3e-7100-4df4-97c9-2fd6186fb125/98be3a95-74c8-4a8a-bf9d-07f6f90f1855"
-					(reference "H8202")
+					(reference "H1202")
 					(unit 1)
 				)
@@
 		(in_pos_files no)
 		(dnp no)
-		(property "Reference" "H8203"
+		(property "Reference" "H1203"
 			(at 243.84 40.64 0)
 			(show_name no)
@@
 			(project "Charging Dock"
 				(path "C:/Program Files/Git/b1780c3e-7100-4df4-97c9-2fd6186fb125/98be3a95-74c8-4a8a-bf9d-07f6f90f1855"
-					(reference "H8203")
+					(reference "H1203")
 					(unit 1)
 				)
@@
 		(in_pos_files no)
 		(dnp no)
-		(property "Reference" "H8204"
+		(property "Reference" "H1204"
 			(at 259.08 40.64 0)
 			(show_name no)
@@
 			(project "Charging Dock"
 				(path "C:/Program Files/Git/b1780c3e-7100-4df4-97c9-2fd6186fb125/98be3a95-74c8-4a8a-bf9d-07f6f90f1855"
-					(reference "H8204")
+					(reference "H1204")
 					(unit 1)
 				)
