File: kicad/cliff-sensor/Cliff Sensor.kicad_sch (KiCad schematic)
At the start: 4 parts, among them J8501 ZX-SH1_0-4PLT, Q8501 PT333-3B

Commit message: Per-board reference ranges, J1 spare header, IMU AD0 pull-down, BOM outputs
- reference ranges: main-phone 1-999, dock 1000s, front ToF 2000s, side 3000s,
  cliff 4000s, rear IR 5000s, Hall 6000s (main-phone 7xxx parts renumbered
  below 1000; sensor boards and dock moved from 8xxx)
- main-phone: J7301 -> J1, a fitted 2x7 0.1" header with spares only
  (3.3 V, 5 V, I2C4, UART PC10/PC11, PA8-PA10, PD4, PE2, PE6, GND)
- IMU: AP_AD0 pulled low by R217 (address 0x68); INT2 on test pad TP1;
  FSYNC reachable on R211; R18/R72 removed
- tools/export.py replaces export_pdfs.py: schematic PDF and JLC-style BOM in
  each board's output/ folder; --pcb adds Gerbers, placement and STEP
- cliff and rear IR projects: fix top-level sheet left over from a copy
- Hall board: visual tidy-up

Co-Authored-By: Claude Opus 5.5 <noreply@anthropic.com>
Parts:
- renumbered D8501 to D4001, J8501 to J4001, Q8501 to Q4001, R8501 to R4001
Other:
- note added: "Assembly (JLC): D4001 and Q4001 THT with the assembly standoff (~2 mm) so the leads can be bent; pin bending to the tilt angle, or bend by hand in the 3D-printed housing. LED: flat side = cathode. Q8501: flat side / square pad = emitter. Spacing D4001-Q4001: 18 mm centre to centre."
- note added: "J4001 to the main board, pin 1 to pin 1: 1 VLED (5 V), 2 LED cathode (main board switches it), 3 OUT, 4 GND"
- note removed: "Assembly (JLC): D8501 and Q8501 THT with the assembly standoff (~2 mm) so the leads can be bent; pin bending to the tilt angle, or bend by hand in the 3D-printed housing. LED: flat side = cathode. Q8501: flat side / square pad = emitter. Spacing D8501-Q8501: 18 mm centre to centre."
- note removed: "J8501 to the main board, pin 1 to pin 1: 1 VLED (5 V), 2 LED cathode (main board switches it), 3 OUT, 4 GND"
Changed lines of the file:
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@@
 		(in_pos_files yes)
 		(dnp no)
-		(property "Reference" "J8501"
+		(property "Reference" "J4001"
 			(at 59.69 88.9 0)
 			(show_name no)
@@
 			(project "Cliff Sensor"
 				(path "/6f0d3b52-3a8e-4b0e-9f5c-2c1e8a7d4b19"
-					(reference "J8501")
+					(reference "J4001")
 					(unit 1)
 				)
@@
 		(in_pos_files yes)
 		(dnp no)
-		(property "Reference" "#PWR8501"
+		(property "Reference" "#PWR4001"
 			(at 72.39 105.41 90)
 			(hide yes)
@@
 			(project "Cliff Sensor"
 				(path "/6f0d3b52-3a8e-4b0e-9f5c-2c1e8a7d4b19"
-					(reference "#PWR8501")
+					(reference "#PWR4001")
 					(unit 1)
 				)
@@
 		(in_pos_files yes)
 		(dnp no)
-		(property "Reference" "#PWR8502"
+		(property "Reference" "#PWR4002"
 			(at 60.96 115.57 0)
 			(hide yes)
@@
 			(project "Cliff Sensor"
 				(path "/6f0d3b52-3a8e-4b0e-9f5c-2c1e8a7d4b19"
-					(reference "#PWR8502")
+					(reference "#PWR4002")
 					(unit 1)
 				)
@@
 		(in_pos_files yes)
 		(dnp no)
-		(property "Reference" "#PWR8503"
+		(property "Reference" "#PWR4003"
 			(at 60.96 87.63 0)
 			(hide yes)
@@
 			(project "Cliff Sensor"
 				(path "/6f0d3b52-3a8e-4b0e-9f5c-2c1e8a7d4b19"
-					(reference "#PWR8503")
+					(reference "#PWR4003")
 					(unit 1)
 				)
@@
 		(in_pos_files yes)
 		(dnp no)
-		(property "Reference" "#FLG8504"
+		(property "Reference" "#FLG4004"
 			(at 72.39 105.41 0)
 			(hide yes)
@@
 			(project "Cliff Sensor"
 				(path "/6f0d3b52-3a8e-4b0e-9f5c-2c1e8a7d4b19"
-					(reference "#FLG8504")
+					(reference "#FLG4004")
 					(unit 1)
 				)
@@
 		)
 	)
-	(text "J8501 to the main board, pin 1 to pin 1:\n1 VLED (5 V), 2 LED cathode (main board\nswitches it), 3 OUT, 4 GND"
+	(text "J4001 to the main board, pin 1 to pin 1:\n1 VLED (5 V), 2 LED cathode (main board\nswitches it), 3 OUT, 4 GND"
 		(exclude_from_sim no)
 		(at 50.8 127 0)
@@
 		(in_pos_files yes)
 		(dnp no)
-		(property "Reference" "R8501"
+		(property "Reference" "R4001"
 			(at 101.6 100.33 0)
 			(show_name no)
@@
 			(project "Cliff Sensor"
 				(path "/6f0d3b52-3a8e-4b0e-9f5c-2c1e8a7d4b19"
-					(reference "R8501")
+					(reference "R4001")
 					(unit 1)
 				)
@@
 		(in_pos_files yes)
 		(dnp no)
-		(property "Reference" "D8501"
+		(property "Reference" "D4001"
 			(at 123.19 96.52 0)
 			(show_name no)
@@
 			(project "Cliff Sensor"
 				(path "/6f0d3b52-3a8e-4b0e-9f5c-2c1e8a7d4b19"
-					(reference "D8501")
+					(reference "D4001")
 					(unit 1)
 				)
@@
 		(in_pos_files yes)
 		(dnp no)
-		(property "Reference" "Q8501"
+		(property "Reference" "Q4001"
 			(at 166.37 100.33 0)
 			(show_name no)
@@
 			)
 		)
-		(property "Description" "NPN phototransistor, 5 mm black (visible-blocking) lens; THT with standoff, leads bent like D8501"
+		(property "Description" "NPN phototransistor, 5 mm black (visible-blocking) lens; THT with standoff, leads bent like D4001"
 			(at 160.02 101.6 0)
 			(hide yes)
@@
 			(project "Cliff Sensor"
 				(path "/6f0d3b52-3a8e-4b0e-9f5c-2c1e8a7d4b19"
-					(reference "Q8501")
+					(reference "Q4001")
 					(unit 1)
 				)
@@
 		(in_pos_files yes)
 		(dnp no)
-		(property "Reference" "#PWR8505"
+		(property "Reference" "#PWR4005"
 			(at 163.83 111.76 0)
 			(hide yes)
@@
 			(project "Cliff Sensor"
 				(path "/6f0d3b52-3a8e-4b0e-9f5c-2c1e8a7d4b19"
-					(reference "#PWR8505")
+					(reference "#PWR4005")
 					(unit 1)
 				)
@@
 		)
 	)
-	(text "OOMWOO cliff sensor board (rev 1, 2026-10-28). One design, fitted 6x. No lenses: narrow-beam 5 mm parts (IR333-A 20 deg,\nPT333-3B black lens) tilted toward each other so their beams cross at the floor. The tilt sets the reference distance:\ncrossing depth = (spacing / 2) / tan(tilt), e.g. 18 mm spacing: 30 deg -> 15.6 mm, 25 deg -> 19.3 mm, 20 deg -> 24.7 mm.\nBeyond the crossing point the beams diverge, so a far floor (a cliff) returns little light even if it is white.\nThe main board switches the LED cathode (CLIFF_LED_EN, modulate it to cancel ambient light) and pulls OUT up (47k).\nRefs 85xx: unique on the OOMWOO panel."
+	(text "OOMWOO cliff sensor board (rev 1, 2026-10-28). One design, fitted 6x. No lenses: narrow-beam 5 mm parts (IR333-A 20 deg,\nPT333-3B black lens) tilted toward each other so their beams cross at the floor. The tilt sets the reference distance:\ncrossing depth = (spacing / 2) / tan(tilt), e.g. 18 mm spacing: 30 deg -> 15.6 mm, 25 deg -> 19.3 mm, 20 deg -> 24.7 mm.\nBeyond the crossing point the beams diverge, so a far floor (a cliff) returns little light even if it is white.\nThe main board switches the LED cathode (CLIFF_LED_EN, modulate it to cancel ambient light) and pulls OUT up (47k).\nRefs in the 4000s: each board has its own range."
 		(exclude_from_sim no)
 		(at 30.48 25.4 0)
@@
 		)
 	)
-	(text "Assembly (JLC): D8501 and Q8501 THT with the assembly standoff (~2 mm) so the leads can be bent;\npin bending to the tilt angle, or bend by hand in the 3D-printed housing. LED: flat side = cathode.\nQ8501: flat side / square pad = emitter. Spacing D8501-Q8501: 18 mm centre to centre."
+	(text "Assembly (JLC): D4001 and Q4001 THT with the assembly standoff (~2 mm) so the leads can be bent;\npin bending to the tilt angle, or bend by hand in the 3D-printed housing. LED: flat side = cathode.\nQ8501: flat side / square pad = emitter. Spacing D4001-Q4001: 18 mm centre to centre."
 		(exclude_from_sim no)
 		(at 88.9 142.24 0)
