File: kicad/front-sensors/Front Sensor.kicad_sch (KiCad schematic)
At the start: 8 parts, among them J8301 ZX-SH1_0-7PWT, U8301 VL53L7CHV0GC/1

Commit message: Per-board reference ranges, J1 spare header, IMU AD0 pull-down, BOM outputs
- reference ranges: main-phone 1-999, dock 1000s, front ToF 2000s, side 3000s,
  cliff 4000s, rear IR 5000s, Hall 6000s (main-phone 7xxx parts renumbered
  below 1000; sensor boards and dock moved from 8xxx)
- main-phone: J7301 -> J1, a fitted 2x7 0.1" header with spares only
  (3.3 V, 5 V, I2C4, UART PC10/PC11, PA8-PA10, PD4, PE2, PE6, GND)
- IMU: AP_AD0 pulled low by R217 (address 0x68); INT2 on test pad TP1;
  FSYNC reachable on R211; R18/R72 removed
- tools/export.py replaces export_pdfs.py: schematic PDF and JLC-style BOM in
  each board's output/ folder; --pcb adds Gerbers, placement and STEP
- cliff and rear IR projects: fix top-level sheet left over from a copy
- Hall board: visual tidy-up

Co-Authored-By: Claude Opus 5.5 <noreply@anthropic.com>
Parts:
- renumbered C8301 to C2001, C8302 to C2002, C8303 to C2003, C8304 to C2004, J8301 to J2001, L8301 to L2001, R8301 to R2001, U8301 to U2001
Other:
- note added: "IOVDD: C2003, C2004 AVDD: C2001, C2002 Place each pair at its pins."
- note added: "J2001 pin 1 to main-board pin 1: use a same-direction (pin 1 - pin 1) SH 7-pin cable"
- note added: "OOMWOO front ToF board (rev 2, 2026-10-27). One design, fitted twice: left and right, each aimed 30 deg off centre. The main board holds the I2C (2.2k), INT, LPn (47k) and I2C_RST (47k) resistors, so this board carries none of them. Refs in the 2000s: each board has its own range."
- note removed: "IOVDD: C8303, C8304 AVDD: C8301, C8302 Place each pair at its pins."
- note removed: "J8301 pin 1 to main-board pin 1: use a same-direction (pin 1 - pin 1) SH 7-pin cable"
- note removed: "OOMWOO front ToF board (rev 2, 2026-10-27). One design, fitted twice: left and right, each aimed 30 deg off centre. The main board holds the I2C (2.2k), INT, LPn (47k) and I2C_RST (47k) resistors, so this board carries none of them. Refs 83xx: unique on the OOMWOO panel."
Changed lines of the file:
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@@
 		(in_pos_files yes)
 		(dnp no)
-		(property "Reference" "J8301"
+		(property "Reference" "J2001"
 			(at 59.69 85.09 0)
 			(show_name no)
@@
 			(project "Front Sensor"
 				(path "/b1780c3e-7100-4df4-97c9-2fd6186fb125"
-					(reference "J8301")
+					(reference "J2001")
 					(unit 1)
 				)
@@
 		(in_pos_files yes)
 		(dnp no)
-		(property "Reference" "#PWR8301"
+		(property "Reference" "#PWR2001"
 			(at 73.66 93.98 90)
 			(hide yes)
@@
 			(project "Front Sensor"
 				(path "/b1780c3e-7100-4df4-97c9-2fd6186fb125"
-					(reference "#PWR8301")
+					(reference "#PWR2001")
 					(unit 1)
 				)
@@
 		(in_pos_files yes)
 		(dnp no)
-		(property "Reference" "#PWR8302"
+		(property "Reference" "#PWR2002"
 			(at 73.66 96.52 90)
 			(hide yes)
@@
 			(project "Front Sensor"
 				(path "/b1780c3e-7100-4df4-97c9-2fd6186fb125"
-					(reference "#PWR8302")
+					(reference "#PWR2002")
 					(unit 1)
 				)
@@
 		(in_pos_files yes)
 		(dnp no)
-		(property "Reference" "#PWR8303"
+		(property "Reference" "#PWR2003"
 			(at 62.23 116.84 0)
 			(hide yes)
@@
 			(project "Front Sensor"
 				(path "/b1780c3e-7100-4df4-97c9-2fd6186fb125"
-					(reference "#PWR8303")
+					(reference "#PWR2003")
 					(unit 1)
 				)
@@
 		(color 0 0 0 0)
 	)
-	(text "J8301 pin 1 to main-board pin 1:\nuse a same-direction (pin 1 - pin 1)\nSH 7-pin cable"
+	(text "J2001 pin 1 to main-board pin 1:\nuse a same-direction (pin 1 - pin 1)\nSH 7-pin cable"
 		(exclude_from_sim no)
 		(at 48.26 132.08 0)
@@
 		(in_pos_files no)
 		(dnp no)
-		(property "Reference" "U8301"
+		(property "Reference" "U2001"
 			(at 147.32 82.55 0)
 			(show_name no)
@@
 			(project "Front Sensor"
 				(path "/b1780c3e-7100-4df4-97c9-2fd6186fb125"
-					(reference "U8301")
+					(reference "U2001")
 					(unit 1)
 				)
@@
 		(in_pos_files yes)
 		(dnp no)
-		(property "Reference" "#PWR8304"
+		(property "Reference" "#PWR2004"
 			(at 129.54 115.57 0)
 			(hide yes)
@@
 			(project "Front Sensor"
 				(path "/b1780c3e-7100-4df4-97c9-2fd6186fb125"
-					(reference "#PWR8304")
+					(reference "#PWR2004")
 					(unit 1)
 				)
@@
 		(in_pos_files yes)
 		(dnp no)
-		(property "Reference" "#PWR8305"
+		(property "Reference" "#PWR2005"
 			(at 173.99 110.49 0)
 			(hide yes)
@@
 			(project "Front Sensor"
 				(path "/b1780c3e-7100-4df4-97c9-2fd6186fb125"
-					(reference "#PWR8305")
+					(reference "#PWR2005")
 					(unit 1)
 				)
@@
 		(in_pos_files yes)
 		(dnp no)
-		(property "Reference" "#PWR8306"
+		(property "Reference" "#PWR2006"
 			(at 181.61 92.71 90)
 			(hide yes)
@@
 			(project "Front Sensor"
 				(path "/b1780c3e-7100-4df4-97c9-2fd6186fb125"
-					(reference "#PWR8306")
+					(reference "#PWR2006")
 					(unit 1)
 				)
@@
 		(in_pos_files yes)
 		(dnp no)
-		(property "Reference" "R8301"
+		(property "Reference" "R2001"
 			(at 179.07 115.57 90)
 			(show_name no)
@@
 			(project "Front Sensor"
 				(path "/b1780c3e-7100-4df4-97c9-2fd6186fb125"
-					(reference "R8301")
+					(reference "R2001")
 					(unit 1)
 				)
@@
 		(in_pos_files yes)
 		(dnp no)
-		(property "Reference" "#PWR8307"
+		(property "Reference" "#PWR2007"
 			(at 187.96 118.11 90)
 			(hide yes)
@@
 			(project "Front Sensor"
 				(path "/b1780c3e-7100-4df4-97c9-2fd6186fb125"
-					(reference "#PWR8307")
+					(reference "#PWR2007")
 					(unit 1)
 				)
@@
 		(in_pos_files yes)
 		(dnp no)
-		(property "Reference" "#PWR8308"
+		(property "Reference" "#PWR2008"
 			(at 190.5 50.8 0)
 			(hide yes)
@@
 			(project "Front Sensor"
 				(path "/b1780c3e-7100-4df4-97c9-2fd6186fb125"
-					(reference "#PWR8308")
+					(reference "#PWR2008")
 					(unit 1)
 				)
@@
 		(in_pos_files yes)
 		(dnp no)
-		(property "Reference" "L8301"
+		(property "Reference" "L2001"
 			(at 199.39 49.53 0)
 			(show_name no)
@@
 			(project "Front Sensor"
 				(path "/b1780c3e-7100-4df4-97c9-2fd6186fb125"
-					(reference "L8301")
+					(reference "L2001")
 					(unit 1)
 				)
@@
 		(in_pos_files yes)
 		(dnp no)
-		(property "Reference" "C8303"
+		(property "Reference" "C2003"
 			(at 176.53 59.69 0)
 			(show_name no)
@@
 			(project "Front Sensor"
 				(path "/b1780c3e-7100-4df4-97c9-2fd6186fb125"
-					(reference "C8303")
+					(reference "C2003")
 					(unit 1)
 				)
@@
 		(in_pos_files yes)
 		(dnp no)
-		(property "Reference" "#PWR8309"
+		(property "Reference" "#PWR2009"
 			(at 175.26 64.77 0)
 			(hide yes)
@@
 			(project "Front Sensor"
 				(path "/b1780c3e-7100-4df4-97c9-2fd6186fb125"
-					(reference "#PWR8309")
+					(reference "#PWR2009")
 					(unit 1)
 				)
@@
 		(in_pos_files yes)
 		(dnp no)
-		(property "Reference" "C8304"
+		(property "Reference" "C2004"
 			(at 161.29 59.69 0)
 			(show_name no)
@@
 			(project "Front Sensor"
 				(path "/b1780c3e-7100-4df4-97c9-2fd6186fb125"
-					(reference "C8304")
+					(reference "C2004")
 					(unit 1)
 				)
@@
 		(in_pos_files yes)
 		(dnp no)
-		(property "Reference" "#PWR8310"
+		(property "Reference" "#PWR2010"
 			(at 160.02 64.77 0)
 			(hide yes)
@@
 			(project "Front Sensor"
 				(path "/b1780c3e-7100-4df4-97c9-2fd6186fb125"
-					(reference "#PWR8310")
+					(reference "#PWR2010")
 					(unit 1)
 				)
@@
 		(in_pos_files yes)
 		(dnp no)
-		(property "Reference" "C8301"
+		(property "Reference" "C2001"
 			(at 217.17 59.69 0)
 			(show_name no)
@@
 			(project "Front Sensor"
 				(path "/b1780c3e-7100-4df4-97c9-2fd6186fb125"
-					(reference "C8301")
+					(reference "C2001")
 					(unit 1)
 				)
@@
 		(in_pos_files yes)
 		(dnp no)
-		(property "Reference" "#PWR8311"
+		(property "Reference" "#PWR2011"
 			(at 215.9 64.77 0)
 			(hide yes)
@@
 			(project "Front Sensor"
 				(path "/b1780c3e-7100-4df4-97c9-2fd6186fb125"
-					(reference "#PWR8311")
+					(reference "#PWR2011")
 					(unit 1)
 				)
@@
 		(in_pos_files yes)
 		(dnp no)
-		(property "Reference" "C8302"
+		(property "Reference" "C2002"
 			(at 232.41 59.69 0)
 			(show_name no)
@@
 			(project "Front Sensor"
 				(path "/b1780c3e-7100-4df4-97c9-2fd6186fb125"
-					(reference "C8302")
+					(reference "C2002")
 					(unit 1)
 				)
@@
 		(in_pos_files yes)
 		(dnp no)
-		(property "Reference" "#PWR8312"
+		(property "Reference" "#PWR2012"
 			(at 231.14 64.77 0)
 			(hide yes)
@@
 			(project "Front Sensor"
 				(path "/b1780c3e-7100-4df4-97c9-2fd6186fb125"
-					(reference "#PWR8312")
+					(reference "#PWR2012")
 					(unit 1)
 				)
@@
 		(in_pos_files yes)
 		(dnp no)
-		(property "Reference" "#FLG8313"
+		(property "Reference" "#FLG2013"
 			(at 160.02 53.34 0)
 			(hide yes)
@@
 			(project "Front Sensor"
 				(path "/b1780c3e-7100-4df4-97c9-2fd6186fb125"
-					(reference "#FLG8313")
+					(reference "#FLG2013")
 					(unit 1)
 				)
@@
 		(in_pos_files yes)
 		(dnp no)
-		(property "Reference" "#FLG8314"
+		(property "Reference" "#FLG2014"
 			(at 62.23 116.84 0)
 			(hide yes)
@@
 			(project "Front Sensor"
 				(path "/b1780c3e-7100-4df4-97c9-2fd6186fb125"
-					(reference "#FLG8314")
+					(reference "#FLG2014")
 					(unit 1)
 				)
@@
 		)
 	)
-	(text "IOVDD: C8303, C8304     AVDD: C8301, C8302\nPlace each pair at its pins."
+	(text "IOVDD: C2003, C2004     AVDD: C2001, C2002\nPlace each pair at its pins."
 		(exclude_from_sim no)
 		(at 160.02 73.66 0)
@@
 		)
 	)
-	(text "OOMWOO front ToF board (rev 2, 2026-10-27). One design, fitted twice: left and right,\neach aimed 30 deg off centre. The main board holds the I2C (2.2k), INT, LPn (47k) and I2C_RST (47k)\nresistors, so this board carries none of them. Refs 83xx: unique on the OOMWOO panel."
+	(text "OOMWOO front ToF board (rev 2, 2026-10-27). One design, fitted twice: left and right,\neach aimed 30 deg off centre. The main board holds the I2C (2.2k), INT, LPn (47k) and I2C_RST (47k)\nresistors, so this board carries none of them. Refs in the 2000s: each board has its own range."
 		(exclude_from_sim no)
 		(at 30.48 30.48 0)
