File: kicad/rear-ir/Rear IR.kicad_sch (KiCad schematic)
At the start: 9 parts, among them J8601 ZX-SH1_0-4PLT, U8601 IRM-H638T/TR2, U8602 IRM-H638T/TR2

Commit message: Per-board reference ranges, J1 spare header, IMU AD0 pull-down, BOM outputs
- reference ranges: main-phone 1-999, dock 1000s, front ToF 2000s, side 3000s,
  cliff 4000s, rear IR 5000s, Hall 6000s (main-phone 7xxx parts renumbered
  below 1000; sensor boards and dock moved from 8xxx)
- main-phone: J7301 -> J1, a fitted 2x7 0.1" header with spares only
  (3.3 V, 5 V, I2C4, UART PC10/PC11, PA8-PA10, PD4, PE2, PE6, GND)
- IMU: AP_AD0 pulled low by R217 (address 0x68); INT2 on test pad TP1;
  FSYNC reachable on R211; R18/R72 removed
- tools/export.py replaces export_pdfs.py: schematic PDF and JLC-style BOM in
  each board's output/ folder; --pcb adds Gerbers, placement and STEP
- cliff and rear IR projects: fix top-level sheet left over from a copy
- Hall board: visual tidy-up

Co-Authored-By: Claude Opus 5.5 <noreply@anthropic.com>
Parts:
- renumbered C8601 to C5001, C8602 to C5002, H8601 to H5001, H8602 to H5002, J8601 to J5001, R8601 to R5001, R8602 to R5002, U8601 to U5001, U8602 to U5002
Other:
- note added: "J5001 to the main board REAR-IR1, pin 1 to pin 1: 1 3.3 V, 2 IR_L, 3 IR_R, 4 GND"
- note added: "OOMWOO rear docking IR board (rev 1, 2026-10-28). Two top-looking 38 kHz receivers (the same part as the side board and the dock's U1202) look out of the board face, which faces backward. Put them ~10 mm apart with a baffle between them: both see the dock = it is straight behind, one = steer that way. The outputs have internal pull-ups. Refs in the 5000s: each board has its own range."
- note added: "U5001 = left, U5002 = right, seen from behind the robot (looking at the board face)."
- note removed: "J8601 to the main board REAR-IR1, pin 1 to pin 1: 1 3.3 V, 2 IR_L, 3 IR_R, 4 GND"
- note removed: "OOMWOO rear docking IR board (rev 1, 2026-10-28). Two top-looking 38 kHz receivers (the same part as the side board and the dock's U8202) look out of the board face, which faces backward. Put them ~10 mm apart with a baffle between them: both see the dock = it is straight behind, one = steer that way. The outputs have internal pull-ups. Refs 86xx: unique on the OOMWOO panel."
- note removed: "U8601 = left, U8602 = right, seen from behind the robot (looking at the board face)."
Changed lines of the file:
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@@
 		(in_pos_files yes)
 		(dnp no)
-		(property "Reference" "J8601"
+		(property "Reference" "J5001"
 			(at 46.99 88.9 0)
 			(show_name no)
@@
 			(project "Rear IR"
 				(path "/8c2f6e1a-4d7b-4f3e-a9c5-1b2d3e4f5a61"
-					(reference "J8601")
+					(reference "J5001")
 					(unit 1)
 				)
@@
 		(in_pos_files yes)
 		(dnp no)
-		(property "Reference" "#PWR8601"
+		(property "Reference" "#PWR5001"
 			(at 59.69 105.41 90)
 			(hide yes)
@@
 			(project "Rear IR"
 				(path "/8c2f6e1a-4d7b-4f3e-a9c5-1b2d3e4f5a61"
-					(reference "#PWR8601")
+					(reference "#PWR5001")
 					(unit 1)
 				)
@@
 		(in_pos_files yes)
 		(dnp no)
-		(property "Reference" "#PWR8602"
+		(property "Reference" "#PWR5002"
 			(at 48.26 115.57 0)
 			(hide yes)
@@
 			(project "Rear IR"
 				(path "/8c2f6e1a-4d7b-4f3e-a9c5-1b2d3e4f5a61"
-					(reference "#PWR8602")
+					(reference "#PWR5002")
 					(unit 1)
 				)
@@
 		(in_pos_files yes)
 		(dnp no)
-		(property "Reference" "#PWR8603"
+		(property "Reference" "#PWR5003"
 			(at 48.26 87.63 0)
 			(hide yes)
@@
 			(project "Rear IR"
 				(path "/8c2f6e1a-4d7b-4f3e-a9c5-1b2d3e4f5a61"
-					(reference "#PWR8603")
+					(reference "#PWR5003")
 					(unit 1)
 				)
@@
 		(in_pos_files yes)
 		(dnp no)
-		(property "Reference" "#FLG8604"
+		(property "Reference" "#FLG5004"
 			(at 59.69 105.41 0)
 			(hide yes)
@@
 			(project "Rear IR"
 				(path "/8c2f6e1a-4d7b-4f3e-a9c5-1b2d3e4f5a61"
-					(reference "#FLG8604")
+					(reference "#FLG5004")
 					(unit 1)
 				)
@@
 		(in_pos_files yes)
 		(dnp no)
-		(property "Reference" "#PWR8605"
+		(property "Reference" "#PWR5005"
 			(at 59.69 92.71 0)
 			(hide yes)
@@
 			(project "Rear IR"
 				(path "/8c2f6e1a-4d7b-4f3e-a9c5-1b2d3e4f5a61"
-					(reference "#PWR8605")
+					(reference "#PWR5005")
 					(unit 1)
 				)
@@
 		(in_pos_files yes)
 		(dnp no)
-		(property "Reference" "#FLG8606"
+		(property "Reference" "#FLG5006"
 			(at 67.31 97.79 0)
 			(hide yes)
@@
 			(project "Rear IR"
 				(path "/8c2f6e1a-4d7b-4f3e-a9c5-1b2d3e4f5a61"
-					(reference "#FLG8606")
+					(reference "#FLG5006")
 					(unit 1)
 				)
@@
 		)
 	)
-	(text "J8601 to the main board REAR-IR1, pin 1 to pin 1:\n1 3.3 V, 2 IR_L, 3 IR_R, 4 GND"
+	(text "J5001 to the main board REAR-IR1, pin 1 to pin 1:\n1 3.3 V, 2 IR_L, 3 IR_R, 4 GND"
 		(exclude_from_sim no)
 		(at 38.1 127 0)
@@
 		(in_pos_files yes)
 		(dnp no)
-		(property "Reference" "U8601"
+		(property "Reference" "U5001"
 			(at 154.94 82.55 0)
 			(show_name no)
@@
 			(project "Rear IR"
 				(path "/8c2f6e1a-4d7b-4f3e-a9c5-1b2d3e4f5a61"
-					(reference "U8601")
+					(reference "U5001")
 					(unit 1)
 				)
@@
 		(in_pos_files yes)
 		(dnp no)
-		(property "Reference" "#PWR8607"
+		(property "Reference" "#PWR5007"
 			(at 139.7 86.36 90)
 			(hide yes)
@@
 			(project "Rear IR"
 				(path "/8c2f6e1a-4d7b-4f3e-a9c5-1b2d3e4f5a61"
-					(reference "#PWR8607")
+					(reference "#PWR5007")
 					(unit 1)
 				)
@@
 		(in_pos_files yes)
 		(dnp no)
-		(property "Reference" "C8601"
+		(property "Reference" "C5001"
 			(at 132.08 100.33 0)
 			(show_name no)
@@
 			(project "Rear IR"
 				(path "/8c2f6e1a-4d7b-4f3e-a9c5-1b2d3e4f5a61"
-					(reference "C8601")
+					(reference "C5001")
 					(unit 1)
 				)
@@
 		(in_pos_files yes)
 		(dnp no)
-		(property "Reference" "#PWR8608"
+		(property "Reference" "#PWR5008"
 			(at 129.54 107.95 0)
 			(hide yes)
@@
 			(project "Rear IR"
 				(path "/8c2f6e1a-4d7b-4f3e-a9c5-1b2d3e4f5a61"
-					(reference "#PWR8608")
+					(reference "#PWR5008")
 					(unit 1)
 				)
@@
 		(in_pos_files yes)
 		(dnp no)
-		(property "Reference" "R8601"
+		(property "Reference" "R5001"
 			(at 119.38 91.44 90)
 			(show_name no)
@@
 			(project "Rear IR"
 				(path "/8c2f6e1a-4d7b-4f3e-a9c5-1b2d3e4f5a61"
-					(reference "R8601")
+					(reference "R5001")
 					(unit 1)
 				)
@@
 		(in_pos_files yes)
 		(dnp no)
-		(property "Reference" "#PWR8609"
+		(property "Reference" "#PWR5009"
 			(at 115.57 88.9 0)
 			(hide yes)
@@
 			(project "Rear IR"
 				(path "/8c2f6e1a-4d7b-4f3e-a9c5-1b2d3e4f5a61"
-					(reference "#PWR8609")
+					(reference "#PWR5009")
 					(unit 1)
 				)
@@
 		(in_pos_files yes)
 		(dnp no)
-		(property "Reference" "U8602"
+		(property "Reference" "U5002"
 			(at 154.94 123.19 0)
 			(show_name no)
@@
 			(project "Rear IR"
 				(path "/8c2f6e1a-4d7b-4f3e-a9c5-1b2d3e4f5a61"
-					(reference "U8602")
+					(reference "U5002")
 					(unit 1)
 				)
@@
 		(in_pos_files yes)
 		(dnp no)
-		(property "Reference" "#PWR8610"
+		(property "Reference" "#PWR5010"
 			(at 139.7 127 90)
 			(hide yes)
@@
 			(project "Rear IR"
 				(path "/8c2f6e1a-4d7b-4f3e-a9c5-1b2d3e4f5a61"
-					(reference "#PWR8610")
+					(reference "#PWR5010")
 					(unit 1)
 				)
@@
 		(in_pos_files yes)
 		(dnp no)
-		(property "Reference" "C8602"
+		(property "Reference" "C5002"
 			(at 132.08 140.97 0)
 			(show_name no)
@@
 			(project "Rear IR"
 				(path "/8c2f6e1a-4d7b-4f3e-a9c5-1b2d3e4f5a61"
-					(reference "C8602")
+					(reference "C5002")
 					(unit 1)
 				)
@@
 		(in_pos_files yes)
 		(dnp no)
-		(property "Reference" "#PWR8611"
+		(property "Reference" "#PWR5011"
 			(at 129.54 148.59 0)
 			(hide yes)
@@
 			(project "Rear IR"
 				(path "/8c2f6e1a-4d7b-4f3e-a9c5-1b2d3e4f5a61"
-					(reference "#PWR8611")
+					(reference "#PWR5011")
 					(unit 1)
 				)
@@
 		(in_pos_files yes)
 		(dnp no)
-		(property "Reference" "R8602"
+		(property "Reference" "R5002"
 			(at 119.38 132.08 90)
 			(show_name no)
@@
 			(project "Rear IR"
 				(path "/8c2f6e1a-4d7b-4f3e-a9c5-1b2d3e4f5a61"
-					(reference "R8602")
+					(reference "R5002")
 					(unit 1)
 				)
@@
 		(in_pos_files yes)
 		(dnp no)
-		(property "Reference" "#PWR8612"
+		(property "Reference" "#PWR5012"
 			(at 115.57 129.54 0)
 			(hide yes)
@@
 			(project "Rear IR"
 				(path "/8c2f6e1a-4d7b-4f3e-a9c5-1b2d3e4f5a61"
-					(reference "#PWR8612")
+					(reference "#PWR5012")
 					(unit 1)
 				)
@@
 		)
 	)
-	(text "OOMWOO rear docking IR board (rev 1, 2026-10-28). Two top-looking 38 kHz receivers (the same part as the side board\nand the dock's U8202) look out of the board face, which faces backward. Put them ~10 mm apart with a baffle between\nthem: both see the dock = it is straight behind, one = steer that way. The outputs have internal pull-ups.\nRefs 86xx: unique on the OOMWOO panel."
+	(text "OOMWOO rear docking IR board (rev 1, 2026-10-28). Two top-looking 38 kHz receivers (the same part as the side board\nand the dock's U1202) look out of the board face, which faces backward. Put them ~10 mm apart with a baffle between\nthem: both see the dock = it is straight behind, one = steer that way. The outputs have internal pull-ups.\nRefs in the 5000s: each board has its own range."
 		(exclude_from_sim no)
 		(at 30.48 25.4 0)
@@
 		)
 	)
-	(text "U8601 = left, U8602 = right, seen from behind the robot\n(looking at the board face)."
+	(text "U5001 = left, U5002 = right, seen from behind the robot\n(looking at the board face)."
 		(exclude_from_sim no)
 		(at 127 160.02 0)
@@
 		(in_pos_files no)
 		(dnp no)
-		(property "Reference" "H8601"
+		(property "Reference" "H5001"
 			(at 78.74 149.86 0)
 			(show_name no)
@@
 			(project "Rear IR"
 				(path "/8c2f6e1a-4d7b-4f3e-a9c5-1b2d3e4f5a61"
-					(reference "H8601")
+					(reference "H5001")
 					(unit 1)
 				)
@@
 		(in_pos_files yes)
 		(dnp no)
-		(property "Reference" "#PWR8613"
+		(property "Reference" "#PWR5013"
 			(at 76.2 157.48 0)
 			(hide yes)
@@
 			(project "Rear IR"
 				(path "/8c2f6e1a-4d7b-4f3e-a9c5-1b2d3e4f5a61"
-					(reference "#PWR8613")
+					(reference "#PWR5013")
 					(unit 1)
 				)
@@
 		(in_pos_files no)
 		(dnp no)
-		(property "Reference" "H8602"
+		(property "Reference" "H5002"
 			(at 93.98 149.86 0)
 			(show_name no)
@@
 			(project "Rear IR"
 				(path "/8c2f6e1a-4d7b-4f3e-a9c5-1b2d3e4f5a61"
-					(reference "H8602")
+					(reference "H5002")
 					(unit 1)
 				)
@@
 		(in_pos_files yes)
 		(dnp no)
-		(property "Reference" "#PWR8614"
+		(property "Reference" "#PWR5014"
 			(at 91.44 157.48 0)
 			(hide yes)
@@
 			(project "Rear IR"
 				(path "/8c2f6e1a-4d7b-4f3e-a9c5-1b2d3e4f5a61"
-					(reference "#PWR8614")
+					(reference "#PWR5014")
 					(unit 1)
 				)
